File: pcb/dk2_00/dk2_00.kicad_sch (KiCad schematic)
At the start: 2 parts

Commit message: i'm back!
Connections:
- net +5V: no longer U?.39 (VSYS)
- net GND: now also U?.13 (GND), U?.18 (GND), U?.23 (GND), U?.28 (GND), U?.38 (GND), U?.8 (GND)
Other:
- sheet Multiplexer in renamed Multiplexer in 1
- added sheet Multiplexer in 2 (muxin.kicad_sch)
- sheet Multiplexer in 1 ports: added 4051_DATA; removed none
- moved on the sheet: U?

Commit message: eurorack thoughts
Other:
- added sheet CV (cv.kicad_sch)
Changed lines of the file:
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@@
+    )
+  )
+  (sheet (at 58.42 143.51) (size 41.91 26.67) (fields_autoplaced)
+    (stroke (width 0.1524) (type solid))
+    (fill (color 0 0 0 0.0000))
+    (property "Sheetname" "CV" (at 58.42 142.7984 0)
+      (effects (font (size 1.27 1.27)) (justify left bottom))
+    )
+    (property "Sheetfile" "cv.kicad_sch" (at 58.42 170.7646 0)
+      (effects (font (size 1.27 1.27)) (justify left top))
+    )
+    (instances
+      (project "dk2_00"
+        (path "/87a59a99-d509-467e-85da-26d34072acb7" (page "9"))
+      )
     )
   )

Commit message: oh that's what a multi unit symbol is
Parts:
- added J7, J8, J9: Conn_01x01_Pin, symbol Connector:Conn_01x01_Pin
- added SW1: SW_Push, symbol Switch:SW_Push
- gave numbers to parts that had none: 2
Connections:
- net +5V: now also U1.40 (VBUS)
- net GND: now also J1.9 (SHIELD), U1.3 (GND), U1.33 (AGND), U1.42 (GND), SW1.2
- net TAP_TEMPO_IN: now also SW1.1
- net GPIO_15: now reaches U1.20 (GPIO15)
- net GPIO_15: now also J7.1 (Pin_1)
- net GPIO_22: now reaches U1.29 (GPIO22)
- net GPIO_22: now also J8.1 (Pin_1)
- net GPIO_28: now reaches U1.34 (GPIO28_ADC2)
- net GPIO_28: now also J9.1 (Pin_1)
- no-connect marks 2 -> 8
Other:
- removed sheet CV
- moved on the sheet: J1

Commit message: not many errors
Parts:
- renumbered J7 to J1, J8 to J2, J9 to J3, J1 to J4
Other:
- moved on the sheet: J1, J2, J3, J4, SW1, U1

Commit message: footprints assigned
Parts:
- J1, J2, J3: footprint (none) -> Connector_PinHeader_2.54mm:PinHeader_1x01_P2.54mm_Vertical
- J4: footprint (none) -> Connector_Card:microSD_HC_Molex_47219-2001
- SW1: footprint (none) -> Button_Switch_THT:SW_PUSH_6mm
- U1: footprint RPi_Pico:RPi_Pico_SMD_TH -> MCU_RaspberryPi_and_Boards:RPi_Pico_SMD_TH
Changed lines of the file:
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@@
       (effects (font (size 1.27 1.27)))
     )
-    (property "Footprint" "RPi_Pico:RPi_Pico_SMD_TH" (at 151.13 67.31 90)
+    (property "Footprint" "MCU_RaspberryPi_and_Boards:RPi_Pico_SMD_TH" (at 151.13 67.31 90)
       (effects (font (size 1.27 1.27)) hide)
     )
@@
       (effects (font (size 1.27 1.27)))
     )
-    (property "Footprint" "" (at 152.4 118.11 0)
+    (property "Footprint" "Connector_PinHeader_2.54mm:PinHeader_1x01_P2.54mm_Vertical" (at 152.4 118.11 0)
       (effects (font (size 1.27 1.27)) hide)
     )
@@
       (effects (font (size 1.27 1.27)))
     )
-    (property "Footprint" "" (at 152.4 125.73 0)
+    (property "Footprint" "Connector_PinHeader_2.54mm:PinHeader_1x01_P2.54mm_Vertical" (at 152.4 125.73 0)
       (effects (font (size 1.27 1.27)) hide)
     )
@@
       (effects (font (size 1.27 1.27)))
     )
-    (property "Footprint" "" (at 152.4 121.92 0)
+    (property "Footprint" "Connector_PinHeader_2.54mm:PinHeader_1x01_P2.54mm_Vertical" (at 152.4 121.92 0)
       (effects (font (size 1.27 1.27)) hide)
     )
@@
       (effects (font (size 1.27 1.27)))
     )
-    (property "Footprint" "" (at 152.4 134.62 0)
+    (property "Footprint" "Button_Switch_THT:SW_PUSH_6mm" (at 152.4 134.62 0)
       (effects (font (size 1.27 1.27)) hide)
     )
@@
       (effects (font (size 1.27 1.27)))
     )
-    (property "Footprint" "" (at 189.23 167.64 0)
-      (effects (font (size 1.27 1.27)) hide)
-    )
+    (property "Footprint" "Connector_Card:microSD_HC_Molex_47219-2001" (at 189.23 167.64 0)
+      (effects (font (size 1.27 1.27)) hide)
+    )

Commit message: eurorack power stuff
Other:
- added sheet Eurorack Power (europower.kicad_sch)
Changed lines of the file:
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@@
+    )
+  )
+  (sheet (at 49.53 138.43) (size 41.91 26.67) (fields_autoplaced)
+    (stroke (width 0.1524) (type solid))
+    (fill (color 0 0 0 0.0000))
+    (property "Sheetname" "Eurorack Power" (at 49.53 137.7184 0)
+      (effects (font (size 1.27 1.27)) (justify left bottom))
+    )
+    (property "Sheetfile" "europower.kicad_sch" (at 49.53 165.6846 0)
+      (effects (font (size 1.27 1.27)) (justify left top))
+    )
+    (property "Field2" "" (at 49.53 138.43 0)
+      (effects (font (size 1.27 1.27)) hide)
+    )
+    (instances
+      (project "dk2_00"
+        (path "/87a59a99-d509-467e-85da-26d34072acb7" (page "9"))
+      )
     )
   )

Commit message: making a mess
Other:
- added sheet CV in (cv_in.kicad_sch)
- added sheet CV out (cv_out.kicad_sch)
Changed lines of the file:
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@@
+    )
+  )
+  (sheet (at 49.53 177.8) (size 41.91 26.67) (fields_autoplaced)
+    (stroke (width 0.1524) (type solid))
+    (fill (color 0 0 0 0.0000))
+    (property "Sheetname" "CV in" (at 49.53 177.0884 0)
+      (effects (font (size 1.27 1.27)) (justify left bottom))
+    )
+    (property "Sheetfile" "cv_in.kicad_sch" (at 49.53 205.0546 0)
+      (effects (font (size 1.27 1.27)) (justify left top))
+    )
+    (property "Field2" "" (at 49.53 177.8 0)
+      (effects (font (size 1.27 1.27)) hide)
+    )
+    (instances
+      (project "dk2_00"
+        (path "/87a59a99-d509-467e-85da-26d34072acb7" (page "10"))
+      )
+    )
+  )
+  (sheet (at 49.53 218.44) (size 41.91 26.67) (fields_autoplaced)
+    (stroke (width 0.1524) (type solid))
+    (fill (color 0 0 0 0.0000))
+    (property "Sheetname" "CV out" (at 49.53 217.7284 0)
+      (effects (font (size 1.27 1.27)) (justify left bottom))
+    )
+    (property "Sheetfile" "cv_out.kicad_sch" (at 49.53 245.6946 0)
+      (effects (font (size 1.27 1.27)) (justify left top))
+    )
+    (property "Field2" "" (at 49.53 218.44 0)
+      (effects (font (size 1.27 1.27)) hide)
+    )
+    (instances
+      (project "dk2_00"
+        (path "/87a59a99-d509-467e-85da-26d34072acb7" (page "11"))
+      )
     )
   )
