File: pcb/dk2_00/cv_in.kicad_sch (KiCad schematic)
At the start: 1 part, among them U14 MCP6002-xSN

Commit message: nothing much
Parts:
- removed U14: MCP6002-xSN, symbol Amplifier_Operational:MCP6002-xSN
- added U15: MCP6002-xSN, symbol Amplifier_Operational:MCP6002-xSN
Changed lines of the file:
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@@
 (kicad_sch (version 20230121) (generator eeschema)
   (paper "A4")
-  (symbol (lib_id "Amplifier_Operational:MCP6002-xSN") (at 136.525 97.79 0) (unit 1)
+  (symbol (lib_id "Amplifier_Operational:MCP6002-xSN") (at 138.43 92.71 0) (unit 2)
     (in_bom yes) (on_board yes) (dnp no) (fields_autoplaced)
-    (property "Reference" "U14" (at 136.525 89.7001 0)
+    (property "Reference" "U15" (at 138.43 84.6201 0)
       (effects (font (size 1.27 1.27)))
     )
-    (property "Value" "MCP6002-xSN" (at 136.525 91.6211 0)
+    (property "Value" "MCP6002-xSN" (at 138.43 86.5411 0)
       (effects (font (size 1.27 1.27)))
     )
-    (property "Footprint" "" (at 136.525 97.79 0)
+    (property "Footprint" "" (at 138.43 92.71 0)
       (effects (font (size 1.27 1.27)) hide)
     )
-    (property "Datasheet" "http://ww1.microchip.com/downloads/en/DeviceDoc/21733j.pdf" (at 136.525 97.79 0)
+    (property "Datasheet" "http://ww1.microchip.com/downloads/en/DeviceDoc/21733j.pdf" (at 138.43 92.71 0)
       (effects (font (size 1.27 1.27)) hide)
     )
@@
       (project "dk2_00"
         (path "/87a59a99-d509-467e-85da-26d34072acb7/25b2e65c-f7ef-4140-a1d7-cd2e01342860"
-          (reference "U14") (unit 1)
-        )
-        (path "/87a59a99-d509-467e-85da-26d34072acb7/5b0f4d64-818d-4913-bde3-c6a16b68a991"
-          (reference "U13") (unit 1)
+          (reference "U15") (unit 2)
         )
       )
+    )
+  )
+  (symbol (lib_id "Amplifier_Operational:MCP6002-xSN") (at 138.43 74.93 0) (unit 1)
+    (in_bom yes) (on_board yes) (dnp no) (fields_autoplaced)
+    (property "Reference" "U15" (at 138.43 66.8401 0)
+      (effects (font (size 1.27 1.27)))
+    )
+    (property "Value" "MCP6002-xSN" (at 138.43 68.7611 0)
+      (effects (font (size 1.27 1.27)))
+    )
+    (property "Footprint" "" (at 138.43 74.93 0)
+      (effects (font (size 1.27 1.27)) hide)
+    )
+    (property "Datasheet" "http://ww1.microchip.com/downloads/en/DeviceDoc/21733j.pdf" (at 138.43 74.93 0)
+      (effects (font (size 1.27 1.27)) hide)
+    )
+    (pin "1")
+    (pin "2")
+    (pin "3")
+    (pin "5")
+    (pin "6")
+    (pin "7")
+    (pin "4")
+    (pin "8")
+    (instances
+      (project "dk2_00"
+        (path "/87a59a99-d509-467e-85da-26d34072acb7/25b2e65c-f7ef-4140-a1d7-cd2e01342860"
+          (reference "U15") (unit 1)
+        )
+      )
+    )
+  )
+  (symbol (lib_id "Amplifier_Operational:MCP6002-xSN") (at 140.335 113.03 0) (unit 3)
+    (in_bom yes) (on_board yes) (dnp no) (fields_autoplaced)
+    (property "Reference" "U15" (at 138.43 112.3863 0)
+      (effects (font (size 1.27 1.27)) (justify left))
+    )
+    (property "Value" "MCP6002-xSN" (at 138.43 114.3073 0)
+      (effects (font (size 1.27 1.27)) (justify left))
+    )
+    (property "Footprint" "" (at 140.335 113.03 0)
+      (effects (font (size 1.27 1.27)) hide)
+    )
+    (property "Datasheet" "http://ww1.microchip.com/downloads/en/DeviceDoc/21733j.pdf" (at 140.335 113.03 0)
+      (effects (font (size 1.27 1.27)) hide)
+    )
+    (pin "1")
+    (pin "2")
+    (pin "3")
+    (pin "5")
+    (pin "6")
+    (pin "7")
+    (pin "4")
+    (pin "8")
+    (instances
+      (project "dk2_00"
+        (path "/87a59a99-d509-467e-85da-26d34072acb7/25b2e65c-f7ef-4140-a1d7-cd2e01342860"
+          (reference "U15") (unit 3)
+        )
+      )
