File: pcb/dk2_00/cv_out.kicad_sch (KiCad schematic)
At the start: 2 parts, among them U13 MCP4922, U15 MCP6002-xSN

Commit message: nothing much
Parts:
- removed U15: MCP6002-xSN, symbol Amplifier_Operational:MCP6002-xSN
- added U14: MCP6002-xSN, symbol Amplifier_Operational:MCP6002-xSN
Changed lines of the file:
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@@
 (kicad_sch (version 20230121) (generator eeschema)
   (paper "A4")
-  (symbol (lib_id "Amplifier_Operational:MCP6002-xSN") (at 131.445 74.93 0) (unit 1)
+  (symbol (lib_id "Amplifier_Operational:MCP6002-xSN") (at 147.955 83.82 0) (unit 2)
     (in_bom yes) (on_board yes) (dnp no) (fields_autoplaced)
-    (property "Reference" "U15" (at 131.445 66.8401 0)
+    (property "Reference" "U14" (at 147.955 75.7301 0)
       (effects (font (size 1.27 1.27)))
     )
-    (property "Value" "MCP6002-xSN" (at 131.445 68.7611 0)
+    (property "Value" "MCP6002-xSN" (at 147.955 77.6511 0)
       (effects (font (size 1.27 1.27)))
     )
-    (property "Footprint" "" (at 131.445 74.93 0)
+    (property "Footprint" "" (at 147.955 83.82 0)
       (effects (font (size 1.27 1.27)) hide)
     )
-    (property "Datasheet" "http://ww1.microchip.com/downloads/en/DeviceDoc/21733j.pdf" (at 131.445 74.93 0)
+    (property "Datasheet" "http://ww1.microchip.com/downloads/en/DeviceDoc/21733j.pdf" (at 147.955 83.82 0)
       (effects (font (size 1.27 1.27)) hide)
     )
@@
       (project "dk2_00"
         (path "/87a59a99-d509-467e-85da-26d34072acb7/5b0f4d64-818d-4913-bde3-c6a16b68a991"
-          (reference "U15") (unit 1)
+          (reference "U14") (unit 2)
         )
       )
+    )
+  )
+  (symbol (lib_id "Amplifier_Operational:MCP6002-xSN") (at 147.955 65.405 0) (unit 1)
+    (in_bom yes) (on_board yes) (dnp no) (fields_autoplaced)
+    (property "Reference" "U14" (at 147.955 57.3151 0)
+      (effects (font (size 1.27 1.27)))
+    )
+    (property "Value" "MCP6002-xSN" (at 147.955 59.2361 0)
+      (effects (font (size 1.27 1.27)))
+    )
+    (property "Footprint" "" (at 147.955 65.405 0)
+      (effects (font (size 1.27 1.27)) hide)
+    )
+    (property "Datasheet" "http://ww1.microchip.com/downloads/en/DeviceDoc/21733j.pdf" (at 147.955 65.405 0)
+      (effects (font (size 1.27 1.27)) hide)
+    )
+    (pin "1")
+    (pin "2")
+    (pin "3")
+    (pin "5")
+    (pin "6")
+    (pin "7")
+    (pin "4")
+    (pin "8")
+    (instances
+      (project "dk2_00"
+        (path "/87a59a99-d509-467e-85da-26d34072acb7/5b0f4d64-818d-4913-bde3-c6a16b68a991"
+          (reference "U14") (unit 1)
+        )
+      )
+    )
+  )
+  (symbol (lib_id "Amplifier_Operational:MCP6002-xSN") (at 150.495 106.68 0) (unit 3)
+    (in_bom yes) (on_board yes) (dnp no) (fields_autoplaced)
+    (property "Reference" "U14" (at 148.59 106.0363 0)
+      (effects (font (size 1.27 1.27)) (justify left))
+    )
+    (property "Value" "MCP6002-xSN" (at 148.59 107.9573 0)
+      (effects (font (size 1.27 1.27)) (justify left))
+    )
+    (property "Footprint" "" (at 150.495 106.68 0)
+      (effects (font (size 1.27 1.27)) hide)
+    )
+    (property "Datasheet" "http://ww1.microchip.com/downloads/en/DeviceDoc/21733j.pdf" (at 150.495 106.68 0)
+      (effects (font (size 1.27 1.27)) hide)
+    )
+    (pin "1")
+    (pin "2")
+    (pin "3")
+    (pin "5")
+    (pin "6")
+    (pin "7")
+    (pin "4")
+    (pin "8")
+    (instances
+      (project "dk2_00"
+        (path "/87a59a99-d509-467e-85da-26d34072acb7/5b0f4d64-818d-4913-bde3-c6a16b68a991"
+          (reference "U14") (unit 3)
+        )
+      )
