File: pcb/dk2_00/shiftregout.kicad_sch (KiCad schematic)
At the start: 17 parts

Commit message: i'm back!
Parts:
- R? (x8): value R -> 200R
Connections:
- net GND: now also U?.13 (~{OE})
- net +3V3: now reaches U?.10 (~{SRCLR})
- net +3V3: now also U?.16 (VCC)
- net 595_CLOCK: now reaches U?.11 (SRCLK)
- net 595_LATCH: now reaches U?.12 (RCLK)
- net 595_DATA: now reaches U?.14 (SER)
- no-connect marks 0 -> 1
Changed lines of the file:
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@@
   (junction (at 162.56 132.08) (diameter 0) (color 0 0 0 0)
   )
+  (junction (at 114.3 80.01) (diameter 0) (color 0 0 0 0)
+  )
   (junction (at 162.56 74.93) (diameter 0) (color 0 0 0 0)
   )
@@
   (junction (at 162.56 120.65) (diameter 0) (color 0 0 0 0)
   )
+  (junction (at 114.3 46.99) (diameter 0) (color 0 0 0 0)
+  )
   (junction (at 162.56 97.79) (diameter 0) (color 0 0 0 0)
   )
+  (no_connect (at 124.46 74.93))
   (wire (pts (xy 162.56 74.93) (xy 162.56 86.36))
     (stroke (width 0) (type default))
@@
     (stroke (width 0) (type default))
   )
+  (wire (pts (xy 88.9 59.69) (xy 104.14 59.69))
+    (stroke (width 0) (type default))
+  )
   (wire (pts (xy 162.56 63.5) (xy 162.56 74.93))
     (stroke (width 0) (type default))
@@
     (stroke (width 0) (type default))
   )
+  (wire (pts (xy 104.14 67.31) (xy 104.14 80.01))
+    (stroke (width 0) (type default))
+  )
   (wire (pts (xy 144.78 59.69) (xy 124.46 59.69))
     (stroke (width 0) (type default))
@@
     (stroke (width 0) (type default))
   )
+  (wire (pts (xy 88.9 46.99) (xy 88.9 59.69))
+    (stroke (width 0) (type default))
+  )
   (wire (pts (xy 124.46 62.23) (xy 143.51 62.23))
     (stroke (width 0) (type default))
@@
     (stroke (width 0) (type default))
   )
+  (wire (pts (xy 104.14 80.01) (xy 114.3 80.01))
+    (stroke (width 0) (type default))
+  )
+  (wire (pts (xy 114.3 46.99) (xy 88.9 46.99))
+    (stroke (width 0) (type default))
+  )
+  (global_label "595_DATA" (shape input) (at 104.14 52.07 180) (fields_autoplaced)
+    (effects (font (size 1.27 1.27)) (justify right))
+    (property "Intersheetrefs" "${INTERSHEET_REFS}" (at 92.2233 52.07 0)
+      (effects (font (size 1.27 1.27)) (justify right) hide)
+    )
+  )
+  (global_label "595_CLOCK" (shape input) (at 104.14 57.15 180) (fields_autoplaced)
+    (effects (font (size 1.27 1.27)) (justify right))
+    (property "Intersheetrefs" "${INTERSHEET_REFS}" (at 90.4695 57.15 0)
+      (effects (font (size 1.27 1.27)) (justify right) hide)
+    )
+  )
+  (global_label "595_LATCH" (shape input) (at 104.14 64.77 180) (fields_autoplaced)
+    (effects (font (size 1.27 1.27)) (justify right))
+    (property "Intersheetrefs" "${INTERSHEET_REFS}" (at 90.9533 64.77 0)
+      (effects (font (size 1.27 1.27)) (justify right) hide)
+    )
+  )
   (symbol (lib_id "Device:R") (at 151.13 120.65 270) (unit 1)
     (in_bom yes) (on_board yes) (dnp no) (fields_autoplaced)
-    (property "Reference" "R?" (at 151.13 114.3 90)
-      (effects (font (size 1.27 1.27)))
-    )
-    (property "Value" "R" (at 151.13 116.84 90)
+    (property "Reference" "R?" (at 151.13 116.6241 90)
+      (effects (font (size 1.27 1.27)))
+    )
+    (property "Value" "200R" (at 151.13 118.5451 90)
       (effects (font (size 1.27 1.27)))
     )
@@
   (symbol (lib_id "Device:R") (at 151.13 63.5 270) (unit 1)
     (in_bom yes) (on_board yes) (dnp no) (fields_autoplaced)
-    (property "Reference" "R?" (at 151.13 57.15 90)
-      (effects (font (size 1.27 1.27)))
-    )
-    (property "Value" "R" (at 151.13 59.69 90)
+    (property "Reference" "R?" (at 151.13 59.4741 90)
+      (effects (font (size 1.27 1.27)))
+    )
+    (property "Value" "200R" (at 151.13 61.3951 90)
       (effects (font (size 1.27 1.27)))
     )
@@
   (symbol (lib_id "Device:R") (at 151.13 132.08 270) (unit 1)
     (in_bom yes) (on_board yes) (dnp no) (fields_autoplaced)
-    (property "Reference" "R?" (at 151.13 125.73 90)
-      (effects (font (size 1.27 1.27)))
-    )
-    (property "Value" "R" (at 151.13 128.27 90)
+    (property "Reference" "R?" (at 151.13 128.0541 90)
+      (effects (font (size 1.27 1.27)))
+    )
+    (property "Value" "200R" (at 151.13 129.9751 90)
       (effects (font (size 1.27 1.27)))
     )
@@
   (symbol (lib_id "Device:R") (at 151.13 86.36 270) (unit 1)
     (in_bom yes) (on_board yes) (dnp no) (fields_autoplaced)
-    (property "Reference" "R?" (at 151.13 80.01 90)
-      (effects (font (size 1.27 1.27)))
-    )
-    (property "Value" "R" (at 151.13 82.55 90)
+    (property "Reference" "R?" (at 151.13 82.3341 90)
+      (effects (font (size 1.27 1.27)))
+    )
+    (property "Value" "200R" (at 151.13 84.2551 90)
       (effects (font (size 1.27 1.27)))
     )
@@
   (symbol (lib_id "Device:R") (at 151.13 74.93 270) (unit 1)
     (in_bom yes) (on_board yes) (dnp no) (fields_autoplaced)
-    (property "Reference" "R?" (at 151.13 68.58 90)
-      (effects (font (size 1.27 1.27)))
-    )
-    (property "Value" "R" (at 151.13 71.12 90)
+    (property "Reference" "R?" (at 151.13 70.9041 90)
+      (effects (font (size 1.27 1.27)))
+    )
+    (property "Value" "200R" (at 151.13 72.8251 90)
       (effects (font (size 1.27 1.27)))
     )
@@
   (symbol (lib_id "Device:R") (at 151.13 109.22 270) (unit 1)
     (in_bom yes) (on_board yes) (dnp no) (fields_autoplaced)
-    (property "Reference" "R?" (at 151.13 102.87 90)
-      (effects (font (size 1.27 1.27)))
-    )
-    (property "Value" "R" (at 151.13 105.41 90)
+    (property "Reference" "R?" (at 151.13 105.1941 90)
+      (effects (font (size 1.27 1.27)))
+    )
+    (property "Value" "200R" (at 151.13 107.1151 90)
       (effects (font (size 1.27 1.27)))
     )
@@
     )
   )
+  (symbol (lib_id "power:+3V3") (at 114.3 46.99 0) (unit 1)
+    (in_bom yes) (on_board yes) (dnp no) (fields_autoplaced)
+    (property "Reference" "#PWR?" (at 114.3 50.8 0)
+      (effects (font (size 1.27 1.27)) hide)
+    )
+    (property "Value" "+3V3" (at 114.3 41.91 0)
+      (effects (font (size 1.27 1.27)))
+    )
+    (property "Footprint" "" (at 114.3 46.99 0)
+      (effects (font (size 1.27 1.27)) hide)
+    )
+    (property "Datasheet" "" (at 114.3 46.99 0)
+      (effects (font (size 1.27 1.27)) hide)
+    )
+    (pin "1")
+    (instances
+      (project "dk2_00"
+        (path "/87a59a99-d509-467e-85da-26d34072acb7"
+          (reference "#PWR?") (unit 1)
+        )
+        (path "/87a59a99-d509-467e-85da-26d34072acb7/ef9ac6f0-c4a3-4cf8-9f87-0e925c926098"
+          (reference "#PWR02") (unit 1)
+        )
+      )
+    )
+  )
   (symbol (lib_id "Device:R") (at 151.13 97.79 270) (unit 1)
     (in_bom yes) (on_board yes) (dnp no) (fields_autoplaced)
-    (property "Reference" "R?" (at 151.13 91.44 90)
-      (effects (font (size 1.27 1.27)))
-    )
-    (property "Value" "R" (at 151.13 93.98 90)
+    (property "Reference" "R?" (at 151.13 93.7641 90)
+      (effects (font (size 1.27 1.27)))
+    )
+    (property "Value" "200R" (at 151.13 95.6851 90)
       (effects (font (size 1.27 1.27)))
     )
@@
   (symbol (lib_id "Device:R") (at 151.13 52.07 270) (unit 1)
     (in_bom yes) (on_board yes) (dnp no) (fields_autoplaced)
-    (property "Reference" "R?" (at 151.13 45.72 90)
-      (effects (font (size 1.27 1.27)))
-    )
-    (property "Value" "R" (at 151.13 48.26 90)
-      (effects (font (size 1.27 1.27)))
-    )
+    (property "Reference" "R?" (at 151.13 48.0441 90)
+      (effects (font (size 1.27 1.27)))
+    )
+    (property "Value" "200R" (at 151.13 49.9651 90)
+      (effects (font (size 1.27 1.27)))
+    )

Commit message: oh that's what a multi unit symbol is
Parts:
- gave numbers to parts that had none: 17
Changed lines of the file:
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@@
   (symbol (lib_id "Device:R") (at 151.13 120.65 270) (unit 1)
     (in_bom yes) (on_board yes) (dnp no) (fields_autoplaced)
-    (property "Reference" "R?" (at 151.13 116.6241 90)
+    (property "Reference" "R7" (at 151.13 116.6241 90)
       (effects (font (size 1.27 1.27)))
     )
@@
       (project "dk2_00"
         (path "/87a59a99-d509-467e-85da-26d34072acb7/ef9ac6f0-c4a3-4cf8-9f87-0e925c926098"
-          (reference "R?") (unit 1)
+          (reference "R7") (unit 1)
         )
       )
@@
   (symbol (lib_id "74xx:74HC595") (at 114.3 62.23 0) (unit 1)
     (in_bom yes) (on_board yes) (dnp no) (fields_autoplaced)
-    (property "Reference" "U?" (at 116.3194 45.8302 0)
+    (property "Reference" "U2" (at 116.3194 45.8302 0)
       (effects (font (size 1.27 1.27)) (justify left))
     )
@@
       (project "dk2_00"
         (path "/87a59a99-d509-467e-85da-26d34072acb7/ef9ac6f0-c4a3-4cf8-9f87-0e925c926098"
-          (reference "U?") (unit 1)
+          (reference "U2") (unit 1)
         )
       )
@@
   (symbol (lib_id "Device:LED") (at 158.75 74.93 180) (unit 1)
     (in_bom yes) (on_board yes) (dnp no)
-    (property "Reference" "D?" (at 160.02 68.58 0)
+    (property "Reference" "D3" (at 160.02 68.58 0)
       (effects (font (size 1.27 1.27)))
     )
@@
       (project "dk2_00"
         (path "/87a59a99-d509-467e-85da-26d34072acb7/ef9ac6f0-c4a3-4cf8-9f87-0e925c926098"
-          (reference "D?") (unit 1)
+          (reference "D3") (unit 1)
         )
       )
@@
   (symbol (lib_id "Device:LED") (at 158.75 63.5 180) (unit 1)
     (in_bom yes) (on_board yes) (dnp no)
-    (property "Reference" "D?" (at 160.02 57.15 0)
+    (property "Reference" "D2" (at 160.02 57.15 0)
       (effects (font (size 1.27 1.27)))
     )
@@
       (project "dk2_00"
         (path "/87a59a99-d509-467e-85da-26d34072acb7/ef9ac6f0-c4a3-4cf8-9f87-0e925c926098"
-          (reference "D?") (unit 1)
+          (reference "D2") (unit 1)
         )
       )
@@
   (symbol (lib_id "Device:R") (at 151.13 63.5 270) (unit 1)
     (in_bom yes) (on_board yes) (dnp no) (fields_autoplaced)
-    (property "Reference" "R?" (at 151.13 59.4741 90)
+    (property "Reference" "R2" (at 151.13 59.4741 90)
       (effects (font (size 1.27 1.27)))
     )
@@
       (project "dk2_00"
         (path "/87a59a99-d509-467e-85da-26d34072acb7/ef9ac6f0-c4a3-4cf8-9f87-0e925c926098"
-          (reference "R?") (unit 1)
+          (reference "R2") (unit 1)
         )
       )
@@
   (symbol (lib_id "power:GND") (at 162.56 135.89 0) (unit 1)
     (in_bom yes) (on_board yes) (dnp no) (fields_autoplaced)
-    (property "Reference" "#PWR?" (at 162.56 142.24 0)
+    (property "Reference" "#PWR08" (at 162.56 142.24 0)
       (effects (font (size 1.27 1.27)) hide)
     )
@@
       (project "dk2_00"
         (path "/87a59a99-d509-467e-85da-26d34072acb7/ef9ac6f0-c4a3-4cf8-9f87-0e925c926098"
-          (reference "#PWR?") (unit 1)
+          (reference "#PWR08") (unit 1)
         )
       )
@@
   (symbol (lib_id "Device:R") (at 151.13 132.08 270) (unit 1)
     (in_bom yes) (on_board yes) (dnp no) (fields_autoplaced)
-    (property "Reference" "R?" (at 151.13 128.0541 90)
+    (property "Reference" "R8" (at 151.13 128.0541 90)
       (effects (font (size 1.27 1.27)))
     )
@@
       (project "dk2_00"
         (path "/87a59a99-d509-467e-85da-26d34072acb7/ef9ac6f0-c4a3-4cf8-9f87-0e925c926098"
-          (reference "R?") (unit 1)
+          (reference "R8") (unit 1)
         )
       )
@@
   (symbol (lib_id "Device:LED") (at 158.75 52.07 180) (unit 1)
     (in_bom yes) (on_board yes) (dnp no)
-    (property "Reference" "D?" (at 160.02 45.72 0)
+    (property "Reference" "D1" (at 160.02 45.72 0)
       (effects (font (size 1.27 1.27)))
     )
@@
       (project "dk2_00"
         (path "/87a59a99-d509-467e-85da-26d34072acb7/ef9ac6f0-c4a3-4cf8-9f87-0e925c926098"
-          (reference "D?") (unit 1)
+          (reference "D1") (unit 1)
         )
       )
@@
   (symbol (lib_id "Device:LED") (at 158.75 132.08 180) (unit 1)
     (in_bom yes) (on_board yes) (dnp no)
-    (property "Reference" "D?" (at 160.02 125.73 0)
+    (property "Reference" "D8" (at 160.02 125.73 0)
       (effects (font (size 1.27 1.27)))
     )
@@
       (project "dk2_00"
         (path "/87a59a99-d509-467e-85da-26d34072acb7/ef9ac6f0-c4a3-4cf8-9f87-0e925c926098"
-          (reference "D?") (unit 1)
+          (reference "D8") (unit 1)
         )
       )
@@
   (symbol (lib_id "Device:LED") (at 158.75 109.22 180) (unit 1)
     (in_bom yes) (on_board yes) (dnp no)
-    (property "Reference" "D?" (at 160.02 102.87 0)
+    (property "Reference" "D6" (at 160.02 102.87 0)
       (effects (font (size 1.27 1.27)))
     )
@@
       (project "dk2_00"
         (path "/87a59a99-d509-467e-85da-26d34072acb7/ef9ac6f0-c4a3-4cf8-9f87-0e925c926098"
-          (reference "D?") (unit 1)
+          (reference "D6") (unit 1)
         )
       )
@@
   (symbol (lib_id "Device:R") (at 151.13 86.36 270) (unit 1)
     (in_bom yes) (on_board yes) (dnp no) (fields_autoplaced)
-    (property "Reference" "R?" (at 151.13 82.3341 90)
+    (property "Reference" "R4" (at 151.13 82.3341 90)
       (effects (font (size 1.27 1.27)))
     )
@@
       (project "dk2_00"
         (path "/87a59a99-d509-467e-85da-26d34072acb7/ef9ac6f0-c4a3-4cf8-9f87-0e925c926098"
-          (reference "R?") (unit 1)
+          (reference "R4") (unit 1)
         )
       )
@@
   (symbol (lib_id "Device:LED") (at 158.75 97.79 180) (unit 1)
     (in_bom yes) (on_board yes) (dnp no)
-    (property "Reference" "D?" (at 160.02 91.44 0)
+    (property "Reference" "D5" (at 160.02 91.44 0)
       (effects (font (size 1.27 1.27)))
     )
@@
       (project "dk2_00"
         (path "/87a59a99-d509-467e-85da-26d34072acb7/ef9ac6f0-c4a3-4cf8-9f87-0e925c926098"
-          (reference "D?") (unit 1)
+          (reference "D5") (unit 1)
         )
       )
@@
   (symbol (lib_id "Device:R") (at 151.13 74.93 270) (unit 1)
     (in_bom yes) (on_board yes) (dnp no) (fields_autoplaced)
-    (property "Reference" "R?" (at 151.13 70.9041 90)
+    (property "Reference" "R3" (at 151.13 70.9041 90)
       (effects (font (size 1.27 1.27)))
     )
@@
       (project "dk2_00"
         (path "/87a59a99-d509-467e-85da-26d34072acb7/ef9ac6f0-c4a3-4cf8-9f87-0e925c926098"
-          (reference "R?") (unit 1)
+          (reference "R3") (unit 1)
         )
       )
@@
   (symbol (lib_id "Device:LED") (at 158.75 120.65 180) (unit 1)
     (in_bom yes) (on_board yes) (dnp no)
-    (property "Reference" "D?" (at 160.02 114.3 0)
+    (property "Reference" "D7" (at 160.02 114.3 0)
       (effects (font (size 1.27 1.27)))
     )
@@
       (project "dk2_00"
         (path "/87a59a99-d509-467e-85da-26d34072acb7/ef9ac6f0-c4a3-4cf8-9f87-0e925c926098"
-          (reference "D?") (unit 1)
+          (reference "D7") (unit 1)
         )
       )
@@
   (symbol (lib_id "Device:R") (at 151.13 109.22 270) (unit 1)
     (in_bom yes) (on_board yes) (dnp no) (fields_autoplaced)
-    (property "Reference" "R?" (at 151.13 105.1941 90)
+    (property "Reference" "R6" (at 151.13 105.1941 90)
       (effects (font (size 1.27 1.27)))
     )
@@
       (project "dk2_00"
         (path "/87a59a99-d509-467e-85da-26d34072acb7/ef9ac6f0-c4a3-4cf8-9f87-0e925c926098"
-          (reference "R?") (unit 1)
+          (reference "R6") (unit 1)
         )
       )
@@
   (symbol (lib_id "power:GND") (at 114.3 80.01 0) (unit 1)
     (in_bom yes) (on_board yes) (dnp no) (fields_autoplaced)
-    (property "Reference" "#PWR?" (at 114.3 86.36 0)
+    (property "Reference" "#PWR07" (at 114.3 86.36 0)
       (effects (font (size 1.27 1.27)) hide)
     )
@@
       (project "dk2_00"
         (path "/87a59a99-d509-467e-85da-26d34072acb7/ef9ac6f0-c4a3-4cf8-9f87-0e925c926098"
-          (reference "#PWR?") (unit 1)
+          (reference "#PWR07") (unit 1)
         )
       )
@@
         )
         (path "/87a59a99-d509-467e-85da-26d34072acb7/ef9ac6f0-c4a3-4cf8-9f87-0e925c926098"
-          (reference "#PWR02") (unit 1)
+          (reference "#PWR06") (unit 1)
         )
       )
@@
   (symbol (lib_id "Device:R") (at 151.13 97.79 270) (unit 1)
     (in_bom yes) (on_board yes) (dnp no) (fields_autoplaced)
-    (property "Reference" "R?" (at 151.13 93.7641 90)
+    (property "Reference" "R5" (at 151.13 93.7641 90)
       (effects (font (size 1.27 1.27)))
     )
@@
       (project "dk2_00"
         (path "/87a59a99-d509-467e-85da-26d34072acb7/ef9ac6f0-c4a3-4cf8-9f87-0e925c926098"
-          (reference "R?") (unit 1)
+          (reference "R5") (unit 1)
         )
       )
@@
   (symbol (lib_id "Device:R") (at 151.13 52.07 270) (unit 1)
     (in_bom yes) (on_board yes) (dnp no) (fields_autoplaced)
-    (property "Reference" "R?" (at 151.13 48.0441 90)
+    (property "Reference" "R1" (at 151.13 48.0441 90)
       (effects (font (size 1.27 1.27)))
     )
@@
       (project "dk2_00"
         (path "/87a59a99-d509-467e-85da-26d34072acb7/ef9ac6f0-c4a3-4cf8-9f87-0e925c926098"
-          (reference "R?") (unit 1)
+          (reference "R1") (unit 1)
         )
       )
@@
   (symbol (lib_id "Device:LED") (at 158.75 86.36 180) (unit 1)
     (in_bom yes) (on_board yes) (dnp no)
-    (property "Reference" "D?" (at 160.02 80.01 0)
+    (property "Reference" "D4" (at 160.02 80.01 0)
       (effects (font (size 1.27 1.27)))
     )
@@
       (project "dk2_00"
         (path "/87a59a99-d509-467e-85da-26d34072acb7/ef9ac6f0-c4a3-4cf8-9f87-0e925c926098"
-          (reference "D?") (unit 1)
-        )
-      )
+          (reference "D4") (unit 1)
+        )
+      )

Commit message: footprints assigned
Parts:
- D1, D2, D3, D4, D5, D6, D7, D8: footprint (none) -> LED_SMD:LED_0805_2012Metric
- R1, R2, R3, R4, R5, R6, R7, R8: footprint (none) -> Resistor_SMD:R_0603_1608Metric
- U2: footprint (none) -> Package_SO:SOIC-16_3.9x9.9mm_P1.27mm
Changed lines of the file:
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@@
       (effects (font (size 1.27 1.27)))
     )
-    (property "Footprint" "" (at 151.13 118.872 90)
+    (property "Footprint" "Resistor_SMD:R_0603_1608Metric" (at 151.13 118.872 90)
       (effects (font (size 1.27 1.27)) hide)
     )
@@
       (effects (font (size 1.27 1.27)) (justify left))
     )
-    (property "Footprint" "" (at 114.3 62.23 0)
+    (property "Footprint" "Package_SO:SOIC-16_3.9x9.9mm_P1.27mm" (at 114.3 62.23 0)
       (effects (font (size 1.27 1.27)) hide)
     )
@@
       (effects (font (size 1.27 1.27)))
     )
-    (property "Footprint" "" (at 158.75 74.93 0)
+    (property "Footprint" "LED_SMD:LED_0805_2012Metric" (at 158.75 74.93 0)
       (effects (font (size 1.27 1.27)) hide)
     )
@@
       (effects (font (size 1.27 1.27)))
     )
-    (property "Footprint" "" (at 158.75 63.5 0)
+    (property "Footprint" "LED_SMD:LED_0805_2012Metric" (at 158.75 63.5 0)
       (effects (font (size 1.27 1.27)) hide)
     )
@@
       (effects (font (size 1.27 1.27)))
     )
-    (property "Footprint" "" (at 151.13 61.722 90)
+    (property "Footprint" "Resistor_SMD:R_0603_1608Metric" (at 151.13 61.722 90)
       (effects (font (size 1.27 1.27)) hide)
     )
@@
       (effects (font (size 1.27 1.27)))
     )
-    (property "Footprint" "" (at 151.13 130.302 90)
+    (property "Footprint" "Resistor_SMD:R_0603_1608Metric" (at 151.13 130.302 90)
       (effects (font (size 1.27 1.27)) hide)
     )
@@
       (effects (font (size 1.27 1.27)))
     )
-    (property "Footprint" "" (at 158.75 52.07 0)
+    (property "Footprint" "LED_SMD:LED_0805_2012Metric" (at 158.75 52.07 0)
       (effects (font (size 1.27 1.27)) hide)
     )
@@
       (effects (font (size 1.27 1.27)))
     )
-    (property "Footprint" "" (at 158.75 132.08 0)
+    (property "Footprint" "LED_SMD:LED_0805_2012Metric" (at 158.75 132.08 0)
       (effects (font (size 1.27 1.27)) hide)
     )
@@
       (effects (font (size 1.27 1.27)))
     )
-    (property "Footprint" "" (at 158.75 109.22 0)
+    (property "Footprint" "LED_SMD:LED_0805_2012Metric" (at 158.75 109.22 0)
       (effects (font (size 1.27 1.27)) hide)
     )
@@
       (effects (font (size 1.27 1.27)))
     )
-    (property "Footprint" "" (at 151.13 84.582 90)
+    (property "Footprint" "Resistor_SMD:R_0603_1608Metric" (at 151.13 84.582 90)
       (effects (font (size 1.27 1.27)) hide)
     )
@@
       (effects (font (size 1.27 1.27)))
     )
-    (property "Footprint" "" (at 158.75 97.79 0)
+    (property "Footprint" "LED_SMD:LED_0805_2012Metric" (at 158.75 97.79 0)
       (effects (font (size 1.27 1.27)) hide)
     )
@@
       (effects (font (size 1.27 1.27)))
     )
-    (property "Footprint" "" (at 151.13 73.152 90)
+    (property "Footprint" "Resistor_SMD:R_0603_1608Metric" (at 151.13 73.152 90)
       (effects (font (size 1.27 1.27)) hide)
     )
@@
       (effects (font (size 1.27 1.27)))
     )
-    (property "Footprint" "" (at 158.75 120.65 0)
+    (property "Footprint" "LED_SMD:LED_0805_2012Metric" (at 158.75 120.65 0)
       (effects (font (size 1.27 1.27)) hide)
     )
@@
       (effects (font (size 1.27 1.27)))
     )
-    (property "Footprint" "" (at 151.13 107.442 90)
+    (property "Footprint" "Resistor_SMD:R_0603_1608Metric" (at 151.13 107.442 90)
       (effects (font (size 1.27 1.27)) hide)
     )
@@
       (effects (font (size 1.27 1.27)))
     )
-    (property "Footprint" "" (at 151.13 96.012 90)
+    (property "Footprint" "Resistor_SMD:R_0603_1608Metric" (at 151.13 96.012 90)
       (effects (font (size 1.27 1.27)) hide)
     )
@@
       (effects (font (size 1.27 1.27)))
     )
-    (property "Footprint" "" (at 151.13 50.292 90)
+    (property "Footprint" "Resistor_SMD:R_0603_1608Metric" (at 151.13 50.292 90)
       (effects (font (size 1.27 1.27)) hide)
     )
@@
       (effects (font (size 1.27 1.27)))
     )
-    (property "Footprint" "" (at 158.75 86.36 0)
-      (effects (font (size 1.27 1.27)) hide)
-    )
+    (property "Footprint" "LED_SMD:LED_0805_2012Metric" (at 158.75 86.36 0)
+      (effects (font (size 1.27 1.27)) hide)
+    )
