File: pcb/dk2_00/shiftregout.kicad_sch (KiCad schematic)
At the start: 17 parts, among them U2 74HC595

Commit message: being decisive
Parts:
- R1, R2, R3, R4, R5, R6, R7, R8: symbol Device:R -> Device:R_US
Changed lines of the file:
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@@
     )
   )
-  (symbol (lib_id "Device:R") (at 151.13 120.65 270) (unit 1)
+  (symbol (lib_id "Device:R_US") (at 151.13 120.65 270) (unit 1)
     (in_bom yes) (on_board yes) (dnp no) (fields_autoplaced)
     (property "Reference" "R7" (at 151.13 116.6241 90)
@@
       (effects (font (size 1.27 1.27)))
     )
-    (property "Footprint" "Resistor_SMD:R_0603_1608Metric" (at 151.13 118.872 90)
+    (property "Footprint" "Resistor_SMD:R_0603_1608Metric" (at 150.876 121.666 90)
       (effects (font (size 1.27 1.27)) hide)
     )
@@
     )
   )
-  (symbol (lib_id "Device:R") (at 151.13 63.5 270) (unit 1)
+  (symbol (lib_id "Device:R_US") (at 151.13 63.5 270) (unit 1)
     (in_bom yes) (on_board yes) (dnp no) (fields_autoplaced)
     (property "Reference" "R2" (at 151.13 59.4741 90)
@@
       (effects (font (size 1.27 1.27)))
     )
-    (property "Footprint" "Resistor_SMD:R_0603_1608Metric" (at 151.13 61.722 90)
+    (property "Footprint" "Resistor_SMD:R_0603_1608Metric" (at 150.876 64.516 90)
       (effects (font (size 1.27 1.27)) hide)
     )
@@
     )
   )
-  (symbol (lib_id "Device:R") (at 151.13 132.08 270) (unit 1)
+  (symbol (lib_id "Device:R_US") (at 151.13 132.08 270) (unit 1)
     (in_bom yes) (on_board yes) (dnp no) (fields_autoplaced)
     (property "Reference" "R8" (at 151.13 128.0541 90)
@@
       (effects (font (size 1.27 1.27)))
     )
-    (property "Footprint" "Resistor_SMD:R_0603_1608Metric" (at 151.13 130.302 90)
+    (property "Footprint" "Resistor_SMD:R_0603_1608Metric" (at 150.876 133.096 90)
       (effects (font (size 1.27 1.27)) hide)
     )
@@
     )
   )
-  (symbol (lib_id "Device:R") (at 151.13 86.36 270) (unit 1)
+  (symbol (lib_id "Device:R_US") (at 151.13 86.36 270) (unit 1)
     (in_bom yes) (on_board yes) (dnp no) (fields_autoplaced)
     (property "Reference" "R4" (at 151.13 82.3341 90)
@@
       (effects (font (size 1.27 1.27)))
     )
-    (property "Footprint" "Resistor_SMD:R_0603_1608Metric" (at 151.13 84.582 90)
+    (property "Footprint" "Resistor_SMD:R_0603_1608Metric" (at 150.876 87.376 90)
       (effects (font (size 1.27 1.27)) hide)
     )
@@
     )
   )
-  (symbol (lib_id "Device:R") (at 151.13 74.93 270) (unit 1)
+  (symbol (lib_id "Device:R_US") (at 151.13 74.93 270) (unit 1)
     (in_bom yes) (on_board yes) (dnp no) (fields_autoplaced)
     (property "Reference" "R3" (at 151.13 70.9041 90)
@@
       (effects (font (size 1.27 1.27)))
     )
-    (property "Footprint" "Resistor_SMD:R_0603_1608Metric" (at 151.13 73.152 90)
+    (property "Footprint" "Resistor_SMD:R_0603_1608Metric" (at 150.876 75.946 90)
       (effects (font (size 1.27 1.27)) hide)
     )
@@
     )
   )
-  (symbol (lib_id "Device:R") (at 151.13 109.22 270) (unit 1)
+  (symbol (lib_id "Device:R_US") (at 151.13 109.22 270) (unit 1)
     (in_bom yes) (on_board yes) (dnp no) (fields_autoplaced)
     (property "Reference" "R6" (at 151.13 105.1941 90)
@@
       (effects (font (size 1.27 1.27)))
     )
-    (property "Footprint" "Resistor_SMD:R_0603_1608Metric" (at 151.13 107.442 90)
+    (property "Footprint" "Resistor_SMD:R_0603_1608Metric" (at 150.876 110.236 90)
       (effects (font (size 1.27 1.27)) hide)
     )
@@
     )
   )
-  (symbol (lib_id "Device:R") (at 151.13 97.79 270) (unit 1)
+  (symbol (lib_id "Device:R_US") (at 151.13 97.79 270) (unit 1)
     (in_bom yes) (on_board yes) (dnp no) (fields_autoplaced)
     (property "Reference" "R5" (at 151.13 93.7641 90)
@@
       (effects (font (size 1.27 1.27)))
     )
-    (property "Footprint" "Resistor_SMD:R_0603_1608Metric" (at 151.13 96.012 90)
+    (property "Footprint" "Resistor_SMD:R_0603_1608Metric" (at 150.876 98.806 90)
       (effects (font (size 1.27 1.27)) hide)
     )
@@
     )
   )
-  (symbol (lib_id "Device:R") (at 151.13 52.07 270) (unit 1)
+  (symbol (lib_id "Device:R_US") (at 151.13 52.07 270) (unit 1)
     (in_bom yes) (on_board yes) (dnp no) (fields_autoplaced)
     (property "Reference" "R1" (at 151.13 48.0441 90)
@@
       (effects (font (size 1.27 1.27)))
     )
-    (property "Footprint" "Resistor_SMD:R_0603_1608Metric" (at 151.13 50.292 90)
-      (effects (font (size 1.27 1.27)) hide)
-    )
+    (property "Footprint" "Resistor_SMD:R_0603_1608Metric" (at 150.876 53.086 90)
+      (effects (font (size 1.27 1.27)) hide)
+    )

Commit message: tidying up, getting close!
Connections:
- net +3V3 renamed +3.3V
Changed lines of the file:
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@@
     )
   )
-  (symbol (lib_id "power:+3V3") (at 114.3 46.99 0) (unit 1)
+  (symbol (lib_id "power:+3.3V") (at 114.3 46.99 0) (unit 1)
     (in_bom yes) (on_board yes) (dnp no) (fields_autoplaced)
     (property "Reference" "#PWR?" (at 114.3 50.8 0)
       (effects (font (size 1.27 1.27)) hide)
     )
-    (property "Value" "+3V3" (at 114.3 41.91 0)
+    (property "Value" "+3.3V" (at 114.3 43.434 0)
       (effects (font (size 1.27 1.27)))
     )
