File: pcb/dk2_00/muxin1.kicad_sch (KiCad schematic)
At the start: 9 parts, among them U7 74HC4051

Commit message: tidying up, getting close!
Connections:
- net +3V3 renamed +3.3V
Changed lines of the file:
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@@
         )
         (path "/87a59a99-d509-467e-85da-26d34072acb7/b61d4abb-9ce0-48d3-9c53-5c624ca490e4"
-          (reference "#PWR031") (unit 1)
+          (reference "#PWR036") (unit 1)
         )
       )
@@
         )
         (path "/87a59a99-d509-467e-85da-26d34072acb7/b61d4abb-9ce0-48d3-9c53-5c624ca490e4"
-          (reference "#PWR029") (unit 1)
+          (reference "#PWR034") (unit 1)
         )
       )
@@
     )
   )
-  (symbol (lib_id "power:+3V3") (at 142.24 46.99 0) (unit 1)
+  (symbol (lib_id "power:+3.3V") (at 142.24 46.99 0) (unit 1)
     (in_bom yes) (on_board yes) (dnp no) (fields_autoplaced)
     (property "Reference" "#PWR032" (at 142.24 50.8 0)
       (effects (font (size 1.27 1.27)) hide)
     )
-    (property "Value" "+3V3" (at 142.24 41.91 0)
+    (property "Value" "+3.3V" (at 142.24 43.434 0)
       (effects (font (size 1.27 1.27)))
     )
@@
         )
         (path "/87a59a99-d509-467e-85da-26d34072acb7/b61d4abb-9ce0-48d3-9c53-5c624ca490e4"
-          (reference "#PWR028") (unit 1)
+          (reference "#PWR033") (unit 1)
         )
       )
@@
         )
         (path "/87a59a99-d509-467e-85da-26d34072acb7/b61d4abb-9ce0-48d3-9c53-5c624ca490e4"
-          (reference "U6") (unit 1)
-        )
-      )
-    )
-  )
-  (symbol (lib_id "power:+3V3") (at 184.15 45.72 0) (unit 1)
+          (reference "U7") (unit 1)
+        )
+      )
+    )
+  )
+  (symbol (lib_id "power:+3.3V") (at 184.15 45.72 0) (unit 1)
     (in_bom yes) (on_board yes) (dnp no) (fields_autoplaced)
     (property "Reference" "#PWR034" (at 184.15 49.53 0)
       (effects (font (size 1.27 1.27)) hide)
     )
-    (property "Value" "+3V3" (at 184.15 40.64 0)
+    (property "Value" "+3.3V" (at 184.15 42.164 0)
       (effects (font (size 1.27 1.27)))
     )
@@
         )
         (path "/87a59a99-d509-467e-85da-26d34072acb7/b61d4abb-9ce0-48d3-9c53-5c624ca490e4"
-          (reference "#PWR030") (unit 1)
-        )
-      )
+          (reference "#PWR035") (unit 1)
+        )
+      )

Commit message: rough layout
Parts:
- RV13, RV14, RV15, RV16: footprint Connector_PinSocket_2.54mm:PinSocket_1x03_P2.54mm_Vertical -> Library:Potentiometer_Alps_RK09K_vertical_biggerholes
Changed lines of the file:
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@@
       (effects (font (size 1.27 1.27)) (justify right))
     )
-    (property "Footprint" "Connector_PinSocket_2.54mm:PinSocket_1x03_P2.54mm_Vertical" (at 176.53 102.87 0)
+    (property "Footprint" "Library:Potentiometer_Alps_RK09K_vertical_biggerholes" (at 176.53 102.87 0)
       (effects (font (size 1.27 1.27)) hide)
     )
@@
       (effects (font (size 1.27 1.27)) (justify right))
     )
-    (property "Footprint" "Connector_PinSocket_2.54mm:PinSocket_1x03_P2.54mm_Vertical" (at 176.53 123.19 0)
+    (property "Footprint" "Library:Potentiometer_Alps_RK09K_vertical_biggerholes" (at 176.53 123.19 0)
       (effects (font (size 1.27 1.27)) hide)
     )
@@
       (effects (font (size 1.27 1.27)) (justify right))
     )
-    (property "Footprint" "Connector_PinSocket_2.54mm:PinSocket_1x03_P2.54mm_Vertical" (at 176.53 113.03 0)
+    (property "Footprint" "Library:Potentiometer_Alps_RK09K_vertical_biggerholes" (at 176.53 113.03 0)
       (effects (font (size 1.27 1.27)) hide)
     )
@@
       (effects (font (size 1.27 1.27)) (justify right))
     )
-    (property "Footprint" "Connector_PinSocket_2.54mm:PinSocket_1x03_P2.54mm_Vertical" (at 176.53 92.71 0)
-      (effects (font (size 1.27 1.27)) hide)
-    )
+    (property "Footprint" "Library:Potentiometer_Alps_RK09K_vertical_biggerholes" (at 176.53 92.71 0)
+      (effects (font (size 1.27 1.27)) hide)
+    )
