File: pcb/dk2_01/muxin1.kicad_sch (KiCad schematic)
At the start: 9 parts, among them U7 74HC4051

Commit message: good pcb progress
Connections:
- net GND: now also U7.6 (~{E})
- no-connect marks 1 -> 0
Changed lines of the file:
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@@
   (junction (at 186.69 119.38) (diameter 0) (color 0 0 0 0)
   )
-  (no_connect (at 134.62 67.31))
   (wire (pts (xy 171.45 72.39) (xy 172.72 72.39))
     (stroke (width 0) (type default))
@@
     (stroke (width 0) (type default))
   )
+  (wire (pts (xy 134.62 74.93) (xy 142.24 74.93))
+    (stroke (width 0) (type default))
+  )
   (wire (pts (xy 165.1 69.85) (xy 152.4 69.85))
     (stroke (width 0) (type default))
@@
   )
   (wire (pts (xy 176.53 68.58) (xy 186.69 68.58))
+    (stroke (width 0) (type default))
+  )
+  (wire (pts (xy 134.62 67.31) (xy 134.62 74.93))
     (stroke (width 0) (type default))
   )
@@
     (stroke (width 0) (type default))
   )
-  (text_box "Mistake! Pin 6 should be pulled low to enable the mux!"
-    (at 116.84 67.31 0) (size 16.51 15.24)
-    (stroke (width 0) (type default))
-    (fill (type none))
-    (effects (font (size 1.27 1.27)) (justify left top))
-  )
   (global_label "4051_ADDRESS_B" (shape input) (at 134.62 59.69 180) (fields_autoplaced)
