File: pcb/dk2_01/shiftregin.kicad_sch (KiCad schematic)
At the start: 17 parts, among them SW2 SW_Push, SW3 SW_Push, SW4 SW_Push, SW5 SW_Push, SW6 SW_Push, SW7 SW_Push, SW8 SW_Push, SW9 SW_Push, U3 74HC165

Commit message: going for a picnic
Parts:
- renumbered R9 to R13, R10 to R14, R11 to R15, R12 to R16, R13 to R17, R14 to R18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
