File: pcb/dk2_01/dk2_01.kicad_sch (KiCad schematic)
At the start: 9 parts, among them J1 GPIO_22, J2 GPIO_28, J3 Micro_SD_Card, SW1 Tap_Tempo_Button, U1 Pico

Commit message: good pcb progress
Parts:
- removed J1: GPIO_22, Connector_PinHeader_2.54mm:PinHeader_1x01_P2.54mm_Vertical, symbol Connector:Conn_01x01_Pin
- removed J2: GPIO_28, Connector_PinHeader_2.54mm:PinHeader_1x01_P2.54mm_Vertical, symbol Connector:Conn_01x01_Pin
- removed SW1: Tap_Tempo_Button, Button_Switch_THT:SW_PUSH_6mm, symbol Switch:SW_Push
- added D1: 1N5819WS, Diode_SMD:D_SOD-323, symbol Diode:1N5819WS
- added SW2 (x2): SW_Push, Button_Switch_THT:SW_PUSH_6mm, symbol Switch:SW_Push
- J3: footprint Connector_Card:microSD_HC_Molex_47219-2001 -> misc:YAMAICHI_MICROSD_VERTICAL
Connections:
- net +5V: now also D1.2 (A); no longer U1.39 (VSYS)
- net GND: now also SW2.1, SW2.1
- net START_STOP_BUTTON: now reaches U1.1 (GPIO0)
- net START_STOP_BUTTON: now also SW2.2
- net TAP_TEMPO_BUTTON: now reaches U1.2 (GPIO1)
- net TAP_TEMPO_BUTTON: now also SW2.2
- net GATE_OUT renamed TRIGGER_OUT_1
- net GPIO_22 renamed TRIGGER_OUT_3
- net GPIO_28 renamed TRIGGER_OUT_2
- net TAP_TEMPO_IN renamed TRIGGER_OUT_4
- new net: D1.1 (K), U1.39 (VSYS)

Commit message: going for a picnic
Parts:
- SW2: footprint Button_Switch_THT:SW_PUSH_6mm -> Button_Switch_THT:SW_PUSH-12mm
- renumbered J3 to J1
Changed lines of the file:
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@@
   (junction (at 193.04 86.36) (diameter 0) (color 0 0 0 0)
+  )
+  (junction (at 172.72 45.72) (diameter 0) (color 0 0 0 0)
   )
   (junction (at 151.13 99.06) (diameter 0) (color 0 0 0 0)
@@
     (stroke (width 0) (type default))
   )
+  (wire (pts (xy 172.72 45.72) (xy 177.165 45.72))
+    (stroke (width 0) (type default))
+  )
   (wire (pts (xy 212.725 114.3) (xy 217.17 114.3))
     (stroke (width 0) (type default))
@@
     (stroke (width 0) (type default))
   )
+  (wire (pts (xy 172.72 36.83) (xy 172.72 45.72))
+    (stroke (width 0) (type default))
+  )
   (wire (pts (xy 115.57 175.26) (xy 137.16 175.26))
     (stroke (width 0) (type default))
@@
     (stroke (width 0) (type default))
   )
+  (wire (pts (xy 167.005 36.83) (xy 172.72 36.83))
+    (stroke (width 0) (type default))
+  )
   (wire (pts (xy 151.13 99.06) (xy 114.3 99.06))
     (stroke (width 0) (type default))
@@
     (stroke (width 0) (type default))
   )
-  (wire (pts (xy 168.91 45.72) (xy 177.165 45.72))
+  (wire (pts (xy 168.91 45.72) (xy 172.72 45.72))
     (stroke (width 0) (type default))
   )
@@
   (symbol (lib_id "power:GND") (at 142.875 141.605 0) (unit 1)
     (in_bom yes) (on_board yes) (dnp no) (fields_autoplaced)
-    (property "Reference" "#PWR077" (at 142.875 147.955 0)
+    (property "Reference" "#PWR04" (at 142.875 147.955 0)
       (effects (font (size 1.27 1.27)) hide)
     )
@@
       (project "dk2_01"
         (path "/87a59a99-d509-467e-85da-26d34072acb7"
-          (reference "#PWR077") (unit 1)
+          (reference "#PWR04") (unit 1)
         )
       )
@@
   (symbol (lib_id "power:+3.3V") (at 185.42 36.83 0) (unit 1)
     (in_bom yes) (on_board yes) (dnp no) (fields_autoplaced)
-    (property "Reference" "#PWR07" (at 185.42 40.64 0)
+    (property "Reference" "#PWR08" (at 185.42 40.64 0)
       (effects (font (size 1.27 1.27)) hide)
     )
@@
       (project "dk2_01"
         (path "/87a59a99-d509-467e-85da-26d34072acb7"
-          (reference "#PWR07") (unit 1)
+          (reference "#PWR08") (unit 1)
         )
       )
@@
   (symbol (lib_id "power:GND") (at 212.725 77.47 0) (unit 1)
     (in_bom yes) (on_board yes) (dnp no) (fields_autoplaced)
-    (property "Reference" "#PWR048" (at 212.725 83.82 0)
+    (property "Reference" "#PWR09" (at 212.725 83.82 0)
       (effects (font (size 1.27 1.27)) hide)
     )
@@
       (project "dk2_01"
         (path "/87a59a99-d509-467e-85da-26d34072acb7"
-          (reference "#PWR048") (unit 1)
+          (reference "#PWR09") (unit 1)
         )
       )
@@
       (effects (font (size 1.27 1.27)))
     )
-    (property "Footprint" "Button_Switch_THT:SW_PUSH_6mm" (at 147.955 121.285 0)
+    (property "Footprint" "Button_Switch_THT:SW_PUSH-12mm" (at 147.955 121.285 0)
       (effects (font (size 1.27 1.27)) hide)
     )
@@
   (symbol (lib_id "power:GND") (at 142.875 126.365 0) (unit 1)
     (in_bom yes) (on_board yes) (dnp no) (fields_autoplaced)
-    (property "Reference" "#PWR058" (at 142.875 132.715 0)
+    (property "Reference" "#PWR03" (at 142.875 132.715 0)
       (effects (font (size 1.27 1.27)) hide)
     )
@@
       (project "dk2_01"
         (path "/87a59a99-d509-467e-85da-26d34072acb7"
-          (reference "#PWR058") (unit 1)
+          (reference "#PWR03") (unit 1)
         )
       )
@@
       (effects (font (size 1.27 1.27)))
     )
-    (property "Footprint" "Button_Switch_THT:SW_PUSH_6mm" (at 147.955 136.525 0)
+    (property "Footprint" "Button_Switch_THT:SW_PUSH-12mm" (at 147.955 136.525 0)
       (effects (font (size 1.27 1.27)) hide)
     )
@@
         )
         (path "/87a59a99-d509-467e-85da-26d34072acb7"
-          (reference "SW18") (unit 1)
+          (reference "SW2") (unit 1)
+        )
+      )
+    )
+  )
+  (symbol (lib_id "power:PWR_FLAG") (at 167.005 36.83 0) (unit 1)
+    (in_bom yes) (on_board yes) (dnp no) (fields_autoplaced)
+    (property "Reference" "#FLG06" (at 167.005 34.925 0)
+      (effects (font (size 1.27 1.27)) hide)
+    )
+    (property "Value" "PWR_FLAG" (at 167.005 33.3281 0)
+      (effects (font (size 1.27 1.27)))
+    )
+    (property "Footprint" "" (at 167.005 36.83 0)
+      (effects (font (size 1.27 1.27)) hide)
+    )
+    (property "Datasheet" "~" (at 167.005 36.83 0)
+      (effects (font (size 1.27 1.27)) hide)
+    )
+    (pin "1")
+    (instances
+      (project "dk2_01"
+        (path "/87a59a99-d509-467e-85da-26d34072acb7"
+          (reference "#FLG06") (unit 1)
         )
       )
@@
   (symbol (lib_id "power:GND") (at 151.13 100.33 0) (unit 1)
     (in_bom yes) (on_board yes) (dnp no) (fields_autoplaced)
-    (property "Reference" "#PWR03" (at 151.13 106.68 0)
+    (property "Reference" "#PWR05" (at 151.13 106.68 0)
       (effects (font (size 1.27 1.27)) hide)
     )
@@
       (project "dk2_01"
         (path "/87a59a99-d509-467e-85da-26d34072acb7"
-          (reference "#PWR03") (unit 1)
+          (reference "#PWR05") (unit 1)
         )
       )
@@
   (symbol (lib_id "power:GND") (at 180.34 190.5 0) (unit 1)
     (in_bom yes) (on_board yes) (dnp no) (fields_autoplaced)
-    (property "Reference" "#PWR06" (at 180.34 196.85 0)
+    (property "Reference" "#PWR07" (at 180.34 196.85 0)
       (effects (font (size 1.27 1.27)) hide)
     )
@@
       (project "dk2_01"
         (path "/87a59a99-d509-467e-85da-26d34072acb7"
+          (reference "#PWR07") (unit 1)
+        )
+      )
+    )
+  )
+  (symbol (lib_id "power:+5V") (at 177.165 36.83 0) (unit 1)
+    (in_bom yes) (on_board yes) (dnp no) (fields_autoplaced)
+    (property "Reference" "#PWR06" (at 177.165 40.64 0)
+      (effects (font (size 1.27 1.27)) hide)
+    )
+    (property "Value" "+5V" (at 177.165 33.3281 0)
+      (effects (font (size 1.27 1.27)))
+    )
+    (property "Footprint" "" (at 177.165 36.83 0)
+      (effects (font (size 1.27 1.27)) hide)
+    )
+    (property "Datasheet" "" (at 177.165 36.83 0)
+      (effects (font (size 1.27 1.27)) hide)
+    )
+    (pin "1")
+    (instances
+      (project "dk2_01"
+        (path "/87a59a99-d509-467e-85da-26d34072acb7"
           (reference "#PWR06") (unit 1)
-        )
-      )
-    )
-  )
-  (symbol (lib_id "power:+5V") (at 177.165 36.83 0) (unit 1)
-    (in_bom yes) (on_board yes) (dnp no) (fields_autoplaced)
-    (property "Reference" "#PWR05" (at 177.165 40.64 0)
-      (effects (font (size 1.27 1.27)) hide)
-    )
-    (property "Value" "+5V" (at 177.165 33.3281 0)
-      (effects (font (size 1.27 1.27)))
-    )
-    (property "Footprint" "" (at 177.165 36.83 0)
-      (effects (font (size 1.27 1.27)) hide)
-    )
-    (property "Datasheet" "" (at 177.165 36.83 0)
-      (effects (font (size 1.27 1.27)) hide)
-    )
-    (pin "1")
-    (instances
-      (project "dk2_01"
-        (path "/87a59a99-d509-467e-85da-26d34072acb7"
-          (reference "#PWR05") (unit 1)
         )
       )
@@
   (symbol (lib_id "Connector:Micro_SD_Card") (at 160.02 175.26 0) (unit 1)
     (in_bom yes) (on_board yes) (dnp no)
-    (property "Reference" "J3" (at 160.02 156.2131 0)
+    (property "Reference" "J1" (at 160.02 156.2131 0)
       (effects (font (size 1.27 1.27)))
     )
@@
       (project "dk2_01"
         (path "/87a59a99-d509-467e-85da-26d34072acb7"
-          (reference "J3") (unit 1)
-        )
-      )
+          (reference "J1") (unit 1)
+        )
+      )
