File: pcb/dk2_01/dac.kicad_sch (KiCad schematic)
At the start: 40 parts, among them J15 Euro_Out_1, J15 Euro_Out_2, J6 Line_Out, U4 AP7333-33SRG, U5 TL072, U6 PCM5102

Commit message: good pcb progress
Parts:
- removed J6: Line_Out, Library:Jack_3.5mm_QingPu_WQP-PJ366ST_Vertical_Labelled, symbol Connector_Audio:AudioJack3
Connections:
- net +3.3VDAC: now also U4.2 (VO); no longer U4.3 (VO)
- net GND: now also U4.3 (GND); no longer U4.2 (GND)
Changed lines of the file:
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@@
   (junction (at 128.27 57.15) (diameter 0) (color 0 0 0 0)
   )
-  (junction (at 214.63 69.85) (diameter 0) (color 0 0 0 0)
-  )
   (junction (at 177.8 57.15) (diameter 0) (color 0 0 0 0)
   )
   (junction (at 58.42 106.045) (diameter 0) (color 0 0 0 0)
   )
-  (junction (at 224.79 36.83) (diameter 0) (color 0 0 0 0)
-  )
   (junction (at 214.63 39.37) (diameter 0) (color 0 0 0 0)
   )
@@
   )
   (junction (at 73.66 94.615) (diameter 0) (color 0 0 0 0)
-  )
-  (junction (at 220.98 39.37) (diameter 0) (color 0 0 0 0)
   )
   (junction (at 177.8 69.85) (diameter 0) (color 0 0 0 0)
@@
     (stroke (width 0) (type default))
   )
-  (wire (pts (xy 214.63 39.37) (xy 220.98 39.37))
+  (wire (pts (xy 214.63 39.37) (xy 227.33 39.37))
     (stroke (width 0) (type default))
   )
@@
     (stroke (width 0) (type default))
   )
-  (wire (pts (xy 224.79 36.83) (xy 224.79 44.45))
-    (stroke (width 0) (type default))
-  )
   (wire (pts (xy 184.15 69.85) (xy 208.28 69.85))
     (stroke (width 0) (type default))
@@
     (stroke (width 0) (type default))
   )
-  (wire (pts (xy 214.63 69.85) (xy 246.38 69.85))
-    (stroke (width 0) (type default))
-  )
   (wire (pts (xy 177.8 39.37) (xy 214.63 39.37))
     (stroke (width 0) (type default))
@@
     (stroke (width 0) (type default))
   )
-  (wire (pts (xy 220.98 46.99) (xy 246.38 46.99))
-    (stroke (width 0) (type default))
-  )
   (wire (pts (xy 128.27 52.07) (xy 128.27 57.15))
     (stroke (width 0) (type default))
   )
-  (wire (pts (xy 246.38 69.85) (xy 246.38 49.53))
-    (stroke (width 0) (type default))
-  )
   (wire (pts (xy 73.66 75.565) (xy 73.66 85.725))
     (stroke (width 0) (type default))
@@
     (stroke (width 0) (type default))
   )
-  (wire (pts (xy 208.28 36.83) (xy 224.79 36.83))
+  (wire (pts (xy 208.28 36.83) (xy 227.33 36.83))
     (stroke (width 0) (type default))
   )
@@
     (stroke (width 0) (type default))
   )
-  (wire (pts (xy 220.98 39.37) (xy 220.98 46.99))
-    (stroke (width 0) (type default))
-  )
   (wire (pts (xy 128.27 44.45) (xy 128.27 49.53))
     (stroke (width 0) (type default))
@@
     (stroke (width 0) (type default))
   )
-  (wire (pts (xy 220.98 39.37) (xy 227.33 39.37))
-    (stroke (width 0) (type default))
-  )
   (wire (pts (xy 156.21 39.37) (xy 170.18 39.37))
     (stroke (width 0) (type default))
@@
     (stroke (width 0) (type default))
   )
-  (wire (pts (xy 224.79 44.45) (xy 246.38 44.45))
-    (stroke (width 0) (type default))
-  )
   (wire (pts (xy 43.18 92.075) (xy 45.72 92.075))
     (stroke (width 0) (type default))
@@
     (stroke (width 0) (type default))
   )
-  (wire (pts (xy 224.79 36.83) (xy 227.33 36.83))
-    (stroke (width 0) (type default))
-  )
   (wire (pts (xy 45.72 99.695) (xy 45.72 106.045))
     (stroke (width 0) (type default))
@@
     (stroke (width 0) (type default))
   )
-  (text_box "THIS PINOUT IS WRONG! MAGIC SMOKE RELEASED ON TEST BOARD!"
+  (text_box "Warning! Default Kicad pin mapping for for this component is wrong! Pins 2 and 3 were swapped, causing magic smoke release on previous board."
     (at 23.495 53.34 0) (size 41.91 10.795)
     (stroke (width 0) (type default))
@@
     )
   )
-  (symbol (lib_id "Connector_Audio:AudioJack3") (at 251.46 46.99 180) (unit 1)
-    (in_bom yes) (on_board yes) (dnp no) (fields_autoplaced)
-    (property "Reference" "J6" (at 259.08 45.72 0)
-      (effects (font (size 1.27 1.27)) (justify right))
-    )
-    (property "Value" "Line_Out" (at 259.08 48.26 0)
-      (effects (font (size 1.27 1.27)) (justify right))
-    )
-    (property "Footprint" "Library:Jack_3.5mm_QingPu_WQP-PJ366ST_Vertical_Labelled" (at 251.46 46.99 0)
-      (effects (font (size 1.27 1.27)) hide)
-    )
-    (property "Datasheet" "~" (at 251.46 46.99 0)
-      (effects (font (size 1.27 1.27)) hide)
-    )
-    (pin "R")
-    (pin "S")
-    (pin "T")
-    (instances
-      (project "dk2_01"
-        (path "/87a59a99-d509-467e-85da-26d34072acb7/a3b4dd4a-c522-40f2-b825-f444d434bc45"
-          (reference "J6") (unit 1)
-        )
-      )
-    )
-  )
   (symbol (lib_id "Device:C") (at 177.8 66.04 0) (unit 1)
     (in_bom yes) (on_board yes) (dnp no)
@@
     )
     (pin "1")
-    (pin "2")
     (pin "3")
-    (instances
-      (project "dk2_01"
+    (pin "2")
+    (instances
+      (project "dk2_01"

Commit message: going for a picnic
Parts:
- renumbered C6 to C10, C7 to C11, C8 to C12, C9 to C13, C10 to C14, C11 to C15, C12 to C16, C13 to C17, C14 to C18, C15 to C19, C16 to C20, C17 to C21, C18 to C22, C19 to C23, C20 to C24, C21 to C25, C1 to C5, C2 to C6, C3 to C7, C4 to C8, C5 to C9, R17 to R41, R18 to R42, R19 to R43, R20 to R44, R21 to R45, R22 to R46, R23 to R47, R24 to R48, R25 to R49, R26 to R50, R27 to R51, R28 to R52, R29 to R53, U4 to U11, U5 to U12, U6 to U13

Commit message: tweaking the front panel based on the pcb
Parts:
- J15: footprint Library:Jack_3.5mm_QingPu_WQP-PJ398SM_Vertical_Labelled -> AudioJacks:Jack_3.5mm_QingPu_WQP-PJ398SM_Vertical
Changed lines of the file:
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@@
       (effects (font (size 1.27 1.27)) (justify right))
     )
-    (property "Footprint" "Library:Jack_3.5mm_QingPu_WQP-PJ398SM_Vertical_Labelled" (at 91.44 94.615 0)
+    (property "Footprint" "AudioJacks:Jack_3.5mm_QingPu_WQP-PJ398SM_Vertical" (at 91.44 94.615 0)
       (effects (font (size 1.27 1.27)) hide)
     )
@@
       (effects (font (size 1.27 1.27)) (justify right))
     )
-    (property "Footprint" "Library:Jack_3.5mm_QingPu_WQP-PJ398SM_Vertical_Labelled" (at 91.44 142.24 0)
-      (effects (font (size 1.27 1.27)) hide)
-    )
+    (property "Footprint" "AudioJacks:Jack_3.5mm_QingPu_WQP-PJ398SM_Vertical" (at 91.44 142.24 0)
+      (effects (font (size 1.27 1.27)) hide)
+    )
