File: pcb/dk2_01/power.kicad_sch (KiCad schematic)
At the start: 7 parts, among them J15 Eurorack_Power, U12 XL1509-5.0

Commit message: going for a picnic
Parts:
- renumbered C25 to C29, C26 to C30, C29 to C31, D10 to D6, J15 to J14, U12 to U17
Changed lines of the file:
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@@
   (symbol (lib_id "Device:C_Polarized_US") (at 105.41 124.46 0) (unit 1)
     (in_bom yes) (on_board yes) (dnp no)
-    (property "Reference" "C25" (at 97.155 123.825 0)
+    (property "Reference" "C29" (at 97.155 123.825 0)
       (effects (font (size 1.27 1.27)) (justify left))
     )
@@
       (project "dk2_01"
         (path "/87a59a99-d509-467e-85da-26d34072acb7/be1ddc4d-f499-4b75-b4b5-b626a320d90d"
-          (reference "C25") (unit 1)
+          (reference "C29") (unit 1)
         )
       )
@@
   (symbol (lib_id "Device:C") (at 113.03 124.46 0) (unit 1)
     (in_bom yes) (on_board yes) (dnp no) (fields_autoplaced)
-    (property "Reference" "C26" (at 115.951 123.8163 0)
+    (property "Reference" "C30" (at 115.951 123.8163 0)
       (effects (font (size 1.27 1.27)) (justify left))
     )
@@
       (project "dk2_01"
         (path "/87a59a99-d509-467e-85da-26d34072acb7/be1ddc4d-f499-4b75-b4b5-b626a320d90d"
-          (reference "C26") (unit 1)
+          (reference "C30") (unit 1)
         )
       )
@@
   (symbol (lib_id "power:GND") (at 120.015 81.28 0) (mirror y) (unit 1)
     (in_bom yes) (on_board yes) (dnp no) (fields_autoplaced)
-    (property "Reference" "#PWR056" (at 120.015 87.63 0)
+    (property "Reference" "#PWR075" (at 120.015 87.63 0)
       (effects (font (size 1.27 1.27)) hide)
     )
@@
       (project "dk2_01"
         (path "/87a59a99-d509-467e-85da-26d34072acb7/be1ddc4d-f499-4b75-b4b5-b626a320d90d"
-          (reference "#PWR056") (unit 1)
+          (reference "#PWR075") (unit 1)
         )
       )
@@
   (symbol (lib_id "power:+5V") (at 168.275 114.3 0) (unit 1)
     (in_bom yes) (on_board yes) (dnp no) (fields_autoplaced)
-    (property "Reference" "#PWR071" (at 168.275 118.11 0)
+    (property "Reference" "#PWR080" (at 168.275 118.11 0)
       (effects (font (size 1.27 1.27)) hide)
     )
@@
       (project "dk2_01"
         (path "/87a59a99-d509-467e-85da-26d34072acb7/be1ddc4d-f499-4b75-b4b5-b626a320d90d"
-          (reference "#PWR071") (unit 1)
+          (reference "#PWR080") (unit 1)
         )
       )
@@
   (symbol (lib_id "Connector_Generic:Conn_02x05_Odd_Even") (at 138.43 71.755 180) (unit 1)
     (in_bom yes) (on_board yes) (dnp no)
-    (property "Reference" "J15" (at 156.845 60.96 0)
+    (property "Reference" "J14" (at 156.845 60.96 0)
       (effects (font (size 1.27 1.27)))
     )
@@
       (project "dk2_01"
         (path "/87a59a99-d509-467e-85da-26d34072acb7/be1ddc4d-f499-4b75-b4b5-b626a320d90d"
-          (reference "J15") (unit 1)
+          (reference "J14") (unit 1)
         )
       )
@@
   (symbol (lib_id "power:GND") (at 154.305 81.28 0) (unit 1)
     (in_bom yes) (on_board yes) (dnp no) (fields_autoplaced)
-    (property "Reference" "#PWR064" (at 154.305 87.63 0)
+    (property "Reference" "#PWR079" (at 154.305 87.63 0)
       (effects (font (size 1.27 1.27)) hide)
     )
@@
       (project "dk2_01"
         (path "/87a59a99-d509-467e-85da-26d34072acb7/be1ddc4d-f499-4b75-b4b5-b626a320d90d"
-          (reference "#PWR064") (unit 1)
+          (reference "#PWR079") (unit 1)
         )
       )
@@
   (symbol (lib_id "power:+12V") (at 105.41 120.65 0) (unit 1)
     (in_bom yes) (on_board yes) (dnp no) (fields_autoplaced)
-    (property "Reference" "#PWR065" (at 105.41 124.46 0)
+    (property "Reference" "#PWR074" (at 105.41 124.46 0)
       (effects (font (size 1.27 1.27)) hide)
     )
@@
       (project "dk2_01"
         (path "/87a59a99-d509-467e-85da-26d34072acb7/be1ddc4d-f499-4b75-b4b5-b626a320d90d"
-          (reference "#PWR065") (unit 1)
+          (reference "#PWR074") (unit 1)
         )
       )
@@
   (symbol (lib_id "power:+12V") (at 137.16 60.325 0) (unit 1)
     (in_bom yes) (on_board yes) (dnp no) (fields_autoplaced)
-    (property "Reference" "#PWR060" (at 137.16 64.135 0)
+    (property "Reference" "#PWR077" (at 137.16 64.135 0)
       (effects (font (size 1.27 1.27)) hide)
     )
@@
       (project "dk2_01"
         (path "/87a59a99-d509-467e-85da-26d34072acb7/be1ddc4d-f499-4b75-b4b5-b626a320d90d"
-          (reference "#PWR060") (unit 1)
+          (reference "#PWR077") (unit 1)
         )
       )
@@
   (symbol (lib_id "Device:C_Polarized_US") (at 168.275 124.46 0) (unit 1)
     (in_bom yes) (on_board yes) (dnp no) (fields_autoplaced)
-    (property "Reference" "C29" (at 171.196 123.1813 0)
+    (property "Reference" "C31" (at 171.196 123.1813 0)
       (effects (font (size 1.27 1.27)) (justify left))
     )
@@
       (project "dk2_01"
         (path "/87a59a99-d509-467e-85da-26d34072acb7/be1ddc4d-f499-4b75-b4b5-b626a320d90d"
-          (reference "C29") (unit 1)
+          (reference "C31") (unit 1)
         )
       )
@@
   (symbol (lib_id "power:GND") (at 133.35 130.81 0) (unit 1)
     (in_bom yes) (on_board yes) (dnp no) (fields_autoplaced)
-    (property "Reference" "#PWR066" (at 133.35 137.16 0)
+    (property "Reference" "#PWR076" (at 133.35 137.16 0)
       (effects (font (size 1.27 1.27)) hide)
     )
@@
       (project "dk2_01"
         (path "/87a59a99-d509-467e-85da-26d34072acb7/be1ddc4d-f499-4b75-b4b5-b626a320d90d"
-          (reference "#PWR066") (unit 1)
+          (reference "#PWR076") (unit 1)
         )
       )
@@
   (symbol (lib_id "Regulator_Switching:XL1509-5.0") (at 133.35 123.19 0) (unit 1)
     (in_bom yes) (on_board yes) (dnp no) (fields_autoplaced)
-    (property "Reference" "U12" (at 133.35 115.1001 0)
+    (property "Reference" "U17" (at 133.35 115.1001 0)
       (effects (font (size 1.27 1.27)))
     )
@@
       (project "dk2_01"
         (path "/87a59a99-d509-467e-85da-26d34072acb7/be1ddc4d-f499-4b75-b4b5-b626a320d90d"
-          (reference "U12") (unit 1)
+          (reference "U17") (unit 1)
         )
       )
@@
   (symbol (lib_id "Diode:1N5820") (at 153.67 124.46 270) (unit 1)
     (in_bom yes) (on_board yes) (dnp no) (fields_autoplaced)
-    (property "Reference" "D10" (at 155.702 123.4988 90)
+    (property "Reference" "D6" (at 155.702 123.4988 90)
       (effects (font (size 1.27 1.27)) (justify left))
     )
@@
       (project "dk2_01"
         (path "/87a59a99-d509-467e-85da-26d34072acb7/be1ddc4d-f499-4b75-b4b5-b626a320d90d"
-          (reference "D10") (unit 1)
+          (reference "D6") (unit 1)
         )
       )
@@
   (symbol (lib_id "power:-12V") (at 137.16 83.82 0) (unit 1)
     (in_bom yes) (on_board yes) (dnp no) (fields_autoplaced)
-    (property "Reference" "#PWR061" (at 137.16 81.28 0)
+    (property "Reference" "#PWR078" (at 137.16 81.28 0)
       (effects (font (size 1.27 1.27)) hide)
     )
@@
       (project "dk2_01"
         (path "/87a59a99-d509-467e-85da-26d34072acb7/be1ddc4d-f499-4b75-b4b5-b626a320d90d"
-          (reference "#PWR061") (unit 1)
-        )
-      )
+          (reference "#PWR078") (unit 1)
+        )
+      )

Commit message: pcb layout going well
Parts:
- C31: footprint Capacitor_THT:CP_Radial_D10.0mm_P5.00mm -> Capacitor_THT:CP_Radial_D8.0mm_P3.50mm
- L1: footprint Inductor_THT:L_Radial_D8.7mm_P5.00mm_Fastron_07HCP -> Inductor_THT:L_Radial_D7.0mm_P3.00mm
Changed lines of the file:
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@@
       (effects (font (size 1.27 1.27)))
     )
-    (property "Footprint" "Inductor_THT:L_Radial_D8.7mm_P5.00mm_Fastron_07HCP" (at 160.655 120.65 0)
+    (property "Footprint" "Inductor_THT:L_Radial_D7.0mm_P3.00mm" (at 160.655 120.65 0)
       (effects (font (size 1.27 1.27)) hide)
     )
@@
       (effects (font (size 1.27 1.27)) (justify left))
     )
-    (property "Footprint" "Capacitor_THT:CP_Radial_D10.0mm_P5.00mm" (at 168.275 124.46 0)
+    (property "Footprint" "Capacitor_THT:CP_Radial_D8.0mm_P3.50mm" (at 168.275 124.46 0)
       (effects (font (size 1.27 1.27)) hide)
     )

Commit message: more layout tweaks
Changed lines of the file:
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@@
     (stroke (width 0) (type default))
+  )
+  (text_box "N.B. \"Keep feedback wiring away from inductor flux\" (per datasheet)"
+    (at 149.225 97.79 0) (size 24.13 10.795)
+    (stroke (width 0) (type default))
+    (fill (type none))
+    (effects (font (size 1.27 1.27)) (justify left top))
+  )
+  (text_box "Datasheet called for 68uH/2A, but did some calculations and think I can get away with 47uH/1A, which is what I used in the first board."
+    (at 179.07 105.41 0) (size 34.29 12.7)
+    (stroke (width 0) (type default))
+    (fill (type none))
+    (effects (font (size 1.27 1.27)) (justify left top))
   )
   (text "Eurorack power input" (at 127.635 51.435 0)
