File: pcb/dk2_01/shiftregout.kicad_sch (KiCad schematic)
At the start: 19 parts, among them U13 CA56-12EWA, U14 74HC595, U2 74HC595

Commit message: good pcb progress
Parts:
- D2: footprint LED_SMD:LED_0805_2012Metric -> LED_THT:LED_D5.0mm
Changed lines of the file:
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@@
+    (effects (font (size 1.27 1.27)) (justify left top))
+  )
+  (text_box "Pinout matches SR410361N, which is cheap on LCSC"
+    (at 189.865 33.655 0) (size 31.115 6.35)
+    (stroke (width 0) (type default))
+    (fill (type none))
     (effects (font (size 1.27 1.27)) (justify left top))
   )
@@
       (effects (font (size 1.27 1.27)))
     )
-    (property "Footprint" "LED_SMD:LED_0805_2012Metric" (at 158.75 118.745 0)
+    (property "Footprint" "LED_THT:LED_D5.0mm" (at 158.75 118.745 0)
       (effects (font (size 1.27 1.27)) hide)
     )

Commit message: going for a picnic
Parts:
- renumbered R2 to R1, R57 to R10, R58 to R11, R59 to R12, R3 to R2, R4 to R3, R5 to R4, R52 to R5, R53 to R6, R54 to R7, R55 to R8, R56 to R9, U14 to U3, U13 to U4

Commit message: pcb layout going well
Changed lines of the file:
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@@
     (effects (font (size 1.27 1.27)) (justify left top))
   )
-  (text_box "Pinout matches SR410361N, which is cheap on LCSC"
-    (at 189.865 33.655 0) (size 31.115 6.35)
+  (text_box "Pinout matches Shenzhen Zhihao Elec C10713, which is cheap on LCSC"
+    (at 189.865 33.655 0) (size 31.115 7.62)
     (stroke (width 0) (type default))
     (fill (type none))

Commit message: more layout tweaks
Parts:
- U4: footprint Display_7Segment:CA56-12EWA -> Library:SR410361N
Changed lines of the file:
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@@
     (effects (font (size 1.27 1.27)) (justify left top))
   )
-  (text_box "Pinout matches Shenzhen Zhihao Elec C10713, which is cheap on LCSC"
+  (text_box "Pinout matches SR410361N (smaller display), which is cheap on LCSC"
     (at 189.865 33.655 0) (size 31.115 7.62)
     (stroke (width 0) (type default))
@@
       (effects (font (size 1.27 1.27)))
     )
-    (property "Footprint" "Display_7Segment:CA56-12EWA" (at 206.375 74.93 0)
-      (effects (font (size 1.27 1.27)) hide)
-    )
+    (property "Footprint" "Library:SR410361N" (at 206.375 74.93 0)
+      (effects (font (size 1.27 1.27)) hide)
+    )
