File: pcb/dk2_02_bottom/dac.kicad_sch (KiCad schematic)
At the start: 37 parts, among them U11 AP7333-33SRG, U12 TL072, U13 PCM5102

Commit message: bottom pcb looks fairly easy
Parts:
- renumbered C5 to C1, C14 to C10, C15 to C11, C16 to C12, C17 to C13, C18 to C14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
