File: pcb/dk2_02_top/muxin2.kicad_sch (KiCad schematic)
At the start: 27 parts, among them J12 CV_In_1, J12 CV_In_2, J12 CV_In_3, J12 CV_In_4, U6 74HC4051, U7 MCP6002-xSN, U8 MCP6002-xSN

Commit message: done for the week, started routing
Parts:
- renumbered J12 to J13, J12 to J14, J12 to J15
Changed lines of the file:
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@@
     )
   )
-  (global_label "CV_IN_3" (shape input) (at 149.225 48.895 0) (fields_autoplaced)
+  (global_label "CV_IN_3" (shape output) (at 149.225 48.895 0) (fields_autoplaced)
     (effects (font (size 1.27 1.27)) (justify left))
     (property "Intersheetrefs" "${INTERSHEET_REFS}" (at 159.5694 48.895 0)
@@
     )
   )
-  (global_label "CV_IN_4" (shape input) (at 149.225 92.71 0) (fields_autoplaced)
+  (global_label "CV_IN_4" (shape output) (at 149.225 92.71 0) (fields_autoplaced)
     (effects (font (size 1.27 1.27)) (justify left))
     (property "Intersheetrefs" "${INTERSHEET_REFS}" (at 159.5694 92.71 0)
@@
     )
   )
-  (global_label "CV_IN_1" (shape input) (at 90.805 48.895 0) (fields_autoplaced)
+  (global_label "CV_IN_1" (shape output) (at 90.805 48.895 0) (fields_autoplaced)
     (effects (font (size 1.27 1.27)) (justify left))
     (property "Intersheetrefs" "${INTERSHEET_REFS}" (at 101.1494 48.895 0)
@@
     )
   )
-  (global_label "CV_IN_2" (shape input) (at 90.805 92.71 0) (fields_autoplaced)
+  (global_label "CV_IN_2" (shape output) (at 90.805 92.71 0) (fields_autoplaced)
     (effects (font (size 1.27 1.27)) (justify left))
     (property "Intersheetrefs" "${INTERSHEET_REFS}" (at 101.1494 92.71 0)
@@
   (symbol (lib_id "Connector_Audio:AudioJack2_SwitchT") (at 116.84 46.355 0) (mirror x) (unit 1)
     (in_bom yes) (on_board yes) (dnp no) (fields_autoplaced)
-    (property "Reference" "J12" (at 112.2681 45.0763 0)
+    (property "Reference" "J14" (at 112.2681 45.0763 0)
       (effects (font (size 1.27 1.27)) (justify right))
     )
@@
   (symbol (lib_id "Connector_Audio:AudioJack2_SwitchT") (at 116.84 90.17 0) (mirror x) (unit 1)
     (in_bom yes) (on_board yes) (dnp no) (fields_autoplaced)
-    (property "Reference" "J12" (at 112.2681 88.8913 0)
+    (property "Reference" "J15" (at 112.2681 88.8913 0)
       (effects (font (size 1.27 1.27)) (justify right))
     )
@@
   (symbol (lib_id "Connector_Audio:AudioJack2_SwitchT") (at 58.42 90.17 0) (mirror x) (unit 1)
     (in_bom yes) (on_board yes) (dnp no) (fields_autoplaced)
-    (property "Reference" "J12" (at 52.705 88.9 0)
-      (effects (font (size 1.27 1.27)) (justify right))
-    )
+    (property "Reference" "J13" (at 52.705 88.9 0)
+      (effects (font (size 1.27 1.27)) (justify right))
+    )
