File: pcb/dk2_02_top/dk2_02_top.kicad_sch (KiCad schematic)
At the start: 17 parts, among them J1 Conn_01x18_Pin, J12 Euro_Out_1, J12 Euro_Out_2, J12 Sync_In, J12 Sync_Out, J12 Trigger_Out_1, J12 Trigger_Out_2, J12 Trigger_Out_3, J12 Trigger_Out_4, J6 Micro_SD_Card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

Commit message: done for the week, started routing
Parts:
- renumbered J12 to J2
Connections:
- net 595_CLOCK: now also J7.11 (Pin_11); no longer J7.7 (Pin_7)
- net 595_DATA: now also J7.10 (Pin_10); no longer J7.6 (Pin_6)
- net 595_LATCH: now also J7.12 (Pin_12); no longer J7.8 (Pin_8)
- net SD_CHIP_SELECT: now also J7.9 (Pin_9); no longer J7.12 (Pin_12)
- net SD_CLOCK: now also J7.6 (Pin_6); no longer J7.9 (Pin_9)
- net SD_SERIAL_IN: now also J7.7 (Pin_7); no longer J7.10 (Pin_10)
- net SD_SERIAL_OUT: now also J7.8 (Pin_8); no longer J7.11 (Pin_11)
Changed lines of the file:
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@@
     )
   )
-  (global_label "SD_SERIAL_IN" (shape output) (at 86.36 46.355 0) (fields_autoplaced)
-    (effects (font (size 1.27 1.27)) (justify left))
-    (property "Intersheetrefs" "${INTERSHEET_REFS}" (at 101.9658 46.355 0)
+  (global_label "SD_SERIAL_IN" (shape output) (at 86.36 38.735 0) (fields_autoplaced)
+    (effects (font (size 1.27 1.27)) (justify left))
+    (property "Intersheetrefs" "${INTERSHEET_REFS}" (at 101.9658 38.735 0)
       (effects (font (size 1.27 1.27)) (justify left) hide)
     )
@@
     )
   )
-  (global_label "595_LATCH" (shape output) (at 86.36 41.275 0) (fields_autoplaced)
-    (effects (font (size 1.27 1.27)) (justify left))
-    (property "Intersheetrefs" "${INTERSHEET_REFS}" (at 99.5467 41.275 0)
+  (global_label "595_LATCH" (shape output) (at 86.36 51.435 0) (fields_autoplaced)
+    (effects (font (size 1.27 1.27)) (justify left))
+    (property "Intersheetrefs" "${INTERSHEET_REFS}" (at 99.5467 51.435 0)
       (effects (font (size 1.27 1.27)) (justify left) hide)
     )
@@
     )
   )
-  (global_label "595_DATA" (shape output) (at 86.36 36.195 0) (fields_autoplaced)
-    (effects (font (size 1.27 1.27)) (justify left))
-    (property "Intersheetrefs" "${INTERSHEET_REFS}" (at 98.2767 36.195 0)
-      (effects (font (size 1.27 1.27)) (justify left) hide)
-    )
-  )
-  (global_label "SD_CHIP_SELECT" (shape output) (at 86.36 51.435 0) (fields_autoplaced)
-    (effects (font (size 1.27 1.27)) (justify left))
-    (property "Intersheetrefs" "${INTERSHEET_REFS}" (at 104.929 51.435 0)
+  (global_label "595_DATA" (shape output) (at 86.36 46.355 0) (fields_autoplaced)
+    (effects (font (size 1.27 1.27)) (justify left))
+    (property "Intersheetrefs" "${INTERSHEET_REFS}" (at 98.2767 46.355 0)
+      (effects (font (size 1.27 1.27)) (justify left) hide)
+    )
+  )
+  (global_label "SD_CHIP_SELECT" (shape output) (at 86.36 43.815 0) (fields_autoplaced)
+    (effects (font (size 1.27 1.27)) (justify left))
+    (property "Intersheetrefs" "${INTERSHEET_REFS}" (at 104.929 43.815 0)
       (effects (font (size 1.27 1.27)) (justify left) hide)
     )
@@
     )
   )
-  (global_label "SD_SERIAL_OUT" (shape input) (at 86.36 48.895 0) (fields_autoplaced)
-    (effects (font (size 1.27 1.27)) (justify left))
-    (property "Intersheetrefs" "${INTERSHEET_REFS}" (at 103.6591 48.895 0)
+  (global_label "SD_SERIAL_OUT" (shape input) (at 86.36 41.275 0) (fields_autoplaced)
+    (effects (font (size 1.27 1.27)) (justify left))
+    (property "Intersheetrefs" "${INTERSHEET_REFS}" (at 103.6591 41.275 0)
       (effects (font (size 1.27 1.27)) (justify left) hide)
     )
@@
     )
   )
-  (global_label "595_CLOCK" (shape output) (at 86.36 38.735 0) (fields_autoplaced)
-    (effects (font (size 1.27 1.27)) (justify left))
-    (property "Intersheetrefs" "${INTERSHEET_REFS}" (at 100.0305 38.735 0)
+  (global_label "595_CLOCK" (shape output) (at 86.36 48.895 0) (fields_autoplaced)
+    (effects (font (size 1.27 1.27)) (justify left))
+    (property "Intersheetrefs" "${INTERSHEET_REFS}" (at 100.0305 48.895 0)
       (effects (font (size 1.27 1.27)) (justify left) hide)
     )
@@
     )
   )
-  (global_label "SD_CLOCK" (shape output) (at 86.36 43.815 0) (fields_autoplaced)
-    (effects (font (size 1.27 1.27)) (justify left))
-    (property "Intersheetrefs" "${INTERSHEET_REFS}" (at 98.8815 43.815 0)
+  (global_label "SD_CLOCK" (shape output) (at 86.36 36.195 0) (fields_autoplaced)
+    (effects (font (size 1.27 1.27)) (justify left))
+    (property "Intersheetrefs" "${INTERSHEET_REFS}" (at 98.8815 36.195 0)
       (effects (font (size 1.27 1.27)) (justify left) hide)
     )
@@
   (symbol (lib_id "Connector_Audio:AudioJack2_SwitchT") (at 50.165 114.935 180) (unit 1)
     (in_bom yes) (on_board yes) (dnp no)
-    (property "Reference" "J12" (at 55.88 113.665 0)
+    (property "Reference" "J2" (at 55.88 113.665 0)
       (effects (font (size 1.27 1.27)) (justify right))
     )
@@
   (symbol (lib_id "Connector_Audio:AudioJack2_SwitchT") (at 50.165 130.175 180) (unit 1)
     (in_bom yes) (on_board yes) (dnp no)
-    (property "Reference" "J12" (at 55.88 128.905 0)
+    (property "Reference" "J2" (at 55.88 128.905 0)
       (effects (font (size 1.27 1.27)) (justify right))
     )
@@
   (symbol (lib_id "Connector_Audio:AudioJack2_SwitchT") (at 100.965 99.695 180) (unit 1)
     (in_bom yes) (on_board yes) (dnp no)
-    (property "Reference" "J12" (at 106.68 98.425 0)
+    (property "Reference" "J2" (at 106.68 98.425 0)
       (effects (font (size 1.27 1.27)) (justify right))
     )
@@
   (symbol (lib_id "power:-12V") (at 86.36 66.675 270) (unit 1)
     (in_bom yes) (on_board yes) (dnp no) (fields_autoplaced)
-    (property "Reference" "#PWR078" (at 88.9 66.675 0)
+    (property "Reference" "#PWR014" (at 88.9 66.675 0)
       (effects (font (size 1.27 1.27)) hide)
     )
@@
   (symbol (lib_id "Connector_Audio:AudioJack2_SwitchT") (at 100.965 114.935 180) (unit 1)
     (in_bom yes) (on_board yes) (dnp no)
-    (property "Reference" "J12" (at 106.68 113.665 0)
+    (property "Reference" "J2" (at 106.68 113.665 0)
       (effects (font (size 1.27 1.27)) (justify right))
     )
@@
   (symbol (lib_id "Connector_Audio:AudioJack2_SwitchT") (at 100.965 84.455 180) (unit 1)
     (in_bom yes) (on_board yes) (dnp no)
-    (property "Reference" "J12" (at 106.68 83.185 0)
+    (property "Reference" "J2" (at 106.68 83.185 0)
       (effects (font (size 1.27 1.27)) (justify right))
     )
@@
   (symbol (lib_id "power:+12V") (at 49.53 59.055 270) (unit 1)
     (in_bom yes) (on_board yes) (dnp no) (fields_autoplaced)
-    (property "Reference" "#PWR077" (at 45.72 59.055 0)
+    (property "Reference" "#PWR07" (at 45.72 59.055 0)
       (effects (font (size 1.27 1.27)) hide)
     )
@@
   (symbol (lib_id "power:+12V") (at 140.335 161.925 270) (unit 1)
     (in_bom yes) (on_board yes) (dnp no) (fields_autoplaced)
-    (property "Reference" "#PWR077" (at 136.525 161.925 0)
+    (property "Reference" "#PWR056" (at 136.525 161.925 0)
       (effects (font (size 1.27 1.27)) hide)
     )
@@
   (symbol (lib_id "power:-12V") (at 140.335 169.545 270) (unit 1)
     (in_bom yes) (on_board yes) (dnp no) (fields_autoplaced)
-    (property "Reference" "#PWR078" (at 142.875 169.545 0)
+    (property "Reference" "#PWR059" (at 142.875 169.545 0)
       (effects (font (size 1.27 1.27)) hide)
     )
@@
   (symbol (lib_id "Connector_Audio:AudioJack2_SwitchT") (at 100.965 130.175 180) (unit 1)
     (in_bom yes) (on_board yes) (dnp no)
-    (property "Reference" "J12" (at 106.68 128.905 0)
+    (property "Reference" "J2" (at 106.68 128.905 0)
       (effects (font (size 1.27 1.27)) (justify right))
     )
@@
   (symbol (lib_id "power:+12V") (at 86.36 59.055 270) (unit 1)
     (in_bom yes) (on_board yes) (dnp no) (fields_autoplaced)
-    (property "Reference" "#PWR077" (at 82.55 59.055 0)
+    (property "Reference" "#PWR011" (at 82.55 59.055 0)
       (effects (font (size 1.27 1.27)) hide)
     )
@@
   (symbol (lib_id "Connector_Audio:AudioJack2_SwitchT") (at 50.165 84.455 180) (unit 1)
     (in_bom yes) (on_board yes) (dnp no)
-    (property "Reference" "J12" (at 55.88 83.185 0)
+    (property "Reference" "J2" (at 55.88 83.185 0)
       (effects (font (size 1.27 1.27)) (justify right))
     )
@@
   (symbol (lib_id "Connector_Audio:AudioJack2_SwitchT") (at 50.165 99.695 180) (unit 1)
     (in_bom yes) (on_board yes) (dnp no)
-    (property "Reference" "J12" (at 55.88 98.425 0)
+    (property "Reference" "J2" (at 55.88 98.425 0)
       (effects (font (size 1.27 1.27)) (justify right))
     )
@@
   (symbol (lib_id "power:-12V") (at 49.53 66.675 270) (unit 1)
     (in_bom yes) (on_board yes) (dnp no) (fields_autoplaced)
-    (property "Reference" "#PWR078" (at 52.07 66.675 0)
-      (effects (font (size 1.27 1.27)) hide)
-    )
+    (property "Reference" "#PWR010" (at 52.07 66.675 0)
+      (effects (font (size 1.27 1.27)) hide)
+    )

Commit message: top routing done
Connections:
- net +12V: no longer J1.15 (Pin_15), J7.15 (Pin_15)
- net -12V: no longer J1.18 (Pin_18)
- no-connect marks 13 -> 16
Changed lines of the file:
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@@
   )
   (no_connect (at 49.53 28.575))
+  (no_connect (at 49.53 66.675))
+  (no_connect (at 86.36 59.055))
+  (no_connect (at 49.53 59.055))
   (no_connect (at 95.885 81.915))
   (no_connect (at 45.085 127.635))
@@
         (path "/87a59a99-d509-467e-85da-26d34072acb7"
           (reference "H3") (unit 1)
-        )
-      )
-    )
-  )
-  (symbol (lib_id "power:+12V") (at 49.53 59.055 270) (unit 1)
-    (in_bom yes) (on_board yes) (dnp no) (fields_autoplaced)
-    (property "Reference" "#PWR07" (at 45.72 59.055 0)
-      (effects (font (size 1.27 1.27)) hide)
-    )
-    (property "Value" "+12V" (at 52.705 59.3718 90)
-      (effects (font (size 1.27 1.27)) (justify left))
-    )
-    (property "Footprint" "" (at 49.53 59.055 0)
-      (effects (font (size 1.27 1.27)) hide)
-    )
-    (property "Datasheet" "" (at 49.53 59.055 0)
-      (effects (font (size 1.27 1.27)) hide)
-    )
-    (pin "1")
-    (instances
-      (project "dk2_02_top"
-        (path "/87a59a99-d509-467e-85da-26d34072acb7"
-          (reference "#PWR07") (unit 1)
         )
       )
@@
     )
   )
-  (symbol (lib_id "power:+12V") (at 86.36 59.055 270) (unit 1)
-    (in_bom yes) (on_board yes) (dnp no) (fields_autoplaced)
-    (property "Reference" "#PWR011" (at 82.55 59.055 0)
-      (effects (font (size 1.27 1.27)) hide)
-    )
-    (property "Value" "+12V" (at 89.535 59.3718 90)
-      (effects (font (size 1.27 1.27)) (justify left))
-    )
-    (property "Footprint" "" (at 86.36 59.055 0)
-      (effects (font (size 1.27 1.27)) hide)
-    )
-    (property "Datasheet" "" (at 86.36 59.055 0)
-      (effects (font (size 1.27 1.27)) hide)
-    )
-    (pin "1")
-    (instances
-      (project "dk2_02_top"
-        (path "/87a59a99-d509-467e-85da-26d34072acb7"
-          (reference "#PWR011") (unit 1)
-        )
-      )
-    )
-  )
   (symbol (lib_id "power:GND") (at 49.53 64.135 90) (unit 1)
     (in_bom yes) (on_board yes) (dnp no) (fields_autoplaced)
@@
         )
       )
-    )
-  )
-  (symbol (lib_id "power:-12V") (at 49.53 66.675 270) (unit 1)
-    (in_bom yes) (on_board yes) (dnp no) (fields_autoplaced)
-    (property "Reference" "#PWR010" (at 52.07 66.675 0)
-      (effects (font (size 1.27 1.27)) hide)
-    )
-    (property "Value" "-12V" (at 52.705 66.9918 90)
-      (effects (font (size 1.27 1.27)) (justify left))
-    )
-    (property "Footprint" "" (at 49.53 66.675 0)
-      (effects (font (size 1.27 1.27)) hide)
-    )
-    (property "Datasheet" "" (at 49.53 66.675 0)
-      (effects (font (size 1.27 1.27)) hide)
-    )
-    (pin "1")
-    (instances
-      (project "dk2_02_top"
-        (path "/87a59a99-d509-467e-85da-26d34072acb7"
-          (reference "#PWR010") (unit 1)
-        )
-      )
