File: pcb/dk2_02_top/dk2_02_top.kicad_pcb (KiCad board)
At the start: 2 copper layers, 120 x 108 mm, 106 parts, among them J1 Conn_01x18_Pin, J10 Sync_Out, J11 Euro_Out_2, J12 CV_In_1, J13 CV_In_2, J14 CV_In_3, J15 CV_In_4, J2 Trigger_Out_1, J3 Trigger_Out_2, J4 Sync_In, J5 Euro_Out_1, J6 Micro_SD_Card, J7 Conn_01x18_Pin, J8 Trigger_Out_3, J9 Trigger_Out_4, SW1 SW_Push, SW10 SW_Push, SW11 SW_Push, SW12 SW_Push, SW13 SW_Push, SW14 SW_Push, SW15 SW_Push, SW16 SW_Push, SW17 SW_Push, SW18 SW_Push, SW2 SW_Push, SW3 SW_Push, SW4 SW_Push, SW5 SW_Push, SW6 SW_Push, SW7 SW_Push, SW8 SW_Push, SW9 SW_Push, U1 74HC595, U2 74HC595, U3 CA56-12EWA, U4 74HC165, U5 74HC165, U6 74HC4051, U7 MCP6002-xSN, U8 MCP6002-xSN, U9 74HC4051

Commit message: done for the week, started routing
Parts:
- moved R30 62.0 mm to (123.2, 119.0), turned to 0 degrees
- moved U6 57.1 mm to (150.5, 57.6)
- moved R36 47.6 mm to (123.2, 135.0), turned to 0 degrees
- moved R35 46.3 mm to (176.4, 122.2)
- moved R39 45.9 mm to (170.8, 117.0)
- moved R32 44.6 mm to (135.2, 119.0), turned to 0 degrees
- moved C3 42.0 mm to (170.8, 118.6)
- moved U9 41.4 mm to (170.5, 57.4)
- moved R37 38.1 mm to (176.4, 123.8)
- moved R40 37.3 mm to (171.9, 129.4)
- moved C4 35.8 mm to (171.9, 127.8)
- moved R29 29.9 mm to (176.3, 138.4)
- moved R33 29.6 mm to (170.7, 132.9)
- moved R38 29.2 mm to (135.2, 135.0), turned to 0 degrees
- moved R31 23.3 mm to (176.3, 140.0)
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Connections:
- J7 pad 10: SD_SERIAL_IN -> 595_DATA
- J7 pad 11: SD_SERIAL_OUT -> 595_CLOCK
- J7 pad 12: SD_CHIP_SELECT -> 595_LATCH
- J7 pad 6: 595_DATA -> SD_CLOCK
- J7 pad 7: 595_CLOCK -> SD_SERIAL_IN
- J7 pad 8: 595_LATCH -> SD_SERIAL_OUT
- J7 pad 9: SD_CLOCK -> SD_CHIP_SELECT
Routing:
- net Net-(U2-QF): track 0.00 -> 121.6 mm
- net Net-(U2-QG): track 0.00 -> 114.0 mm
- net Net-(U2-QH): track 0.00 -> 101.9 mm
- net Net-(U2-QE): track 0.00 -> 78.0 mm
- net Net-(U1-QB): track 0.00 -> 45.0 mm
- net Net-(U1-QC): track 0.00 -> 26.1 mm
- net Net-(U1-QA): track 0.00 -> 23.2 mm
- net Net-(U1-QD): track 0.00 -> 21.4 mm
- net Net-(U1-QF): track 0.00 -> 19.4 mm
- net Net-(U1-QE): track 0.00 -> 19.4 mm
- net Net-(U3-f): track 0.00 -> 2.97 mm
- net Net-(U3-b): track 0.00 -> 2.97 mm
- net Net-(U3-a): track 0.00 -> 2.97 mm
- net Net-(D3-A): track 0.00 -> 2.92 mm
- net Net-(D1-A): track 0.00 -> 2.80 mm
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- added copper zone on F.Cu, net GND

Commit message: routing again
Parts:
- moved RV10 3.00 mm to (175.0, 53.0)
- moved RV12 3.00 mm to (175.0, 73.0)
- moved RV1 2.00 mm to (80.0, 53.0)
- moved RV11 2.00 mm to (156.0, 73.0)
- moved RV5 2.00 mm to (80.0, 73.0)
- moved RV9 2.00 mm to (156.0, 53.0)
- moved U9 2.00 mm to (168.5, 57.4)
- moved RV2 1.00 mm to (99.0, 53.0)
- moved RV4 1.00 mm to (137.0, 53.0)
- moved RV6 1.00 mm to (99.0, 73.0)
- moved U6 1.00 mm to (149.5, 57.6)
- moved RV8 0.60 mm to (137.0, 73.0)
Routing:
- net CV_IN_2: track 0.00 -> 118.9 mm, vias 0 -> 2
- net CV_IN_4: track 0.00 -> 117.0 mm, vias 0 -> 2
- net CV_IN_3: track 0.00 -> 113.2 mm
- net Net-(U6-A4): track 0.00 -> 98.2 mm
- net Net-(U8A--): track 0.00 -> 97.7 mm, vias 0 -> 2
- net +3.3V: track 0.00 -> 96.1 mm
- net EURO_OUT_1: track 0.00 -> 93.5 mm
- net Net-(U5-D7): track 2.56 -> 91.5 mm
- net EURO_OUT_2: track 0.00 -> 85.5 mm
- net Net-(U7A--): track 0.00 -> 84.2 mm
- net Net-(U5-D6): track 2.56 -> 84.8 mm
- net Net-(U8B--): track 0.00 -> 74.5 mm, vias 0 -> 2
- net Net-(U5-D5): track 2.56 -> 74.9 mm
- net Net-(U6-A0): track 0.00 -> 71.0 mm
- net 595_LATCH: track 0.00 -> 67.0 mm, vias 0 -> 2
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
Commit message: nearly routed
Routing:
- net +3.3V: track 96.1 -> 565.7 mm, vias 0 -> 6
- net GND: track 0.00 -> 201.7 mm, vias 0 -> 11
- net CV_IN_1: track 3.89 -> 104.7 mm, vias 0 -> 2
- net 4051_READING_0: track 0.00 -> 73.9 mm, vias 0 -> 1
- net Net-(U5-D3): track 0.00 -> 60.7 mm, vias 0 -> 1
- net Net-(U6-A5): track 0.00 -> 60.1 mm, vias 0 -> 2
- net Net-(U4-D7): track 0.00 -> 55.3 mm
- net Net-(U4-D3): track 0.00 -> 54.8 mm, vias 0 -> 2
- net 4051_ADDRESS_B: track 0.00 -> 54.1 mm
- net 4051_ADDRESS_A: track 0.00 -> 54.0 mm
- net 4051_ADDRESS_C: track 0.00 -> 53.4 mm
- net Net-(U5-D2): track 0.00 -> 50.6 mm, vias 0 -> 3
- net Net-(U4-D6): track 0.00 -> 47.6 mm
- net Net-(U6-A6): track 0.00 -> 45.4 mm, vias 0 -> 2
- net Net-(U4-D2): track 0.00 -> 44.9 mm, vias 0 -> 1
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
Commit message: top routing done
Connections:
- J1 pad 15: +12V -> unconnected-(J1-Pin_15-Pad15)
- J1 pad 18: -12V -> unconnected-(J1-Pin_18-Pad18)
- J7 pad 15: +12V -> unconnected-(J7-Pin_15-Pad15)
Routing:
- net +3.3V: track 565.7 -> 586.9 mm, vias 6 -> 8
- net TAP_TEMPO_BUTTON: track 20.9 -> 37.6 mm
- net START_STOP_BUTTON: track 7.89 -> 20.4 mm
- net GND: track 201.7 -> 213.7 mm, vias 11 -> 13
- net Net-(U5-D3): track 60.7 -> 63.3 mm
- net 595_CLOCK: track 60.7 -> 63.0 mm
- net Net-(U1-QH'): track 7.13 -> 9.44 mm
- net CV_IN_3: track 114.6 -> 116.1 mm
- net EURO_OUT_1: track 93.5 -> 94.2 mm
- net EURO_OUT_2: track 85.5 -> 86.1 mm
- net Net-(U9-A2): track 23.7 -> 23.0 mm

Commit message: ready for jlcpcb
Other:
- board text added: "Drumkid 2.02 (Eurorack)"
Changed lines of the file:
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@@
   (gr_rect (start 70 40) (end 190 148)
     (stroke (width 0.1) (type default)) (fill none) (layer "Edge.Cuts"))
+  (gr_text "Drumkid 2.02 (Eurorack)" (at 84 59) (layer "F.SilkS")
+    (effects (font (size 3 3) (thickness 0.15)) (justify left bottom))
+  )
   (segment (start 176.175 139.125) (end 175.45 138.4) (width 0.25) (layer "B.Cu") (net 1))
   (segment (start 176.175 143.325) (end 176.175 139.125) (width 0.25) (layer "B.Cu") (net 1))
