File: pcb/dk2_03_top/dac.kicad_sch (KiCad schematic)
At the start: 34 parts, among them U3 TL072, U4 PCM5102

Commit message: getting ready for next PCBs
Parts:
- added C5, C8: 1uF, Capacitor_SMD:C_0603_1608Metric, symbol Device:C
- added J15: Euro_Out_1, AudioJacks:Jack_3.5mm_QingPu_WQP-PJ398SM_Vertical, symbol Connector_Audio:AudioJack2_SwitchT
- added J15: Euro_Out_2, AudioJacks:Jack_3.5mm_QingPu_WQP-PJ398SM_Vertical, symbol Connector_Audio:AudioJack2_SwitchT
- added U11: AP7333-33SRG, Package_TO_SOT_SMD:SOT-23, symbol Regulator_Linear:SPX2920M3-3.3_SOT223
- renumbered C6 to C10, C7 to C11, C8 to C12, C9 to C13, C10 to C14, C11 to C15, C12 to C16, C13 to C17, C14 to C18, C15 to C19, C16 to C20, C17 to C21, C18 to C22, C19 to C23, C20 to C24, C21 to C25, C2 to C6, C3 to C7, C5 to C9, R1 to R41, R2 to R42, R3 to R43, R4 to R44, R5 to R45, R6 to R46, R7 to R47, R8 to R48, R9 to R49, R10 to R50, R11 to R51, R12 to R52, R13 to R53, U3 to U12, U4 to U13
Connections:
- net +3.3VDAC: now also C8.1, U11.2 (VO)
- net GND: now also C5.2, C8.2, J15.S, J15.S, U11.3 (GND)
- net EURO_OUT_1: no longer names the net of R47.2
- net EURO_OUT_1: now also J15.T
- net EURO_OUT_2: no longer names the net of R48.2
- net EURO_OUT_2: now also J15.T
- new net +5V: C5.1, U11.1 (VI)
- no-connect marks 0 -> 2
Other:
- note added: "Voltage regulator for DAC, provides low-noise signal. AP7333-33SRG, as used by Pimoroni. Cheap and available on JLCPCB. Possible alternative is MIC5219-3.3YM5."
