File: pcb/dk2_03_top/europower.kicad_sch (KiCad schematic)
At the start: 11 parts, among them J3 Eurorack_Power, U2 AP7333-33SAG, U8 XL1509-5.0

Commit message: getting ready for next PCBs
Parts:
- removed C1, C4: 1uF, Capacitor_SMD:C_0603_1608Metric, symbol Device:C
- removed U2: AP7333-33SAG, Package_TO_SOT_SMD:SOT-23, symbol Regulator_Linear:SPX2920M3-3.3_SOT223
- added C26: 0.33uF, symbol Device:C
- added C27: 0.1uF, symbol Device:C
- added J16: Barrel_Jack_Switch, symbol Connector:Barrel_Jack_Switch
- added U13: L7805, symbol Regulator_Linear:L7805
- C24: renamed from C25; footprint Capacitor_THT:CP_Radial_D10.0mm_P5.00mm -> (none)
- C25: renamed from C26; footprint Capacitor_SMD:C_0603_1608Metric -> (none)
- C28: renamed from C27; footprint Capacitor_THT:CP_Radial_D8.0mm_P3.50mm -> (none)
- J15: renamed from J3; value Eurorack_Power -> Conn_02x05_Odd_Even; footprint Connector_IDC:IDC-Header_2x05_P2.54mm_Vertical -> (none)
- JP1: footprint Connector_PinHeader_2.54mm:PinHeader_1x03_P2.54mm_Vertical -> (none)
- L1: footprint Inductor_THT:L_Radial_D7.0mm_P3.00mm -> (none)
- renumbered D2 to D10, U8 to U12
Connections:
- net +3.3VDAC is gone; now on net +5V: JP1.2 (C)
- net +12V: now also C26.1, J16.2, U13.1 (IN)
- net +5V: no longer C28.1, L1.2, U12.3 (FB)
- net GND: now also C26.2, C27.2, J16.1, U13.2 (GND)
- net 5V_LDO: now reaches JP1.1 (A)
- net 5V_LDO: now also C27.1, U13.3 (OUT)
- net +3.3V renamed 5V_BUCK
- net 5V_BUCK: now also C28.1, L1.2, U12.3 (FB)
- no-connect marks 0 -> 1
Other:
- note removed: "5V source for Pico"
- note removed: "Jumper allows choice of "clean" or "dirty" 3.3V power to the DAC."
- note removed: "Voltage regulator for DAC, provides low-noise signal. AP7333-33SRG used by Pimoroni but I'm using AP7333-33SAG. Cheap and available on JLCPCB. Possible alternative is MIC5219-3.3YM5."
- moved on the sheet: C24, C25, C28, D10, J15, L1, U12
