File: pcb/dk2_03_top/power.kicad_sch (KiCad schematic)
At the start: 11 parts, among them J3 Eurorack_Power, U2 AP7333-33SAG, U8 XL1509-5.0

Commit message: getting ready for next PCBs
Parts:
- removed C1, C4: 1uF, Capacitor_SMD:C_0603_1608Metric, symbol Device:C
- removed JP1: Jumper_3_Open, Connector_PinHeader_2.54mm:PinHeader_1x03_P2.54mm_Vertical, symbol Jumper:Jumper_3_Open
- removed U2: AP7333-33SAG, Package_TO_SOT_SMD:SOT-23, symbol Regulator_Linear:SPX2920M3-3.3_SOT223
- renumbered C25 to C29, C26 to C30, C27 to C31, D2 to D6, J3 to J14, U8 to U17
Other:
- note removed: "Jumper allows choice of "clean" or "dirty" 3.3V power to the DAC."
- note removed: "Voltage regulator for DAC, provides low-noise signal. AP7333-33SRG used by Pimoroni but I'm using AP7333-33SAG. Cheap and available on JLCPCB. Possible alternative is MIC5219-3.3YM5."
- moved on the sheet: J14
