File: pcb/dk2_03_top/shiftreginx.kicad_sch (KiCad schematic)
At the start: 8 parts, among them J1 Conn_01x05_Pin, SW3 SW_Push, SW4 SW_Push, SW5 SW_Push, U4 74HC165

Commit message: routing top pcb
Parts:
- renumbered J1 to J16
Changed lines of the file:
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@@
         )
         (path "/87a59a99-d509-467e-85da-26d34072acb7/1a91e583-926b-4126-a95f-efd256f8eb1b"
-          (reference "SW2") (unit 1)
+          (reference "SW18") (unit 1)
         )
       )
@@
         )
         (path "/87a59a99-d509-467e-85da-26d34072acb7/1a91e583-926b-4126-a95f-efd256f8eb1b"
-          (reference "#PWR07") (unit 1)
+          (reference "#PWR061") (unit 1)
         )
       )
@@
         )
         (path "/87a59a99-d509-467e-85da-26d34072acb7/1a91e583-926b-4126-a95f-efd256f8eb1b"
-          (reference "#PWR010") (unit 1)
+          (reference "#PWR062") (unit 1)
         )
       )
@@
         )
         (path "/87a59a99-d509-467e-85da-26d34072acb7/1a91e583-926b-4126-a95f-efd256f8eb1b"
-          (reference "#PWR011") (unit 1)
+          (reference "#PWR063") (unit 1)
         )
       )
@@
   (symbol (lib_id "Connector:Conn_01x05_Pin") (at 149.86 73.66 0) (unit 1)
     (in_bom yes) (on_board yes) (dnp no)
-    (property "Reference" "J1" (at 140.97 73.025 0)
+    (property "Reference" "J16" (at 140.97 73.025 0)
       (effects (font (size 1.27 1.27)))
     )
@@
       (project "dk2_03_top"
         (path "/87a59a99-d509-467e-85da-26d34072acb7/1a91e583-926b-4126-a95f-efd256f8eb1b"
-          (reference "J1") (unit 1)
+          (reference "J16") (unit 1)
         )
       )
@@
         )
         (path "/87a59a99-d509-467e-85da-26d34072acb7/1a91e583-926b-4126-a95f-efd256f8eb1b"
-          (reference "#PWR020") (unit 1)
+          (reference "#PWR064") (unit 1)
         )
       )
@@
         )
         (path "/87a59a99-d509-467e-85da-26d34072acb7/1a91e583-926b-4126-a95f-efd256f8eb1b"
-          (reference "SW1") (unit 1)
-        )
-      )
+          (reference "SW17") (unit 1)
+        )
+      )
