File: pcb/dk2_03_top/dk2_03_top.kicad_sch (KiCad schematic)
At the start: 17 parts, among them J1 Conn_01x18_Pin, J2 Euro_Out_1, J2 Euro_Out_2, J2 Sync_In, J2 Sync_Out, J2 Trigger_Out_1, J2 Trigger_Out_2, J2 Trigger_Out_3, J2 Trigger_Out_4, J6 Micro_SD_Card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

Commit message: pcb progress
Parts:
- removed J1, J7: Conn_01x18_Pin, Connector_PinHeader_2.54mm:PinHeader_1x18_P2.54mm_Vertical, symbol Connector:Conn_01x18_Pin
- removed SW2 (x2): SW_Push, Button_Switch_THT:SW_PUSH-12mm, symbol Switch:SW_Push
- added J1: Conn_01x20_Pin, symbol Connector:Conn_01x20_Pin
- added J7: Conn_01x16_Pin, symbol Connector:Conn_01x16_Pin
Connections:
- net +12V: now also J1.16 (Pin_16), J7.12 (Pin_12)
- net +3.3V: now also J1.18 (Pin_18), J7.14 (Pin_14)
- net -12V: now also J1.20 (Pin_20), J7.16 (Pin_16)
- net 165_CLOCK: now also J1.8 (Pin_8)
- net 165_DATA: now also J1.9 (Pin_9)
- net 165_LOAD: now also J1.7 (Pin_7)
- net 4051_ADDRESS_A: now also J1.2 (Pin_2)
- net 4051_ADDRESS_B: now also J1.3 (Pin_3)
- net 4051_ADDRESS_C: now also J1.4 (Pin_4)
- net 4051_READING_0: now also J1.6 (Pin_6)
- net 4051_READING_1: now also J1.5 (Pin_5)
- net 595_CLOCK: now also J7.8 (Pin_8)
- net 595_DATA: now also J7.7 (Pin_7)
- net 595_LATCH: now also J7.9 (Pin_9)
- net EURO_OUT_1: now also J7.10 (Pin_10)
- net EURO_OUT_2: now also J7.11 (Pin_11)
- net GND: now also J1.19 (Pin_19), J7.15 (Pin_15)
- net SD_CHIP_SELECT: now also J7.6 (Pin_6)
- net SD_CLOCK: now also J7.3 (Pin_3)
- net SD_SERIAL_IN: now also J7.4 (Pin_4)
- net SD_SERIAL_OUT: now also J7.5 (Pin_5)
- net SYNC_IN_EURO: now also J1.14 (Pin_14)
- net SYNC_OUT_EURO: now also J1.15 (Pin_15)
- net TRIGGER_OUT_1_EURO: now also J1.10 (Pin_10)
- net TRIGGER_OUT_2_EURO: now also J1.11 (Pin_11)
- net TRIGGER_OUT_3_EURO: now also J1.12 (Pin_12)
- net TRIGGER_OUT_4_EURO: now also J1.13 (Pin_13)
- new net +3.3VDAC: J1.17 (Pin_17), J7.13 (Pin_13)
- no-connect marks 16 -> 13
Other:
- added sheet Shift register in 3 (shiftregin.kicad_sch)
- moved on the sheet: H1, H2, H3, H4

Commit message: bottom pcb shrunk
Parts:
- removed J1: Conn_01x20_Pin, symbol Connector:Conn_01x20_Pin
- removed J7: Conn_01x16_Pin, symbol Connector:Conn_01x16_Pin
- added J16: Conn_01x20_Socket, symbol Connector:Conn_01x20_Socket
- added J18: Conn_01x16_Socket, symbol Connector:Conn_01x16_Socket
Connections:
- net +12V: now also J16.16 (Pin_16), J18.12 (Pin_12)
- net +3.3V: now also J16.18 (Pin_18), J18.14 (Pin_14)
- net +3.3VDAC: now also J16.17 (Pin_17), J18.13 (Pin_13)
- net -12V: now also J16.20 (Pin_20), J18.16 (Pin_16)
- net 165_CLOCK: now also J16.8 (Pin_8)
- net 165_DATA: now also J16.9 (Pin_9)
- net 165_LOAD: now also J16.7 (Pin_7)
- net 4051_ADDRESS_A: now also J16.2 (Pin_2)
- net 4051_ADDRESS_B: now also J16.3 (Pin_3)
- net 4051_ADDRESS_C: now also J16.4 (Pin_4)
- net 4051_READING_0: now also J16.6 (Pin_6)
- net 4051_READING_1: now also J16.5 (Pin_5)
- net 595_CLOCK: now also J18.8 (Pin_8)
- net 595_DATA: now also J18.7 (Pin_7)
- net 595_LATCH: now also J18.9 (Pin_9)
- net EURO_OUT_1: now also J18.10 (Pin_10)
- net EURO_OUT_2: now also J18.11 (Pin_11)
- net GND: now also J16.19 (Pin_19), J18.15 (Pin_15)
- net SD_CHIP_SELECT: now also J18.6 (Pin_6)
- net SD_CLOCK: now also J18.3 (Pin_3)
- net SD_SERIAL_IN: now also J18.4 (Pin_4)
- net SD_SERIAL_OUT: now also J18.5 (Pin_5)
- net SYNC_IN_EURO: now also J16.14 (Pin_14)
- net SYNC_OUT_EURO: now also J16.15 (Pin_15)
- net TRIGGER_OUT_1_EURO: now also J16.10 (Pin_10)
- net TRIGGER_OUT_2_EURO: now also J16.11 (Pin_11)
- net TRIGGER_OUT_3_EURO: now also J16.12 (Pin_12)
- net TRIGGER_OUT_4_EURO: now also J16.13 (Pin_13)

Commit message: a commit before i mess up all the buttons
Parts:
- J16: footprint (none) -> Connector_PinSocket_2.54mm:PinSocket_1x20_P2.54mm_Vertical
- J18: footprint (none) -> Connector_PinSocket_2.54mm:PinSocket_1x16_P2.54mm_Vertical
Other:
- sheet Shift register in 3: file shiftregin.kicad_sch -> shiftreginx.kicad_sch
- moved on the sheet: J2, J6

Commit message: routing top pcb
Parts:
- renumbered J16 to J1, J18 to J7

Commit message: top pcb routed
Connections:
- net +12V: no longer J1.16 (Pin_16)
- net +3.3VDAC: no longer J1.17 (Pin_17), J7.13 (Pin_13)
- net -12V: no longer J1.20 (Pin_20)
- no-connect marks 13 -> 17
Changed lines of the file:
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@@
   (no_connect (at 50.8 19.05))
   (no_connect (at 96.52 82.55))
+  (no_connect (at 50.8 57.15))
   (no_connect (at 45.72 128.27))
   (no_connect (at 96.52 97.79))
   (no_connect (at 96.52 128.27))
   (no_connect (at 87.63 31.75))
+  (no_connect (at 50.8 59.69))
+  (no_connect (at 87.63 59.69))
   (no_connect (at 50.8 173.99))
   (no_connect (at 50.8 156.21))
@@
   (no_connect (at 45.72 97.79))
   (no_connect (at 45.72 113.03))
+  (no_connect (at 50.8 67.31))
   (wire (pts (xy 152.4 88.9) (xy 154.94 88.9))
     (stroke (width 0) (type default))
@@
         (path "/87a59a99-d509-467e-85da-26d34072acb7"
           (reference "J9") (unit 1)
-        )
-      )
-    )
-  )
-  (symbol (lib_id "power:+3.3VDAC") (at 50.8 59.69 270) (unit 1)
-    (in_bom yes) (on_board yes) (dnp no)
-    (property "Reference" "#PWR08" (at 49.53 63.5 0)
-      (effects (font (size 1.27 1.27)) hide)
-    )
-    (property "Value" "+3.3VDAC" (at 58.42 59.69 90)
-      (effects (font (size 1.27 1.27)))
-    )
-    (property "Footprint" "" (at 50.8 59.69 0)
-      (effects (font (size 1.27 1.27)) hide)
-    )
-    (property "Datasheet" "" (at 50.8 59.69 0)
-      (effects (font (size 1.27 1.27)) hide)
-    )
-    (pin "1")
-    (instances
-      (project "dk2_03_top"
-        (path "/87a59a99-d509-467e-85da-26d34072acb7"
-          (reference "#PWR08") (unit 1)
         )
       )
@@
     )
   )
-  (symbol (lib_id "power:+12V") (at 50.8 57.15 270) (unit 1)
-    (in_bom yes) (on_board yes) (dnp no) (fields_autoplaced)
-    (property "Reference" "#PWR07" (at 46.99 57.15 0)
-      (effects (font (size 1.27 1.27)) hide)
-    )
-    (property "Value" "+12V" (at 53.975 57.4668 90)
-      (effects (font (size 1.27 1.27)) (justify left))
-    )
-    (property "Footprint" "" (at 50.8 57.15 0)
-      (effects (font (size 1.27 1.27)) hide)
-    )
-    (property "Datasheet" "" (at 50.8 57.15 0)
-      (effects (font (size 1.27 1.27)) hide)
-    )
-    (pin "1")
-    (instances
-      (project "dk2_03_top"
-        (path "/87a59a99-d509-467e-85da-26d34072acb7"
-          (reference "#PWR07") (unit 1)
-        )
-      )
-    )
-  )
-  (symbol (lib_id "power:-12V") (at 50.8 67.31 270) (unit 1)
-    (in_bom yes) (on_board yes) (dnp no) (fields_autoplaced)
-    (property "Reference" "#PWR011" (at 53.34 67.31 0)
-      (effects (font (size 1.27 1.27)) hide)
-    )
-    (property "Value" "-12V" (at 53.975 67.6268 90)
-      (effects (font (size 1.27 1.27)) (justify left))
-    )
-    (property "Footprint" "" (at 50.8 67.31 0)
-      (effects (font (size 1.27 1.27)) hide)
-    )
-    (property "Datasheet" "" (at 50.8 67.31 0)
-      (effects (font (size 1.27 1.27)) hide)
-    )
-    (pin "1")
-    (instances
-      (project "dk2_03_top"
-        (path "/87a59a99-d509-467e-85da-26d34072acb7"
-          (reference "#PWR011") (unit 1)
-        )
-      )
-    )
-  )
   (symbol (lib_id "power:GND") (at 45.72 133.35 0) (unit 1)
     (in_bom yes) (on_board yes) (dnp no) (fields_autoplaced)
@@
         )
       )
-    )
-  )
-  (symbol (lib_id "power:+3.3VDAC") (at 87.63 59.69 270) (unit 1)
-    (in_bom yes) (on_board yes) (dnp no)
-    (property "Reference" "#PWR013" (at 86.36 63.5 0)
-      (effects (font (size 1.27 1.27)) hide)
-    )
-    (property "Value" "+3.3VDAC" (at 95.25 59.69 90)
-      (effects (font (size 1.27 1.27)))
-    )
-    (property "Footprint" "" (at 87.63 59.69 0)
-      (effects (font (size 1.27 1.27)) hide)
-    )
-    (property "Datasheet" "" (at 87.63 59.69 0)
-      (effects (font (size 1.27 1.27)) hide)
-    )
-    (pin "1")
-    (instances
-      (project "dk2_03_top"
-        (path "/87a59a99-d509-467e-85da-26d34072acb7"
-          (reference "#PWR013") (unit 1)
-        )
-      )
