File: pcb/dk2_03_bottom/dac.kicad_sch (KiCad schematic)
At the start: 34 parts, among them U3 TL072, U4 PCM5102

Commit message: a commit before i mess up all the buttons
Other:
- moved on the sheet: C10, C11, C14, C16, C18, C2, C20, C5, C6, C7, C9, R1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
