File: pcb/dk2_03_bottom/digital-in-out.kicad_sch (KiCad schematic)
At the start: 24 parts, among them Q2 MMBT3904, U5 TL072, U6 TL072, U7 TL072

Commit message: a commit before i mess up all the buttons
Other:
- moved on the sheet: C5, R42, R45, R46, R49, R50, R53, U5C, U6A, U6B, U6C, U7B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
