File: pcb/dk2_03_bottom/power.kicad_sch (KiCad schematic)
At the start: 11 parts, among them J3 Eurorack_Power, U2 AP7333-33SAG, U8 XL1509-5.0

Commit message: pcb progress
Changed lines of the file:
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@@
-    (effects (font (size 1.27 1.27)) (justify left top))
-  )
-  (text_box "Warning! Default Kicad pin mapping for this component is wrong! Pins 2 and 3 were swapped, causing magic smoke release on previous board."
-    (at 69.215 71.12 0) (size 33.02 13.97)
-    (stroke (width 0) (type default))
-    (fill (type none))
-    (effects (font (size 1.27 1.27)) (justify left top))
-  )
-  (text_box "Yet another note! Might be good to power the pots/ADC ref(?) via this supply if I can actually get the pins right..."
-    (at 137.795 71.12 0) (size 27.94 13.97)
-    (stroke (width 0) (type default))
-    (fill (type none))
-    (effects (font (size 1.27 1.27)) (justify left top))
-  )
-  (text_box "Another warning! JLCPCB lists this as SOT-23, but it's actually SOT-23R, which has a different pinout!!"
-    (at 103.505 71.12 0) (size 33.02 13.97)
-    (stroke (width 0) (type default))
-    (fill (type none))
     (effects (font (size 1.27 1.27)) (justify left top))
   )

Commit message: a commit before i mess up all the buttons
Other:
- moved on the sheet: C1, C27, C4, D2, J3, JP1, L1, U2
