File: pcb/dk2_03_panel/dk2_03_panel.kicad_pcb (KiCad board)
At the start: 2 copper layers, 121.9 x 128.5 mm, 55 parts

Commit message: fixed an issue where i forgot to rotate the pots on the pcb
Parts:
- H15: value Sync out -> Clk out
- H21, H22, H23, H24, H25, H26, H27, H28, H29, H30, H31, H32, H33, H34, H35, H36: footprint Panel:MountingHole_4.3mm_M4 -> Panel:Button_Hole
- H37: renamed from H53; footprint Panel:MountingHole_4.3mm_M4 -> Panel:Button_Hole
- H38: renamed from H54; footprint Panel:MountingHole_4.3mm_M4 -> Panel:Button_Hole
- H39: renamed from H55; footprint Panel:MountingHole_4.3mm_M4 -> Panel:Button_Hole
- H40: renamed from H37; footprint Panel:MountingHole_6.4mm_M6 -> Panel:Pot_Hole
- H41: renamed from H38; footprint Panel:MountingHole_6.4mm_M6 -> Panel:Pot_Hole
- H42: renamed from H39; footprint Panel:MountingHole_6.4mm_M6 -> Panel:Pot_Hole
- H43: renamed from H40; footprint Panel:MountingHole_6.4mm_M6 -> Panel:Pot_Hole
- H44: renamed from H41; footprint Panel:MountingHole_6.4mm_M6 -> Panel:Pot_Hole
- H45: renamed from H42; footprint Panel:MountingHole_6.4mm_M6 -> Panel:Pot_Hole
- H46: renamed from H43; footprint Panel:MountingHole_6.4mm_M6 -> Panel:Pot_Hole
- H47: renamed from H44; footprint Panel:MountingHole_6.4mm_M6 -> Panel:Pot_Hole
- H48: renamed from H45; footprint Panel:MountingHole_6.4mm_M6 -> Panel:Pot_Hole
- H49: renamed from H46; footprint Panel:MountingHole_6.4mm_M6 -> Panel:Pot_Hole
- H50: renamed from H47; footprint Panel:MountingHole_6.4mm_M6 -> Panel:Pot_Hole
- H51: renamed from H48; footprint Panel:MountingHole_6.4mm_M6 -> Panel:Pot_Hole
- H52: renamed from H49; value LED -> Error; footprint Panel:MountingHole_3.2mm_M3 -> Panel:LED_Hole
- H53: renamed from H50; value LED -> Pulse; footprint Panel:MountingHole_3.2mm_M3 -> Panel:LED_Hole
- H54: renamed from H51; value LED -> Clock in; footprint Panel:MountingHole_3.2mm_M3 -> Panel:LED_Hole
- H55: renamed from H52; value LED -> Clock out; footprint Panel:MountingHole_3.2mm_M3 -> Panel:LED_Hole
- H9: value Sync in -> Clk in
- moved H39 85.0 mm to (125.2, 99.2)
- moved H38 76.0 mm to (115.2, 99.2)
- moved H37 69.3 mm to (105.2, 99.2)
- moved H33 35.0 mm to (60.2, 99.2)
- moved H34 35.0 mm to (70.2, 99.2)
- moved H35 35.0 mm to (80.2, 99.2)
- moved H25 32.3 mm to (80.2, 75.2)
- moved H31 30.0 mm to (40.2, 99.2)
- moved H32 30.0 mm to (50.2, 99.2)
- moved H36 30.0 mm to (95.2, 99.2)
- moved H29 23.3 mm to (70.2, 87.2)
- moved H30 23.3 mm to (80.2, 87.2)
- moved H26 20.0 mm to (40.2, 87.2)
- moved H27 20.0 mm to (50.2, 87.2)
- moved H28 20.0 mm to (60.2, 87.2)
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
Commit message: panel nearly done
Parts:
- H15: value Clk out -> Clock
- H21: value SmallButton -> Play
- H22: value SmallButton -> Tap
- H23: value SmallButton -> Live
- H24: value SmallButton -> Step
- H25: value SmallButton -> X
- H26: value SmallButton -> Save
- H27: value SmallButton -> Beat
- H28: value SmallButton -> Tempo
- H29: value SmallButton -> Tuplet
- H30: value SmallButton -> Y
- H31: value SmallButton -> Menu
- H32: value SmallButton -> Kit
- H33: value SmallButton -> T sig
- H34: value SmallButton -> Clear
- H35: value SmallButton -> Back
- H36: value SmallButton -> +
- H37: value SmallButton -> -
- H38: value SmallButton -> Yes
- H39: value SmallButton -> No
- H40: value Pot -> Chance
- H41: value Pot -> Zoom
- H42: value Pot -> Cluster
- H43: value Pot -> Crop
- H44: value Pot -> Crush
- H45: value Pot -> Pitch
- H46: value Pot -> Vel
- H47: value Pot -> Vel range
- H48: value Pot -> Magnet
- H49: value Pot -> Swing
- H50: value Pot -> Drop rand
- H51: value Pot -> Drop all
- H9: value Clk in -> Clock

Commit message: panel very nearly done
Parts:
- H10, H11, H14, H15, H16, H17, H20: footprint Panel:Jack_Hole -> Panel:Output_Jack_Hole
- H12, H13, H18, H19, H9: footprint Panel:Jack_Hole -> Panel:Input_Jack_Hole

Commit message: panel finished!
Parts:
- H13: value Velo -> Vel
- H25: value X -> A
- H30: value Y -> B
- H33: value T sig -> T.sig
- H39: value No -> X
