File: pcb/dk2_04_top/shiftreginx.kicad_sch (KiCad schematic)
At the start: 10 parts, among them J16 Conn_01x05_Pin, SW3 SW_Push, SW4 SW_Push, SW5 SW_Push, U4 74HC165

Commit message: pcb 2.04 tweaks
Parts:
- removed J16: Conn_01x05_Pin, Connector_PinHeader_2.54mm:PinHeader_1x05_P2.54mm_Vertical, symbol Connector:Conn_01x05_Pin
- added J16: Conn_01x04_Pin, symbol Connector:Conn_01x04_Pin
- R13: value 10k -> 330k
- R14: value 10k -> 100k
Connections:
- net +12V: now also R13.2
- net GND: now also R14.1
- net 12V DETECTION: now reaches U4.14 (D3)
- net 12V DETECTION: now also R13.1, R14.2
- net at U4.3 (D4): now also J16.1 (Pin_1)
- net at U4.4 (D5): now also J16.2 (Pin_2)
- net at U4.5 (D6): now also J16.3 (Pin_3)
- net at U4.6 (D7): now also J16.4 (Pin_4)
Other:
- moved on the sheet: R13, R14
Changed lines of the file:
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@@
   (junction (at 107.95 58.42) (diameter 0) (color 0 0 0 0)
+  )
+  (junction (at 59.69 63.5) (diameter 0) (color 0 0 0 0)
   )
   (junction (at 118.11 81.28) (diameter 0) (color 0 0 0 0)
@@
     (stroke (width 0) (type default))
   )
+  (wire (pts (xy 59.69 63.5) (xy 62.23 63.5))
+    (stroke (width 0) (type default))
+  )
   (wire (pts (xy 107.95 69.85) (xy 107.95 81.28))
     (stroke (width 0) (type default))
@@
     (stroke (width 0) (type default))
   )
+  (wire (pts (xy 59.69 63.5) (xy 59.69 64.77))
+    (stroke (width 0) (type default))
+  )
   (wire (pts (xy 118.11 58.42) (xy 118.11 60.96))
     (stroke (width 0) (type default))
@@
     (stroke (width 0) (type default))
   )
+  (wire (pts (xy 59.69 62.23) (xy 59.69 63.5))
+    (stroke (width 0) (type default))
+  )
   (wire (pts (xy 118.11 83.82) (xy 118.11 81.28))
     (stroke (width 0) (type default))
@@
     (stroke (width 0) (type default))
   )
-  (text_box "Voltage divider from 12V rail down to 3V to detect power off"
-    (at 33.02 88.9 0) (size 38.1 22.86)
+  (text_box "Voltage divider from 12V rail down to ~2.8V to detect power off"
+    (at 41.91 40.64 0) (size 38.1 7.62)
     (stroke (width 0) (type default))
     (fill (type none))
     (effects (font (size 1.27 1.27)) (justify left top))
+  )
+  (global_label "12V DETECTION" (shape input) (at 62.23 63.5 0) (fields_autoplaced)
+    (effects (font (size 1.27 1.27)) (justify left))
+    (property "Intersheetrefs" "${INTERSHEET_REFS}" (at 79.65 63.5 0)
+      (effects (font (size 1.27 1.27)) (justify left) hide)
+    )
   )
   (global_label "165_CLOCK" (shape input) (at 154.94 88.9 180) (fields_autoplaced)
     (effects (font (size 1.27 1.27)) (justify right))
     (property "Intersheetrefs" "${INTERSHEET_REFS}" (at 141.2695 88.9 0)
+      (effects (font (size 1.27 1.27)) (justify right) hide)
+    )
+  )
+  (global_label "12V DETECTION" (shape input) (at 154.94 68.58 180) (fields_autoplaced)
+    (effects (font (size 1.27 1.27)) (justify right))
+    (property "Intersheetrefs" "${INTERSHEET_REFS}" (at 137.52 68.58 0)
       (effects (font (size 1.27 1.27)) (justify right) hide)
     )
@@
     )
   )
+  (symbol (lib_id "Connector:Conn_01x04_Pin") (at 149.86 73.66 0) (unit 1)
+    (in_bom yes) (on_board yes) (dnp no)
+    (property "Reference" "J16" (at 142.24 74.93 0)
+      (effects (font (size 1.27 1.27)))
+    )
+    (property "Value" "Conn_01x04_Pin" (at 142.24 77.47 0)
+      (effects (font (size 1.27 1.27)))
+    )
+    (property "Footprint" "" (at 149.86 73.66 0)
+      (effects (font (size 1.27 1.27)) hide)
+    )
+    (property "Datasheet" "~" (at 149.86 73.66 0)
+      (effects (font (size 1.27 1.27)) hide)
+    )
+    (pin "1")
+    (pin "2")
+    (pin "3")
+    (pin "4")
+    (instances
+      (project "dk2_04_top"
+        (path "/87a59a99-d509-467e-85da-26d34072acb7/1a91e583-926b-4126-a95f-efd256f8eb1b"
+          (reference "J16") (unit 1)
+        )
+      )
+    )
+  )
   (symbol (lib_id "Switch:SW_Push") (at 113.03 81.28 0) (unit 1)
     (in_bom yes) (on_board yes) (dnp no) (fields_autoplaced)
@@
     )
   )
-  (symbol (lib_id "Device:R_US") (at 45.72 68.58 90) (unit 1)
-    (in_bom yes) (on_board yes) (dnp no) (fields_autoplaced)
-    (property "Reference" "R14" (at 45.72 62.23 90)
-      (effects (font (size 1.27 1.27)))
-    )
-    (property "Value" "10k" (at 45.72 64.77 90)
-      (effects (font (size 1.27 1.27)))
-    )
-    (property "Footprint" "Resistor_SMD:R_0603_1608Metric" (at 45.974 67.564 90)
-      (effects (font (size 1.27 1.27)) hide)
-    )
-    (property "Datasheet" "~" (at 45.72 68.58 0)
+  (symbol (lib_id "Device:R_US") (at 59.69 68.58 180) (unit 1)
+    (in_bom yes) (on_board yes) (dnp no) (fields_autoplaced)
+    (property "Reference" "R14" (at 61.341 67.9363 0)
+      (effects (font (size 1.27 1.27)) (justify right))
+    )
+    (property "Value" "100k" (at 61.341 69.8573 0)
+      (effects (font (size 1.27 1.27)) (justify right))
+    )
+    (property "Footprint" "Resistor_SMD:R_0603_1608Metric" (at 58.674 68.326 90)
+      (effects (font (size 1.27 1.27)) hide)
+    )
+    (property "Datasheet" "~" (at 59.69 68.58 0)
       (effects (font (size 1.27 1.27)) hide)
     )
@@
     )
   )
-  (symbol (lib_id "power:GND") (at 59.69 74.93 0) (unit 1)
-    (in_bom yes) (on_board yes) (dnp no) (fields_autoplaced)
-    (property "Reference" "#PWR029" (at 59.69 81.28 0)
-      (effects (font (size 1.27 1.27)) hide)
-    )
-    (property "Value" "GND" (at 59.69 80.01 0)
-      (effects (font (size 1.27 1.27)))
-    )
-    (property "Footprint" "" (at 59.69 74.93 0)
-      (effects (font (size 1.27 1.27)) hide)
-    )
-    (property "Datasheet" "" (at 59.69 74.93 0)
+  (symbol (lib_id "power:GND") (at 59.69 72.39 0) (unit 1)
+    (in_bom yes) (on_board yes) (dnp no) (fields_autoplaced)
+    (property "Reference" "#PWR029" (at 59.69 78.74 0)
+      (effects (font (size 1.27 1.27)) hide)
+    )
+    (property "Value" "GND" (at 59.69 77.47 0)
+      (effects (font (size 1.27 1.27)))
+    )
+    (property "Footprint" "" (at 59.69 72.39 0)
+      (effects (font (size 1.27 1.27)) hide)
+    )
+    (property "Datasheet" "" (at 59.69 72.39 0)
       (effects (font (size 1.27 1.27)) hide)
     )
@@
     )
   )
-  (symbol (lib_id "Device:R_US") (at 45.72 57.15 90) (unit 1)
-    (in_bom yes) (on_board yes) (dnp no) (fields_autoplaced)
-    (property "Reference" "R13" (at 45.72 50.8 90)
-      (effects (font (size 1.27 1.27)))
-    )
-    (property "Value" "10k" (at 45.72 53.34 90)
-      (effects (font (size 1.27 1.27)))
-    )
-    (property "Footprint" "Resistor_SMD:R_0603_1608Metric" (at 45.974 56.134 90)
-      (effects (font (size 1.27 1.27)) hide)
-    )
-    (property "Datasheet" "~" (at 45.72 57.15 0)
+  (symbol (lib_id "Device:R_US") (at 59.69 58.42 180) (unit 1)
+    (in_bom yes) (on_board yes) (dnp no) (fields_autoplaced)
+    (property "Reference" "R13" (at 61.341 57.7763 0)
+      (effects (font (size 1.27 1.27)) (justify right))
+    )
+    (property "Value" "330k" (at 61.341 59.6973 0)
+      (effects (font (size 1.27 1.27)) (justify right))
+    )
+    (property "Footprint" "Resistor_SMD:R_0603_1608Metric" (at 58.674 58.166 90)
+      (effects (font (size 1.27 1.27)) hide)
+    )
+    (property "Datasheet" "~" (at 59.69 58.42 0)
       (effects (font (size 1.27 1.27)) hide)
     )
@@
     )
   )
-  (symbol (lib_id "Connector:Conn_01x05_Pin") (at 149.86 73.66 0) (unit 1)
-    (in_bom yes) (on_board yes) (dnp no)
-    (property "Reference" "J16" (at 140.97 73.025 0)
-      (effects (font (size 1.27 1.27)))
-    )
-    (property "Value" "Conn_01x05_Pin" (at 140.97 75.565 0)
-      (effects (font (size 1.27 1.27)))
-    )
-    (property "Footprint" "Connector_PinHeader_2.54mm:PinHeader_1x05_P2.54mm_Vertical" (at 149.86 73.66 0)
-      (effects (font (size 1.27 1.27)) hide)
-    )
-    (property "Datasheet" "~" (at 149.86 73.66 0)
-      (effects (font (size 1.27 1.27)) hide)
-    )
-    (pin "1")
-    (pin "2")
-    (pin "3")
-    (pin "4")
-    (pin "5")
-    (instances
-      (project "dk2_04_top"
-        (path "/87a59a99-d509-467e-85da-26d34072acb7/1a91e583-926b-4126-a95f-efd256f8eb1b"
-          (reference "J16") (unit 1)
-        )
-      )
-    )
-  )
   (symbol (lib_id "power:GND") (at 167.64 99.06 0) (unit 1)
     (in_bom yes) (on_board yes) (dnp no) (fields_autoplaced)
@@
     )
   )
-  (symbol (lib_id "power:+12V") (at 60.96 52.07 270) (unit 1)
-    (in_bom yes) (on_board yes) (dnp no) (fields_autoplaced)
-    (property "Reference" "#PWR012" (at 57.15 52.07 0)
-      (effects (font (size 1.27 1.27)) hide)
-    )
-    (property "Value" "+12V" (at 64.135 52.3868 90)
+  (symbol (lib_id "power:+12V") (at 59.69 54.61 0) (unit 1)
+    (in_bom yes) (on_board yes) (dnp no) (fields_autoplaced)
+    (property "Reference" "#PWR012" (at 59.69 58.42 0)
+      (effects (font (size 1.27 1.27)) hide)
+    )
+    (property "Value" "+12V" (at 61.087 53.6568 0)
       (effects (font (size 1.27 1.27)) (justify left))
     )
-    (property "Footprint" "" (at 60.96 52.07 0)
-      (effects (font (size 1.27 1.27)) hide)
-    )
-    (property "Datasheet" "" (at 60.96 52.07 0)
-      (effects (font (size 1.27 1.27)) hide)
-    )
+    (property "Footprint" "" (at 59.69 54.61 0)
+      (effects (font (size 1.27 1.27)) hide)
+    )
+    (property "Datasheet" "" (at 59.69 54.61 0)
+      (effects (font (size 1.27 1.27)) hide)
+    )

Commit message: rejigged top board, smaller connectors
Parts:
- J16: footprint (none) -> Connector_PinHeader_2.54mm:PinHeader_1x04_P2.54mm_Vertical
Changed lines of the file:
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@@
       (effects (font (size 1.27 1.27)))
     )
-    (property "Footprint" "" (at 149.86 73.66 0)
+    (property "Footprint" "Connector_PinHeader_2.54mm:PinHeader_1x04_P2.54mm_Vertical" (at 149.86 73.66 0)
       (effects (font (size 1.27 1.27)) hide)
     )
