File: pcb/dk2_04_bottom/dk2_04_bottom.kicad_pcb (KiCad board)
At the start: 2 copper layers, 120 x 60 mm, 76 parts, among them J1 Conn_01x20_Pin, J2 Conn_01x16_Pin, J3 Eurorack_Power, J4 Conn_01x20_Pin, J5 Conn_01x20_Pin, J6 Conn_01x03_Pin, Q1 MMBT3904, U1 Pico, U2 AP7333-33SAG, U3 TL072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

Commit message: autosave works
Parts:
- removed D1: 1N5819WS, Diode_SMD:D_SOD-323
- removed JP1: Jumper_3_Open, Connector_PinHeader_2.54mm:PinHeader_1x03_P2.54mm_Vertical
- added C28: 2200uF, Capacitor_THT:CP_Radial_D13.0mm_P5.00mm, B.Cu at (130.1, 83.1)
- added D3: 1N5819WS, Diode_SMD:D_SOD-323, F.Cu at (131.7, 72.2)
- added JP2: SolderJumper_2_Open, Jumper:SolderJumper-2_P1.3mm_Open_Pad1.0x1.5mm, F.Cu at (128.8, 72.3)
- D2: value 1N5820 -> 1N5819WS; footprint Diode_THT:D_DO-201AD_P15.24mm_Horizontal -> Diode_SMD:D_SOD-323; moved to F.Cu
- J1: value Conn_01x20_Pin -> Left_Header; footprint Connector_PinHeader_2.54mm:PinHeader_1x20_P2.54mm_Vertical -> Connector_PinHeader_2.54mm:PinHeader_1x16_P2.54mm_Vertical
- J2: value Conn_01x16_Pin -> Right_Header; footprint Connector_PinHeader_2.54mm:PinHeader_1x16_P2.54mm_Vertical -> Connector_PinHeader_2.54mm:PinHeader_1x12_P2.54mm_Vertical
- moved D2 10.0 mm to (115.7, 72.9), turned to 180 degrees
- moved J2 5.00 mm to (196.0, 66.0)
- moved J1 2.58 mm to (84.0, 58.5)
Connections:
- C27 pad 1: +5V -> Net-(D3-A)
- C4 pad 1: Net-(JP1-A) -> +3.3VDAC
- J1 pad 1: unconnected-(J1-Pin_1-Pad1) -> 4051_ADDRESS_A
- J1 pad 10: TRIGGER_OUT_1_EURO -> TRIGGER_OUT_2_EURO
- J1 pad 11: TRIGGER_OUT_2_EURO -> TRIGGER_OUT_3_EURO
- J1 pad 12: TRIGGER_OUT_3_EURO -> TRIGGER_OUT_4_EURO
- J1 pad 13: TRIGGER_OUT_4_EURO -> SYNC_IN_EURO
- J1 pad 14: SYNC_IN_EURO -> SYNC_OUT_EURO
- J1 pad 15: SYNC_OUT_EURO -> +3.3V
- J1 pad 16: +12V -> GND
- J1 pad 2: 4051_ADDRESS_A -> 4051_ADDRESS_B
- J1 pad 3: 4051_ADDRESS_B -> 4051_ADDRESS_C
- J1 pad 4: 4051_ADDRESS_C -> 4051_READING_1
- J1 pad 5: 4051_READING_1 -> 4051_READING_0
- J1 pad 6: 4051_READING_0 -> 165_LOAD
- J1 pad 7: 165_LOAD -> 165_CLOCK
- J1 pad 8: 165_CLOCK -> 165_DATA
- J1 pad 9: 165_DATA -> TRIGGER_OUT_1_EURO
- J2 pad 1: unconnected-(J2-Pin_1-Pad1) -> SD_CLOCK
- J2 pad 10: EURO_OUT_1 -> +12V
- J2 pad 11: EURO_OUT_2 -> +3.3V
- J2 pad 12: +12V -> -12V
- J2 pad 2: unconnected-(J2-Pin_2-Pad2) -> SD_SERIAL_IN
- J2 pad 3: SD_CLOCK -> SD_SERIAL_OUT
- J2 pad 4: SD_SERIAL_IN -> SD_CHIP_SELECT
- J2 pad 5: SD_SERIAL_OUT -> 595_DATA
- J2 pad 6: SD_CHIP_SELECT -> 595_CLOCK
- J2 pad 7: 595_DATA -> 595_LATCH
- J2 pad 8: 595_CLOCK -> EURO_OUT_1
- J2 pad 9: 595_LATCH -> EURO_OUT_2
- J5 pad 2: Net-(#FLG02-pwr) -> +5V
- L1 pad 2: +5V -> Net-(D3-A)
- U1 pad 39: Net-(#FLG02-pwr) -> +5V
- U2 pad 2: Net-(JP1-A) -> +3.3VDAC
- U8 pad 3: +5V -> Net-(D3-A)
Routing:
- net +3.3VDAC: track 250.0 -> 63.8 mm, vias 1 -> 0
- net GND: track 233.0 -> 387.6 mm, vias 17 -> 19
- net +12V: track 254.5 -> 212.8 mm
- net -12V: track 204.9 -> 177.7 mm, vias 2 -> 1
- net Net-(D3-A): track 0.00 -> 23.9 mm
- net Net-(JP1-A): track 18.0 -> 0.00 mm
- net +5V: track 95.3 -> 108.3 mm, vias 0 -> 1
- net Net-(#FLG02-pwr): track 11.9 -> 0.00 mm
- net Net-(D2-K): track 30.1 -> 18.4 mm
- net +3.3V: track 266.9 -> 265.5 mm
Other:
- board text added: "Bradshaw Instruments Drumkid 2.04"
- board text removed: "AP7333 DAC PICO"
- board text removed: "Bradshaw Instruments Drumkid 2.03"
