File: pcb/dk2_04_bottom/dk2_04_bottom.kicad_sch (KiCad schematic)
At the start: 7 parts, among them J1 Conn_01x20_Pin, J2 Conn_01x16_Pin, J4 Conn_01x20_Pin, J5 Conn_01x20_Pin, J6 Conn_01x03_Pin, U1 Pico

Commit message: pcb 2.04 tweaks
Parts:
- removed D1: 1N5819WS, Diode_SMD:D_SOD-323, symbol Diode:1N5819WS
Connections:
- net +5V: now also J5.2 (Pin_2), U1.39 (VSYS)
Changed lines of the file:
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@@
     (stroke (width 0) (type default))
   )
-  (wire (pts (xy 116.84 21.59) (xy 116.84 25.4))
+  (wire (pts (xy 116.84 21.59) (xy 116.84 33.02))
     (stroke (width 0) (type default))
   )
@@
         )
       )
-    )
-  )
-  (symbol (lib_id "Diode:1N5819WS") (at 116.84 29.21 90) (unit 1)
-    (in_bom yes) (on_board yes) (dnp no) (fields_autoplaced)
-    (property "Reference" "D1" (at 118.872 28.8838 90)
-      (effects (font (size 1.27 1.27)) (justify right))
-    )
-    (property "Value" "1N5819WS" (at 118.872 30.8048 90)
-      (effects (font (size 1.27 1.27)) (justify right))
-    )
-    (property "Footprint" "Diode_SMD:D_SOD-323" (at 121.285 29.21 0)
-      (effects (font (size 1.27 1.27)) hide)
-    )
-    (property "Datasheet" "https://datasheet.lcsc.com/lcsc/2204281430_Guangdong-Hottech-1N5819WS_C191023.pdf" (at 116.84 29.21 0)
-      (effects (font (size 1.27 1.27)) hide)
-    )
-    (pin "1")
-    (pin "2")
-    (instances
-      (project "dk2_04_bottom"
-        (path "/87a59a99-d509-467e-85da-26d34072acb7"
-          (reference "D1") (unit 1)
-        )
-      )

Commit message: autosave works
Parts:
- J1: value Conn_01x20_Pin -> Left_Header; footprint Connector_PinHeader_2.54mm:PinHeader_1x20_P2.54mm_Vertical -> Connector_PinHeader_2.54mm:PinHeader_1x16_P2.54mm_Vertical; symbol Connector:Conn_01x20_Pin -> Connector:Conn_01x16_Pin
- J2: value Conn_01x16_Pin -> Right_Header; footprint Connector_PinHeader_2.54mm:PinHeader_1x16_P2.54mm_Vertical -> Connector_PinHeader_2.54mm:PinHeader_1x12_P2.54mm_Vertical; symbol Connector:Conn_01x16_Pin -> Connector:Conn_01x12_Pin
Connections:
- net +12V: now also J2.10 (Pin_10); no longer J1.16 (Pin_16), J2.12 (Pin_12)
- net +3.3V: now also J1.15 (Pin_15), J2.11 (Pin_11); no longer J1.18 (Pin_18), J2.14 (Pin_14)
- net -12V: now also J2.12 (Pin_12); no longer J1.20 (Pin_20), J2.16 (Pin_16)
- net 165_CLOCK: now also J1.7 (Pin_7); no longer J1.8 (Pin_8)
- net 165_DATA: now also J1.8 (Pin_8); no longer J1.9 (Pin_9)
- net 165_LOAD: now also J1.6 (Pin_6); no longer J1.7 (Pin_7)
- net 4051_ADDRESS_A: now also J1.1 (Pin_1); no longer J1.2 (Pin_2)
- net 4051_ADDRESS_B: now also J1.2 (Pin_2); no longer J1.3 (Pin_3)
- net 4051_ADDRESS_C: now also J1.3 (Pin_3); no longer J1.4 (Pin_4)
- net 4051_READING_0: now also J1.5 (Pin_5); no longer J1.6 (Pin_6)
- net 4051_READING_1: now also J1.4 (Pin_4); no longer J1.5 (Pin_5)
- net 595_CLOCK: now also J2.6 (Pin_6); no longer J2.8 (Pin_8)
- net 595_DATA: now also J2.5 (Pin_5); no longer J2.7 (Pin_7)
- net 595_LATCH: now also J2.7 (Pin_7); no longer J2.9 (Pin_9)
- net EURO_OUT_1: now also J2.8 (Pin_8); no longer J2.10 (Pin_10)
- net EURO_OUT_2: now also J2.9 (Pin_9); no longer J2.11 (Pin_11)
- net GND: now also J1.16 (Pin_16); no longer J1.19 (Pin_19), J2.15 (Pin_15)
- net SD_CHIP_SELECT: now also J2.4 (Pin_4); no longer J2.6 (Pin_6)
- net SD_CLOCK: now also J2.1 (Pin_1); no longer J2.3 (Pin_3)
- net SD_SERIAL_IN: now also J2.2 (Pin_2); no longer J2.4 (Pin_4)
- net SD_SERIAL_OUT: now also J2.3 (Pin_3); no longer J2.5 (Pin_5)
- net SYNC_IN_EURO: now also J1.13 (Pin_13); no longer J1.14 (Pin_14)
- net SYNC_OUT_EURO: now also J1.14 (Pin_14); no longer J1.15 (Pin_15)
- net TRIGGER_OUT_1_EURO: now also J1.9 (Pin_9); no longer J1.10 (Pin_10)
- net TRIGGER_OUT_2_EURO: now also J1.10 (Pin_10); no longer J1.11 (Pin_11)
- net TRIGGER_OUT_3_EURO: now also J1.11 (Pin_11); no longer J1.12 (Pin_12)
- net TRIGGER_OUT_4_EURO: now also J1.12 (Pin_12); no longer J1.13 (Pin_13)
- removed net +3.3VDAC: J1.17 (Pin_17), J2.13 (Pin_13)
- no-connect marks 9 -> 6
