File: pcb/dk2_04b_top/dk2_04b_top.kicad_pcb (KiCad board)
At the start: 2 copper layers, 120 x 108 mm, 114 parts, among them J1 Left_Header, J10 Sync_Out, J11 Euro_Out_2, J12 CV_In_1, J13 CV_In_2, J14 CV_In_3, J15 CV_In_4, J16 Conn_01x04_Pin, J2 Trigger_Out_1, J3 Trigger_Out_2, J4 Sync_In, J5 Euro_Out_1, J6 Micro_SD_Card, J7 Right_Header, J8 Trigger_Out_3, J9 Trigger_Out_4, SW1 SW_Push, SW10 SW_Push, SW11 SW_Push, SW12 SW_Push, SW13 SW_Push, SW14 SW_Push, SW15 SW_Push, SW16 SW_Push, SW17 SW_Push, SW18 SW_Push, SW19 SW_Push, SW2 SW_Push, SW3 SW_Push, SW4 SW_Push, SW5 SW_Push, SW6 SW_Push, SW7 SW_Push, SW8 SW_Push, SW9 SW_Push, U1 74HC595, U10 74HC165, U2 74HC595, U3 CA56-12EWA, U4 74HC165, U5 74HC165, U6 74HC4051, U7 MCP6002-xSN, U8 MCP6002-xSN, U9 74HC4051

Commit message: haven't committed for ages because i did something stupid in git
Other:
- board text added: "+"
- board text added: "Drumkid 2.04b (Eurorack)"
- board text removed: "Drumkid 2.04 (Eurorack)"
Changed lines of the file:
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@@
   (gr_circle (center 139.5 66.5) (end 143 66.5)
     (stroke (width 0.2) (type default)) (fill none) (layer "User.1"))
-  (gr_text "Drumkid 2.04 (Eurorack)" (at 84 59) (layer "F.SilkS")
+  (gr_text "+" (at 161 129.25) (layer "F.SilkS")
+    (effects (font (size 1.5 1.5) (thickness 0.3) bold) (justify left bottom))
+  )
+  (gr_text "+" (at 161 134.75) (layer "F.SilkS")
+    (effects (font (size 1.5 1.5) (thickness 0.3) bold) (justify left bottom))
+  )
+  (gr_text "+" (at 161 140.5) (layer "F.SilkS")
+    (effects (font (size 1.5 1.5) (thickness 0.3) bold) (justify left bottom))
+  )
+  (gr_text "Drumkid 2.04b (Eurorack)" (at 84 59) (layer "F.SilkS")
     (effects (font (size 3 3) (thickness 0.15)) (justify left bottom))
   )
+  (gr_text "+" (at 161 123.75) (layer "F.SilkS")
+    (effects (font (size 1.5 1.5) (thickness 0.3) bold) (justify left bottom))
+  )
   (segment (start 129.55 124.55) (end 145.513604 124.55) (width 0.25) (layer "B.Cu") (net 1))
