File: pcb/dk2_05/dk2_05.kicad_sch (KiCad schematic)
At the start: 11 parts, among them J1 Trigger_Out_1, J10 Conn_01x03_Pin, J2 Trigger_Out_2, J3 Sync_In, J4 Euro_Out_1, J5 Micro_SD_Card, J6 Trigger_Out_3, J7 Trigger_Out_4, J8 Sync_Out, J9 Euro_Out_2

Commit message: panel and pcb are aligned
Parts:
- A1: footprint Library:RaspberryPi_Pico_Common_THT -> Library:RaspberryPi_Pico_Common_THT_dk2
Changed lines of the file:
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@@
 			)
 		)
-		(property "Footprint" "Library:RaspberryPi_Pico_Common_THT"
+		(property "Footprint" "Library:RaspberryPi_Pico_Common_THT_dk2"
 			(at 62.865 -4.445 0)
 			(effects
@@
 		(dnp no)
 		(fields_autoplaced yes)
-		(property "Reference" "#PWR021"
+		(property "Reference" "#PWR016"
 			(at 211.455 -62.23 0)
 			(effects
@@
 			(project "dk2_05"
 				(path "/87a59a99-d509-467e-85da-26d34072acb7"
-					(reference "#PWR021")
+					(reference "#PWR016")
 					(unit 1)
 				)
@@
 		(dnp no)
 		(fields_autoplaced yes)
-		(property "Reference" "#PWR022"
+		(property "Reference" "#PWR017"
 			(at 212.09 77.47 0)
 			(effects
@@
 			(project "dk2_04_top"
 				(path "/87a59a99-d509-467e-85da-26d34072acb7"
-					(reference "#PWR022")
+					(reference "#PWR017")
 					(unit 1)
 				)
@@
 		(dnp no)
 		(fields_autoplaced yes)
-		(property "Reference" "#PWR0103"
+		(property "Reference" "#PWR010"
 			(at 85.725 -22.225 0)
 			(effects
@@
 			(project "dk2_05"
 				(path "/87a59a99-d509-467e-85da-26d34072acb7"
-					(reference "#PWR0103")
+					(reference "#PWR010")
 					(unit 1)
 				)
@@
 		(dnp no)
 		(fields_autoplaced yes)
-		(property "Reference" "#PWR0102"
+		(property "Reference" "#PWR08"
 			(at 62.865 -9.525 0)
 			(effects
@@
 			(project ""
 				(path "/87a59a99-d509-467e-85da-26d34072acb7"
-					(reference "#PWR0102")
-					(unit 1)
-				)
+					(reference "#PWR08")
+					(unit 1)
+				)
