File: pcb/dk2_05/dk2_05.kicad_pcb (KiCad board)
At the start: 4 copper layers, 120 x 108 mm, 189 parts, among them J1 Trigger_Out_1, J10 Conn_01x03_Pin, J11 CV_In_1, J12 CV_In_2, J13 CV_In_3, J14 CV_In_4, J15 Conn_01x04_Pin, J16 Eurorack_Power, J2 Trigger_Out_2, J3 Sync_In, J4 Euro_Out_1, J5 Micro_SD_Card, J6 Trigger_Out_3, J7 Trigger_Out_4, J8 Sync_Out, J9 Euro_Out_2, Q1 MMBT3904, SW1 SW_Push, SW10 SW_Push, SW11 SW_Push, SW12 SW_Push, SW13 SW_Push, SW14 SW_Push, SW15 SW_Push, SW16 SW_Push, SW17 SW_Push, SW18 SW_Push, SW19 SW_Push, SW2 SW_Push, SW3 SW_Push, SW4 SW_Push, SW5 SW_Push, SW6 SW_Push, SW7 SW_Push, SW8 SW_Push, SW9 SW_Push, U1 74HC595, U10 74HC165, U11 AP7333-33SAG, U12 TPS54331DR, U13 TL072, U14 PCM5102, U15 TL072, U16 TL072, U17 TL072, U2 74HC595, U3 CA56-12EWA, U4 74HC165, U5 74HC165, U6 74HC4051, U7 MCP6002-xSN, U8 MCP6002-xSN, U9 74HC4051

Commit message: all this layout stuff better be worth it
Parts:
- U15, U16, U17: moved to B.Cu
- moved R74 172.9 mm to (67.4, 140.3)
- moved R77 172.9 mm to (67.4, 132.7)
- moved R64 172.9 mm to (59.4, 140.3)
- moved R66 172.9 mm to (59.4, 135.2)
- moved R67 172.9 mm to (59.4, 132.7)
- moved R69 172.9 mm to (63.4, 140.3)
- moved R71 172.9 mm to (63.4, 135.2)
- moved R72 172.9 mm to (63.4, 132.7)
- moved R75 172.9 mm to (67.4, 137.8)
- moved R76 172.9 mm to (67.4, 135.2)
- moved R78 172.9 mm to (67.4, 130.2)
- moved R65 172.9 mm to (59.4, 137.8)
- moved R68 172.9 mm to (59.4, 130.2)
- moved R70 172.9 mm to (63.4, 137.8)
- moved R73 172.9 mm to (63.4, 130.2)
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
Commit message: layout starting to feel okay, routing will be bad..?
Parts:
- moved R56 77.1 mm to (140.5, 135.0)
- moved R51 72.3 mm to (130.0, 111.2), turned to 180 degrees
- moved R49 71.6 mm to (130.0, 109.5)
- moved R53 70.8 mm to (133.2, 114.2), turned to 180 degrees
- moved R54 68.4 mm to (136.5, 114.2), turned to 180 degrees
- moved R55 67.4 mm to (140.5, 119.0)
- moved J10 65.1 mm to (186.1, 79.3)
- moved C20 63.9 mm to (130.0, 107.8)
- moved C17 63.7 mm to (130.0, 113.0)
- moved C21 62.9 mm to (133.2, 116.0), turned to 180 degrees
- moved R52 62.0 mm to (141.0, 111.2)
- moved R50 60.9 mm to (141.0, 109.5)
- moved C22 60.6 mm to (136.5, 116.0), turned to 180 degrees
- moved U10 58.2 mm to (130.0, 74.3), turned to 180 degrees
- moved C19 53.8 mm to (141.0, 114.8)
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
Commit message: panel and pcb are aligned
Parts:
- A1: footprint Library:RaspberryPi_Pico_Common_THT -> Library:RaspberryPi_Pico_Common_THT_dk2; moved to B.Cu
- J15: moved to B.Cu
- moved J15 119.9 mm to (146.2, 58.2), turned to -90 degrees
- moved R68 46.2 mm to (104.2, 119.0)
- moved R74 37.2 mm to (104.2, 135.0)
- moved R69 35.8 mm to (92.2, 119.0)
- moved J10 32.2 mm to (185.0, 111.5), turned to 0 degrees
- moved R41 32.1 mm to (157.8, 117.8)
- moved R42 32.1 mm to (156.1, 117.8)
- moved R65 27.4 mm to (75.8, 115.8)
- moved R75 25.0 mm to (92.2, 135.0)
- moved R64 22.2 mm to (75.8, 125.2)
- moved R67 21.4 mm to (72.5, 115.8)
- moved A1 18.1 mm to (181.5, 101.5), turned to 90 degrees
- moved R66 16.5 mm to (72.5, 125.2)
- moved R71 14.8 mm to (75.8, 127.0)
- moved R70 12.4 mm to (75.8, 136.2)
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
Commit message: started routing
Routing:
- net TRIGGER_OUT_2: track 0.00 -> 151.8 mm, vias 0 -> 2
- net Net-(U1-QD): track 0.00 -> 55.8 mm, vias 0 -> 2
- net Net-(U2-QH): track 0.00 -> 54.8 mm, vias 0 -> 2
- net Net-(U1-QH): track 0.00 -> 51.5 mm, vias 0 -> 2
- net Net-(U2-QG): track 0.00 -> 44.6 mm, vias 0 -> 2
- net Net-(U2-QE): track 0.00 -> 44.2 mm
- net Net-(U2-QF): track 0.00 -> 44.2 mm, vias 0 -> 2
- net Net-(U1-QE): track 0.00 -> 37.9 mm
- net Net-(U1-QC): track 0.00 -> 37.3 mm, vias 0 -> 2
- net Net-(U1-QB): track 0.00 -> 35.4 mm, vias 0 -> 2
- net Net-(U1-QF): track 0.00 -> 29.6 mm, vias 0 -> 2
- net Net-(U1-QG): track 0.00 -> 27.7 mm, vias 0 -> 2
- net Net-(U1-QA): track 0.00 -> 26.0 mm
- net Net-(U2-QA): track 0.00 -> 25.6 mm, vias 0 -> 2
- net Net-(U2-QB): track 0.00 -> 20.9 mm
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- added copper zone on In2.Cu, net +3.3V
- added copper zone on In1.Cu, net GND

Commit message: routing going well
Parts:
- moved U6 2.38 mm to (89.9, 58.7)
- moved R32 2.05 mm to (125.2, 119.5)
- moved R38 1.80 mm to (125.2, 135.3)
- moved U4 1.61 mm to (90.0, 74.7)
- moved R36 1.60 mm to (126.8, 135.3)
- moved R30 1.30 mm to (126.8, 119.5)
- moved U9 1.25 mm to (110.0, 58.5)
- moved U5 0.70 mm to (110.1, 75.0)
Routing:
- net 595_DATA: track 0.00 -> 46.1 mm, vias 0 -> 1
- net 595_LATCH: track 0.00 -> 45.7 mm, vias 0 -> 1
- net 595_CLOCK: track 0.00 -> 38.4 mm, vias 0 -> 3
- net GND: track 0.00 -> 31.9 mm, vias 0 -> 3
- net +12V: track 0.00 -> 29.1 mm
- net +3.3V: track 8.75 -> 37.5 mm, vias 0 -> 3
- net SD_SERIAL_OUT: track 0.00 -> 24.2 mm
- net SD_CHIP_SELECT: track 0.00 -> 23.5 mm
- net +5V: track 0.00 -> 22.4 mm
- net SD_CLOCK: track 0.00 -> 16.6 mm
- net Net-(U7B--): track 0.00 -> 16.1 mm
- net SD_SERIAL_IN: track 0.00 -> 15.7 mm
- net Net-(U8B--): track 0.00 -> 15.1 mm
- net Net-(U1-QH'): track 0.00 -> 14.5 mm
- net Net-(U8A--): track 0.00 -> 14.3 mm
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
Commit message: more routing
Parts:
- moved R62 1.45 mm to (80.8, 118.8), turned to 180 degrees
- turned U6 to 180 degrees
Routing:
- net 4051_READING_0: track 2.54 -> 89.0 mm, vias 0 -> 1
- net Net-(U9-A3): track 0.00 -> 85.4 mm, vias 0 -> 2
- net Net-(U10-D0): track 0.00 -> 85.3 mm
- net 4051_ADDRESS_B: track 2.54 -> 85.6 mm, vias 0 -> 2
- net 4051_ADDRESS_C: track 2.54 -> 83.5 mm, vias 0 -> 2
- net 4051_ADDRESS_A: track 2.54 -> 83.1 mm, vias 0 -> 2
- net 4051_READING_1: track 2.54 -> 80.9 mm, vias 0 -> 2
- net Net-(U6-A3): track 0.00 -> 75.7 mm
- net Net-(U9-A2): track 0.00 -> 72.3 mm, vias 0 -> 2
- net Net-(U5-D7): track 0.00 -> 69.5 mm
- net Net-(U6-A7): track 0.00 -> 63.3 mm, vias 0 -> 2
- net Net-(U9-A0): track 0.00 -> 57.3 mm
- net CV_IN_1: track 4.10 -> 45.9 mm, vias 0 -> 2
- net CV_IN_3: track 4.10 -> 44.6 mm, vias 0 -> 2
- net Net-(U6-A2): track 0.00 -> 38.9 mm
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
Commit message: ROUTING
Routing:
- net +12V: track 55.1 -> 223.6 mm, vias 0 -> 4
- net -12V: track 14.4 -> 175.3 mm, vias 0 -> 5
- net GND: track 47.2 -> 188.2 mm, vias 3 -> 38
- net SYNC_OUT: track 2.54 -> 100.1 mm, vias 0 -> 3
- net Net-(U10-D2): track 9.86 -> 91.7 mm, vias 0 -> 3
- net Net-(U10-D1): track 9.86 -> 81.4 mm, vias 0 -> 3
- net CV_IN_4: track 41.8 -> 111.5 mm, vias 2 -> 4
- net CV_IN_3: track 44.6 -> 110.4 mm, vias 2 -> 4
- net Net-(U5-D2): track 10.0 -> 62.9 mm, vias 0 -> 1
- net +5V: track 22.4 -> 75.0 mm
- net CV_IN_2: track 39.9 -> 90.0 mm, vias 2 -> 4
- net CV_IN_1: track 45.9 -> 95.5 mm, vias 2 -> 4
- net Net-(U5-D5): track 10.0 -> 58.0 mm, vias 0 -> 1
- net Net-(D6-A): track 0.00 -> 46.8 mm
- net Net-(U5-D3): track 10.0 -> 56.7 mm, vias 0 -> 1
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
Commit message: 27 unrouted, nearly there...
Routing:
- net TRIGGER_OUT_4: track 2.54 -> 116.4 mm, vias 0 -> 4
- net TRIGGER_OUT_3: track 2.54 -> 92.1 mm, vias 0 -> 4
- net 165_LOAD: track 2.54 -> 87.9 mm, vias 0 -> 4
- net 165_CLOCK: track 2.54 -> 87.8 mm, vias 0 -> 4
- net SYNC_IN: track 5.81 -> 85.6 mm, vias 0 -> 2
- net 12V DETECTION: track 2.38 -> 77.2 mm, vias 0 -> 4
- net TRIGGER_OUT_1: track 2.54 -> 75.1 mm, vias 0 -> 4
- net Net-(R66-Pad1): track 2.87 -> 67.2 mm, vias 0 -> 4
- net -12V: track 175.3 -> 212.2 mm, vias 5 -> 7
- net +5V: track 75.0 -> 111.5 mm, vias 0 -> 2
- net 165_DATA: track 2.54 -> 31.5 mm, vias 0 -> 1
- net LINE_OUT_R: track 1.65 -> 27.4 mm, vias 0 -> 2
- net Net-(C22-Pad2): track 13.0 -> 34.4 mm
- net LINE_OUT_L: track 1.65 -> 22.8 mm, vias 0 -> 2
- net GND: track 188.2 -> 203.6 mm, vias 38 -> 40
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