File: pcb/dk2_05/power.kicad_sch (KiCad schematic)
At the start: 21 parts, among them J16 Eurorack_Power, U11 AP7333-33SAG, U12 TPS54331DR

Commit message: jlcpcb stuff done
Parts:
- R46: value 42.2k -> 43.2k
- R47: value 10.2k -> 10k
- R48: value 1.69k -> 1.65k
Changed lines of the file:
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@@
 		)
 	)
-	(text_box "These two resistors form a divider which determines the output voltage using the following formula:\nVout = Vref x (Rtop / Rbottom + 1)\n(where Vref = 0.8V, see datasheet). Aiming for 5.6V to negate diode drop."
+	(text_box "These two resistors form a divider which determines the output voltage using the following formula:\nVout = Vref x (Rtop / Rbottom + 1)\n(where Vref = 0.8V, see datasheet). Aiming for 5.7V, should be dropped to ~5.3V with diode drop, 5.5V absolute max, within Pico specs."
 		(exclude_from_sim no)
 		(at 178.435 127 0)
-		(size 26.67 24.13)
+		(size 26.67 29.21)
 		(margins 0.9525 0.9525 0.9525 0.9525)
 		(stroke
@@
 			)
 		)
-		(property "Value" "42.2k"
+		(property "Value" "43.2k"
 			(at 143.256 123.1321 0)
 			(effects
@@
 			)
 		)
-		(property "Value" "1.69k"
+		(property "Value" "1.65k"
 			(at 173.736 123.1321 0)
 			(effects
@@
 			)
 		)
-		(property "Value" "10.2k"
+		(property "Value" "10k"
 			(at 173.736 115.5121 0)
 			(effects
