File: pcb/dk2_05_panel/dk2_05_panel.kicad_pcb (KiCad board)
At the start: 2 copper layers, 121.9 x 128.5 mm, 51 parts

Commit message: all this layout stuff better be worth it
Parts:
- moved H52 1.82 mm to (107.0, 115.5)
- moved H53 1.82 mm to (107.0, 121.0)
- moved H54 1.82 mm to (107.0, 126.6)
- moved H55 1.82 mm to (107.0, 132.2)

Commit message: panel and pcb are aligned
Parts:
- H1, H2, H3, H4: value Rail -> RAIL
- H10: value Kick -> KICK
- H11: value Snare -> SNARE
- H12, H40: value Chance -> CHANCE
- H13, H46: value Vel -> VEL
- H14: value Out 1 -> OUT 1
- H15, H9: value Clock -> CLOCK
- H16: value Hat -> HAT
- H17: value Tom -> TOM
- H18, H45: value Pitch -> PITCH
- H19, H41: value Zoom -> ZOOM
- H20: value Out 2 -> OUT 2
- H21: value Play -> PLAY
- H22: value Tap -> TAP
- H23: value Live -> LIVE
- H24: value Step -> STEP
- H26: value Save -> SAVE
- H27: value Beat -> BEAT
- H28: value Tempo -> TEMPO
- H29: value Tuplet -> TUPLET
- H31: value Menu -> MENU
- H32: value Kit -> KIT
- H33: value T.sig -> T.SIG
- H34: value Clear -> CLEAR
- H35: value Back -> BACK
- H38: value Yes -> YES
- H42: value Cluster -> CLUSTER
- H43: value Crop -> CROP
- H44: value Crush -> CRUSH
- H47: value Vel range -> VEL RANGE
- H48: value Magnet -> MAGNET
- H49: value Swing -> SWING
- H50: value Drop rand -> DROP RAND
- H51: value Drop all -> DROP ALL
- H52: value Error -> ERROR
- H53: value Pulse -> PULSE
- H54: value Clock in -> CLOCK IN
- H55: value Clock out -> CLOCK OUT
- moved H21 52.6 mm to (82.5, 85.5)
- moved H22 52.6 mm to (92.5, 85.5)
- moved H23 52.6 mm to (102.5, 85.5)
- moved H24 52.6 mm to (112.5, 85.5)
- moved H25 52.6 mm to (122.5, 85.5)
- moved H26 52.6 mm to (82.5, 97.5)
- moved H27 52.6 mm to (92.5, 97.5)
- moved H28 52.6 mm to (102.5, 97.5)
- moved H29 52.6 mm to (112.5, 97.5)
- moved H30 52.6 mm to (122.5, 97.5)
- moved H31 52.6 mm to (82.5, 109.5)
- moved H32 52.6 mm to (92.5, 109.5)
- moved H33 52.6 mm to (102.5, 109.5)
- moved H34 52.6 mm to (112.5, 109.5)
- moved H35 52.6 mm to (122.5, 109.5)
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Other:
- outline, holes or cut-outs redrawn
- board text added: "exec(open({dblquote}./allcaps.py{dblquote}).read())"
