File: pcb/dk2_07/dk2_07.kicad_pcb (KiCad board)
At the start: 4 copper layers, 120 x 108 mm, 189 parts, among them J1 Trigger_Out_1, J10 Conn_01x03_Pin, J11 CV_In_1, J12 CV_In_2, J13 CV_In_3, J14 CV_In_4, J15 Conn_01x04_Pin, J16 Eurorack_Power, J2 Trigger_Out_2, J3 Sync_In, J4 Euro_Out_1, J5 Micro_SD_Card, J6 Trigger_Out_3, J7 Trigger_Out_4, J8 Sync_Out, J9 Euro_Out_2, Q1 MMBT3904, SW1 SW_Push, SW10 SW_Push, SW11 SW_Push, SW12 SW_Push, SW13 SW_Push, SW14 SW_Push, SW15 SW_Push, SW16 SW_Push, SW17 SW_Push, SW18 SW_Push, SW19 SW_Push, SW2 SW_Push, SW3 SW_Push, SW4 SW_Push, SW5 SW_Push, SW6 SW_Push, SW7 SW_Push, SW8 SW_Push, SW9 SW_Push, U1 74HC595, U10 74HC165, U11 AP7333-33SAG, U12 TPS54331DR, U13 TL072, U14 PCM5102, U15 TL072, U16 TL072, U17 TL072, U2 74HC595, U3 CA56-12EWA, U4 74HC165, U5 74HC165, U6 74HC4051, U7 MCP6002-xSN, U8 MCP6002-xSN, U9 74HC4051

Commit message: pcb v2.07 nearly done
Other:
- board text added: "-"
- board text added: "BACK"
- board text added: "Bradshaw Instruments Drumkid 2.07 (Eurorack)"
- board text added: "FRONT"
- board text added: "Header goes on inner row, here"
- board text added: "Ignore (extra digital input pins)"
- board text added: "Long leg on LED is positive"
- board text added: "Order of operations: 1) Solder these parts: a Display (front, raised) b SD socket (front) c Pico headers (back) d Power socket (back) 2) Place front parts: a Pots with detents b Pots without detents c Buttons d 3.5mm jacks e LEDs with spacers 3) Add display filter 4) Add front panel 5) Add 4x washers/nuts 6) Solder placed parts 7) Solder Pico pins 8) Fit Pico into headers 9) All washers/nuts"
- board text added: "Outer row is breakout, nothing goes here"
- board text added: "RED STRIPE (-12V)"
- board text added: "RX G TX"
- board text added: "detent"
- board text removed: "Drumkid 2.06 (Eurorack)"
Changed lines of the file:
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@@
 		(layer "Edge.Cuts")
 	)
+	(gr_text "-"
+		(at 154.8 128.45 180)
+		(layer "F.SilkS")
+		(effects
+			(font
+				(size 1.5 1.5)
+				(thickness 0.3)
+				(bold yes)
+			)
+			(justify left bottom)
+		)
+	)
+	(gr_text "-"
+		(at 154.8 122.7 180)
+		(layer "F.SilkS")
+		(effects
+			(font
+				(size 1.5 1.5)
+				(thickness 0.3)
+				(bold yes)
+			)
+			(justify left bottom)
+		)
+	)
+	(gr_text "Order of operations:\n1) Solder these parts:\n  a Display (front, raised)\n  b SD socket (front)\n  c Pico headers (back)\n  d Power socket (back)\n2) Place front parts:\n  a Pots with detents\n  b Pots without detents\n  c Buttons\n  d 3.5mm jacks\n  e LEDs with spacers\n3) Add display filter\n4) Add front panel\n5) Add 4x washers/nuts\n6) Solder placed parts\n7) Solder Pico pins\n8) Fit Pico into headers\n9) All washers/nuts"
+		(at 169 145 0)
+		(layer "F.SilkS")
+		(effects
+			(font
+				(size 1 1)
+				(thickness 0.15)
+			)
+			(justify left bottom)
+		)
+	)
+	(gr_text "-"
+		(at 154.8 133.95 180)
+		(layer "F.SilkS")
+		(effects
+			(font
+				(size 1.5 1.5)
+				(thickness 0.3)
+				(bold yes)
+			)
+			(justify left bottom)
+		)
+	)
+	(gr_text "detent"
+		(at 180 56 0)
+		(layer "F.SilkS")
+		(effects
+			(font
+				(size 1 1)
+				(thickness 0.15)
+			)
+			(justify bottom)
+		)
+	)
+	(gr_text "Long leg on LED\nis positive"
+		(at 151.4 145.5 0)
+		(layer "F.SilkS")
+		(effects
+			(font
+				(size 1 1)
+				(thickness 0.15)
+			)
+			(justify left bottom)
+		)
+	)
+	(gr_text "detent"
+		(at 140 78 0)
+		(layer "F.SilkS")
+		(effects
+			(font
+				(size 1 1)
+				(thickness 0.15)
+			)
+			(justify bottom)
+		)
+	)
+	(gr_text "-"
+		(at 154.8 139.45 180)
+		(layer "F.SilkS")
+		(effects
+			(font
+				(size 1.5 1.5)
+				(thickness 0.3)
+				(bold yes)
+			)
+			(justify left bottom)
+		)
+	)
+	(gr_text "detent"
+		(at 160 78 0)
+		(layer "F.SilkS")
+		(effects
+			(font
+				(size 1 1)
+				(thickness 0.15)
+			)
+			(justify bottom)
+		)
+	)
+	(gr_text "detent"
+		(at 180 78 0)
+		(layer "F.SilkS")
+		(effects
+			(font
+				(size 1 1)
+				(thickness 0.15)
+			)
+			(justify bottom)
+		)
+	)
 	(gr_text "+"
 		(at 159.25 129.75 0)
@@
 		)
 	)
-	(gr_text "Drumkid 2.06 (Eurorack)"
-		(at 84 59 0)
+	(gr_text "Bradshaw Instruments\nDrumkid 2.07 (Eurorack)"
+		(at 86.4 61.8 0)
+		(layer "F.SilkS")
+		(effects
+			(font
+				(size 2.5 2.5)
+				(thickness 0.3125)
+			)
+			(justify left bottom)
+		)
+	)
+	(gr_text "+"
+		(at 159.25 124.25 0)
+		(layer "F.SilkS")
+		(effects
+			(font
+				(size 1.5 1.5)
+				(thickness 0.3)
+				(bold yes)
+			)
+			(justify left bottom)
+		)
+	)
+	(gr_text "FRONT"
+		(at 162.4 60.6 0)
 		(layer "F.SilkS")
 		(effects
 			(font
 				(size 3 3)
-				(thickness 0.15)
-			)
-			(justify left bottom)
-		)
-	)
-	(gr_text "+"
-		(at 159.25 124.25 0)
-		(layer "F.SilkS")
-		(effects
-			(font
-				(size 1.5 1.5)
-				(thickness 0.3)
-				(bold yes)
-			)
-			(justify left bottom)
-		)
-	)
-	(gr_text "+"
-		(at 158.5 132.25 180)
-		(layer "B.SilkS")
-		(effects
-			(font
-				(size 1.5 1.5)
-				(thickness 0.3)
-				(bold yes)
-			)
-			(justify left bottom mirror)
-		)
-	)
-	(gr_text "+"
-		(at 158.5 126.75 180)
-		(layer "B.SilkS")
-		(effects
-			(font
-				(size 1.5 1.5)
-				(thickness 0.3)
-				(bold yes)
-			)
-			(justify left bottom mirror)
-		)
-	)
-	(gr_text "+"
-		(at 158.5 137.75 180)
-		(layer "B.SilkS")
-		(effects
-			(font
-				(size 1.5 1.5)
-				(thickness 0.3)
-				(bold yes)
-			)
-			(justify left bottom mirror)
-		)
-	)
-	(gr_text "+"
-		(at 158.5 121 180)
-		(layer "B.SilkS")
-		(effects
-			(font
-				(size 1.5 1.5)
-				(thickness 0.3)
-				(bold yes)
-			)
-			(justify left bottom mirror)
+				(thickness 0.375)
+			)
+			(justify left bottom)
+		)
+	)
+	(gr_text "Outer row is breakout, nothing goes here"
+		(at 165.8 106.1 0)
+		(layer "B.SilkS")
+		(effects
+			(font
+				(size 1 1)
+				(thickness 0.15)
+			)
+			(justify left bottom mirror)
+		)
+	)
+	(gr_text "Header goes on inner row, here"
+		(at 157.36 100.15 0)
+		(layer "B.SilkS")
+		(effects
+			(font
+				(size 1 1)
+				(thickness 0.15)
+			)
+			(justify left bottom mirror)
+		)
+	)
+	(gr_text "Ignore\n(extra digital\ninput pins)"
+		(at 154.5 64.3 0)
+		(layer "B.SilkS")
+		(effects
+			(font
+				(size 1 1)
+				(thickness 0.15)
+			)
+			(justify left bottom mirror)
+		)
+	)
+	(gr_text "BACK"
+		(at 175.7 60.6 0)
+		(layer "B.SilkS")
+		(effects
+			(font
+				(size 3 3)
+				(thickness 0.375)
+			)
+			(justify left bottom mirror)
+		)
+	)
+	(gr_text "RED\nSTRIPE\n(-12V)"
+		(at 168.8 139.5 0)
+		(layer "B.SilkS")
+		(effects
+			(font
+				(size 1 1)
+				(thickness 0.15)
+			)
+			(justify left bottom mirror)
+		)
+	)
+	(gr_text "Header goes on inner row, here"
+		(at 156.7 86.4 0)
+		(layer "B.SilkS")
+		(effects
+			(font
+				(size 1 1)
+				(thickness 0.15)
+			)
+			(justify left bottom mirror)
+		)
+	)
+	(gr_text "RX\nG\nTX"
+		(at 186.4 112.6 0)
+		(layer "B.SilkS")
+		(effects
+			(font
+				(size 1.6 1.6)
+				(thickness 0.2)
+			)
+			(justify right bottom mirror)
+		)
+	)
+	(gr_text "Outer row is breakout, nothing goes here"
+		(at 166.8 80.2 0)
+		(layer "B.SilkS")
+		(effects
+			(font
+				(size 1 1)
+				(thickness 0.15)
+			)
+			(justify left bottom mirror)

Commit message: better led placement
Parts:
- moved R1 13.4 mm to (164.2, 136.5), turned to 0 degrees
- moved R2 10.9 mm to (164.2, 139.8), turned to 0 degrees
- moved R3 9.93 mm to (165.5, 143.0), turned to 0 degrees
- moved R4 7.73 mm to (165.5, 146.2), turned to 0 degrees
Routing:
- net Net-(D1-A): track 2.22 -> 15.1 mm
- net Net-(U2-QE): track 44.2 -> 56.4 mm
- net Net-(U2-QF): track 44.2 -> 55.8 mm
- net Net-(D2-A): track 2.11 -> 12.8 mm
- net Net-(D3-A): track 2.34 -> 11.1 mm
- net Net-(U2-QG): track 44.6 -> 53.2 mm
- net Net-(D4-A): track 2.15 -> 8.94 mm
- net Net-(U2-QH): track 54.8 -> 60.7 mm

Commit message: serial number silkscreen, assembly order adjusted
Other:
- board text added: "Order of operations: 1) Solder these parts: a Display (front, raised) b SD socket (front) c Pico headers (back) d Buttons (front) e Power socket (back) 2) Place front parts: a Pots with detents b Pots without detents c 3.5mm jacks d LEDs with spacers 3) Add display filter 4) Add front panel 5) Add 4x washers/nuts 6) Solder placed parts 7) Solder Pico pins 8) Fit Pico into headers 9) All washers/n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"
- board text added: "QC"
- board text added: "serial number:"
- board text removed: "Order of operations: 1) Solder these parts: a Display (front, raised) b SD socket (front) c Pico headers (back) d Power socket (back) 2) Place front parts: a Pots with detents b Pots without detents c Buttons d 3.5mm jacks e LEDs with spacers 3) Add display filter 4) Add front panel 5) Add 4x washers/nuts 6) Solder placed parts 7) Solder Pico pins 8) Fit Pico into headers 9) All washers/nuts"
Changed lines of the file:
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@@
+	)
+	(gr_rect
+		(start 165.75 58.25)
+		(end 188.75 64.25)
+		(stroke
+			(width 0.2)
+			(type solid)
+		)
+		(fill yes)
+		(layer "B.SilkS")
+	)
+	(gr_rect
+		(start 157 58.25)
+		(end 163.5 64.25)
+		(stroke
+			(width 0.2)
+			(type solid)
+		)
+		(fill yes)
+		(layer "B.SilkS")
 	)
 	(gr_rect
@@
 		)
 	)
-	(gr_text "Order of operations:\n1) Solder these parts:\n  a Display (front, raised)\n  b SD socket (front)\n  c Pico headers (back)\n  d Power socket (back)\n2) Place front parts:\n  a Pots with detents\n  b Pots without detents\n  c Buttons\n  d 3.5mm jacks\n  e LEDs with spacers\n3) Add display filter\n4) Add front panel\n5) Add 4x washers/nuts\n6) Solder placed parts\n7) Solder Pico pins\n8) Fit Pico into headers\n9) All washers/nuts"
+	(gr_text "Order of operations:\n1) Solder these parts:\n  a Display (front, raised)\n  b SD socket (front)\n  c Pico headers (back)\n  d Buttons (front)\n  e Power socket (back)\n2) Place front parts:\n  a Pots with detents\n  b Pots without detents\n  c 3.5mm jacks\n  d LEDs with spacers\n3) Add display filter\n4) Add front panel\n5) Add 4x washers/nuts\n6) Solder placed parts\n7) Solder Pico pins\n8) Fit Pico into headers\n9) All washers/nuts"
 		(at 169 145 0)
 		(layer "F.SilkS")
@@
 		)
 	)
+	(gr_text "serial number:"
+		(at 189 57.75 0)
+		(layer "B.SilkS")
+		(effects
+			(font
+				(size 1.5 1.5)
+				(thickness 0.3)
+				(bold yes)
+			)
+			(justify left bottom mirror)
+		)
+	)
 	(gr_text "Header goes on inner row, here"
 		(at 157.36 100.15 0)
@@
 		)
 	)
+	(gr_text "QC"
+		(at 163.75 57.75 0)
+		(layer "B.SilkS")
+		(effects
+			(font
+				(size 1.5 1.5)
+				(thickness 0.3)
+				(bold yes)
+			)
+			(justify left bottom mirror)
+		)
+	)
 	(gr_text "Ignore\n(extra digital\ninput pins)"
 		(at 154.5 64.3 0)
@@
 	)
 	(gr_text "BACK"
-		(at 175.7 60.6 0)
-		(layer "B.SilkS")
-		(effects
+		(at 135.75 60.75 0)
+		(layer "B.SilkS")
+		(effects

Commit message: firmware v2 started
Other:
- board text added: "Use spacers for 7-segment display! Do not solder directly to PCB!"
Changed lines of the file:
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@@
+		)
+	)
+	(gr_text "Use spacers for 7-segment\ndisplay! Do not solder\ndirectly to PCB!"
+		(at 152.5 94.75 0)
+		(layer "F.SilkS")
+		(effects
+			(font
+				(size 1 1)
+				(thickness 0.15)
+			)
+			(justify left bottom)
 		)
 	)
@@
 	)
 	(gr_text "Long leg on LED\nis positive"
-		(at 151.4 145.5 0)
+		(at 150.25 120.75 0)
 		(layer "F.SilkS")
 		(effects

Commit message: looking at ways to do longer samples for v2 firmware
Other:
- board text added: "JLCJLCJLCJLC"
Changed lines of the file:
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@@
+		)
+	)
+	(gr_text "JLCJLCJLCJLC"
+		(at 78.25 92.25 0)
+		(layer "F.SilkS")
+		(effects
+			(font
+				(size 1 1)
+				(thickness 0.15)
+			)
+			(justify left bottom)
 		)
 	)
